File: TSAL_NEW/KiCad/TSAL/TSAL.sch (KiCad schematic (older format))
At the start: 6 parts

Commit message: More TSAL work
More TSAL work
Parts:
- added J2: HV GND, symbol Connector_Generic:Conn_01x02
- added J3, J4, J5: Conn_01x02, symbol Connector_Generic:Conn_01x02
- added Q1: BSS84, Package_TO_SOT_SMD:SOT-23, symbol Transistor_FET:BSS84
- added R?: 180k, symbol Device:R_US
- added R?: 20k, symbol Device:R_US
- added U3: LDB-350L, symbol AERO_custom_symbols:LDB-350L
- C1: renamed from C?; value C -> 2u
- R1: renamed from R?; value R -> 100k
- R2: renamed from R?; value R -> 235k
- gave numbers to parts that had none: 3
Connections:
- net labels added: +12V, +24V, 555_OUTPUT, LED_GREEN+, LED_RED+
- net labels removed: HV-
- wire segments 20 -> 65
Other:
- note added: "Buck Converter\n12V --> 24V"
- note added: "HV GND"
- note added: "HV INPUT"
- note added: "Have removable jumper or similar to allow disabling green\n"
- note added: "LED OUTPUT CONNECTORS"
- note added: "Part DOES meet clearence reqs"
- note added: "RED LED\n2.8Hz Driver"
- note added: "Still need isolated gnd"
- note added: "This part only supplies 250mA, check all datasheets\n"
- note added: "Use SCWN03A-12 to isolate HV ground from GND, GND should be GLV GND"
- moved on the sheet: C1, R1, R2, U2

Commit message: update
Parts:
- added C?: .1u, symbol Device:C
- added J?: Conn_01x02, symbol Connector_Generic:Conn_01x02
- added U?: HCPL-314J, Package_SO:SOIC-16W-12_7.5x10.3mm_P1.27mm, symbol Driver_FET:HCPL-314J
- U3: symbol AERO_custom_symbols:LDB-350L -> AERO:LDB-350L
Connections:
- net labels added: +12VA, GLV+, GNDA
- wire segments 65 -> 76
Other:
- note added: "Boost Converter\n12V --> 24V"
- note removed: "Buck Converter\n12V --> 24V"
- note removed: "HV GND"
- note removed: "Still need isolated gnd"
- note removed: "Use SCWN03A-12 to isolate HV ground from GND, GND should be GLV GND"
- moved on the sheet: C1, J1, J2, Q1, R1, R2, R?, U1, U2

Commit message: add Green LED driver
Parts:
- added Q?: BSS84, Package_TO_SOT_SMD:SOT-23, symbol Transistor_FET:BSS84
- added R? (x3): R, symbol Device:R
- U3: symbol AERO:LDB-350L -> TSAL-rescue:LDB-350L-AERO
Connections:
- wire segments 76 -> 87
Other:
- note added: "GLV Input"
- note added: "GREEN is on when GLV+ is present\noff when 12V (from optoisolator) is present"
- note added: "HIGH VOLTAGE"
- note removed: "Have removable jumper or similar to allow disabling green\n"
- note removed: "Part DOES meet clearence reqs"
- note removed: "This part only supplies 250mA, check all datasheets\n"
- moved on the sheet: C?, J1, J2, J3, J4, J5, J?, R?, U1

Commit message: TSAL Comments
Parts:
- removed C?: .1u, symbol Device:C
- removed R?: R, symbol Device:R
- removed U?: HCPL-314J, Package_SO:SOIC-16W-12_7.5x10.3mm_P1.27mm, symbol Driver_FET:HCPL-314J
- added R?: R_US, symbol Device:R_US
- added R?: 10k, symbol Device:R_US
- added U?: LTV-817S, Package_DIP:SMDIP-4_W9.53mm, symbol Isolator:LTV-817S
- C1: value 2u -> 0.1uF
- R1: value 100k -> 28.7k
- R2: value 235k -> 7.19M
Connections:
- wire segments 87 -> 81
Other:
- note added: "Better connector; Figure out how will interface with HV int board, or consider HV connector board\n"
- note added: "Boost is not necessary, unless you want it\n"
- note added: "Please check this, something seems wrong\n"
- note added: "Spice sim?\n"
- note added: "Technically LED can run off just 10V, VS=10-30V"
- note added: "Why this opto? weird weird choice\n"
- note added: "name your nets better plz"
Changed lines of the file:
@@
 EESchema Schematic File Version 4
+LIBS:TSAL-cache
 EELAYER 30 0
 EELAYER END
@@
 P 6425 1925
 F 0 "R1" H 6495 1971 50  0000 L CNN
-F 1 "100k" H 6495 1880 50  0000 L CNN
+F 1 "28.7k" H 6495 1880 50  0000 L CNN
 F 2 "" V 6355 1925 50  0001 C CNN
 F 3 "~" H 6425 1925 50  0001 C CNN
@@
 P 6425 2475
 F 0 "R2" H 6495 2521 50  0000 L CNN
-F 1 "235k" H 6495 2430 50  0000 L CNN
+F 1 "7.19M" H 6495 2430 50  0000 L CNN
 F 2 "" V 6355 2475 50  0001 C CNN
 F 3 "~" H 6425 2475 50  0001 C CNN
@@
 P 6425 2925
 F 0 "C1" H 6310 2879 50  0000 R CNN
-F 1 "2u" H 6310 2970 50  0000 R CNN
+F 1 "0.1uF" H 6310 2970 50  0000 R CNN
 F 2 "" H 6463 2775 50  0001 C CNN
 F 3 "~" H 6425 2925 50  0001 C CNN
@@
 $EndComp
 $Comp
-L Driver_FET:HCPL-314J U?
-U 1 1 5E33883D
-P 1875 3325
-F 0 "U?" H 1875 3842 50  0000 C CNN
-F 1 "HCPL-314J" H 1875 3751 50  0000 C CNN
-F 2 "Package_SO:SOIC-16W-12_7.5x10.3mm_P1.27mm" H 1875 2925 50  0001 C CIN
-F 3 "https://docs.broadcom.com/docs/AV02-0169EN" H 1785 3330 50  0001 L CNN
-	1    1875 3325
-	1    0    0    -1
-$EndComp
-$Comp
 L power:+12VA #PWR?
 U 1 1 5E33E334
@@
 	3600 1525 3600 1625
 Connection ~ 3600 1625
-$Comp
-L power:+12VA #PWR?
-U 1 1 5E34005F
-P 1275 3025
-F 0 "#PWR?" H 1275 2875 50  0001 C CNN
-F 1 "+12VA" H 1290 3198 50  0000 C CNN
-F 2 "" H 1275 3025 50  0001 C CNN
-F 3 "" H 1275 3025 50  0001 C CNN
-	1    1275 3025
-	1    0    0    -1
-$EndComp
-Wire Wire Line
-	1275 3025 1475 3025
-$Comp
-L power:GNDA #PWR?
-U 1 1 5E341B32
-P 1300 3625
-F 0 "#PWR?" H 1300 3375 50  0001 C CNN
-F 1 "GNDA" H 1305 3452 50  0000 C CNN
-F 2 "" H 1300 3625 50  0001 C CNN
-F 3 "" H 1300 3625 50  0001 C CNN
-	1    1300 3625
-	1    0    0    -1
-$EndComp
-Wire Wire Line
-	1300 3625 1475 3625
-$Comp
-L Device:C C?
-U 1 1 5E34385B
-P 2750 3325
-F 0 "C?" H 2865 3371 50  0000 L CNN
-F 1 ".1u" H 2865 3280 50  0000 L CNN
-F 2 "" H 2788 3175 50  0001 C CNN
-F 3 "~" H 2750 3325 50  0001 C CNN
-	1    2750 3325
-	1    0    0    -1
-$EndComp
-Wire Wire Line
-	2275 3025 2750 3025
-Wire Wire Line
-	2750 3025 2750 3175
-Wire Wire Line
-	2275 3625 2750 3625
-Wire Wire Line
-	2750 3625 2750 3475
-$Comp
-L power:GND #PWR?
-U 1 1 5E35317C
-P 2750 3625
-F 0 "#PWR?" H 2750 3375 50  0001 C CNN
-F 1 "GND" H 2755 3452 50  0000 C CNN
-F 2 "" H 2750 3625 50  0001 C CNN
-F 3 "" H 2750 3625 50  0001 C CNN
-	1    2750 3625
-	1    0    0    -1
-$EndComp
-Connection ~ 2750 3625
-$Comp
-L power:+12V #PWR?
-U 1 1 5E353890
-P 2475 3325
-F 0 "#PWR?" H 2475 3175 50  0001 C CNN
-F 1 "+12V" H 2490 3498 50  0000 C CNN
-F 2 "" H 2475 3325 50  0001 C CNN
-F 3 "" H 2475 3325 50  0001 C CNN
-	1    2475 3325
-	1    0    0    -1
-$EndComp
 $Comp
 L Connector_Generic:Conn_01x02 J?
@@
 	-1   0    0    1
 $EndComp
-Wire Wire Line
-	2275 3325 2475 3325
-Text Label 2750 3025 2    50   ~ 0
-GLV+
 Text Label 10375 1725 2    50   ~ 0
 GLV+
@@
 Text Label 10250 5750 1    50   ~ 0
 GLV+
-Text Label 10250 4400 3    50   ~ 0
-LED_GREEN+
 Wire Wire Line
 	10250 5750 10250 5300
@@
 Wire Wire Line
 	9550 4750 9550 4400
-$Comp
-L power:GND #PWR?
-U 1 1 5E38B565
-P 10600 4400
-F 0 "#PWR?" H 10600 4150 50  0001 C CNN
-F 1 "GND" H 10605 4227 50  0000 C CNN
-F 2 "" H 10600 4400 50  0001 C CNN
-F 3 "" H 10600 4400 50  0001 C CNN
-	1    10600 4400
-	1    0    0    -1
-$EndComp
 Wire Wire Line
 	9550 4400 10250 4400
-$Comp
-L Device:R R?
-U 1 1 5E38F5CE
-P 10250 5100
-F 0 "R?" H 10320 5146 50  0000 L CNN
-F 1 "R" H 10320 5055 50  0000 L CNN
-F 2 "" V 10180 5100 50  0001 C CNN
-F 3 "~" H 10250 5100 50  0001 C CNN
-	1    10250 5100
-	1    0    0    -1
-$EndComp
 Wire Wire Line
 	10250 5250 10250 5300
 Connection ~ 10250 5300
-Wire Wire Line
-	10250 4950 10250 4400
-Connection ~ 10250 4400
-Wire Wire Line
-	10250 4400 10600 4400
 $Comp
 L Device:R R?
@@
 Wire Wire Line
 	9075 1075 9075 650
+Text Notes 8500 5950 0    50   ~ 0
+Please check this, something seems wrong\n
+Text Notes 9650 6100 0    50   ~ 0
+Spice sim?\n
+Text Notes 3350 3250 0    50   ~ 0
+name your nets better plz
+Text Notes 1900 4150 0    50   ~ 0
+Why this opto? weird weird choice\n
+Text Notes 7400 3800 0    50   ~ 0
+Better connector; Figure out how will interface with HV int board, or consider HV connector board\n
+Text Notes 5750 5700 0    50   ~ 0
+Technically LED can run off just 10V, VS=10-30V
+Text Notes 5900 5900 0    50   ~ 0
+Boost is not necessary, unless you want it\n
+Text Label 9650 4400 0    50   ~ 0
+LED_GREEN+
+$Comp
+L Device:R_US R?
+U 1 1 5E3321DD
+P 10400 4400
+F 0 "R?" V 10195 4400 50  0000 C CNN
+F 1 "R_US" V 10286 4400 50  0000 C CNN
+F 2 "" V 10440 4390 50  0001 C CNN
+F 3 "~" H 10400 4400 50  0001 C CNN
+	1    10400 4400
+	0    1    1    0
+$EndComp
+$Comp
+L power:GND #PWR?
+U 1 1 5E333832
+P 10550 4550
+F 0 "#PWR?" H 10550 4300 50  0001 C CNN
+F 1 "GND" H 10555 4377 50  0000 C CNN
+F 2 "" H 10550 4550 50  0001 C CNN
+F 3 "" H 10550 4550 50  0001 C CNN
+	1    10550 4550
+	1    0    0    -1
+$EndComp
+Wire Wire Line
+	10550 4400 10550 4550
+$Comp
+L Isolator:LTV-817S U?
+U 1 1 5E3364C4
+P 1850 3150
+F 0 "U?" H 1850 3475 50  0000 C CNN
+F 1 "LTV-817S" H 1850 3384 50  0000 C CNN
+F 2 "Package_DIP:SMDIP-4_W9.53mm" H 1850 2850 50  0001 C CNN
+F 3 "http://www.us.liteon.com/downloads/LTV-817-827-847.PDF" H 1500 3450 50  0001 C CNN
+	1    1850 3150
+	1    0    0    -1
+$EndComp
+$Comp
+L power:+12VA #PWR?
+U 1 1 5E33E1BD
+P 1550 3050
+F 0 "#PWR?" H 1550 2900 50  0001 C CNN
+F 1 "+12VA" H 1565 3223 50  0000 C CNN
+F 2 "" H 1550 3050 50  0001 C CNN
+F 3 "" H 1550 3050 50  0001 C CNN
+	1    1550 3050
+	1    0    0    -1
+$EndComp
+$Comp
+L power:GNDA #PWR?
+U 1 1 5E33F030
+P 1550 3250
+F 0 "#PWR?" H 1550 3000 50  0001 C CNN
+F 1 "GNDA" H 1555 3077 50  0000 C CNN
+F 2 "" H 1550 3250 50  0001 C CNN
+F 3 "" H 1550 3250 50  0001 C CNN
+	1    1550 3250
+	1    0    0    -1
+$EndComp
+$Comp
+L Device:R_US R?
+U 1 1 5E33F945
+P 2150 3400
+F 0 "R?" H 2218 3446 50  0000 L CNN
+F 1 "10k" H 2218 3355 50  0000 L CNN
+F 2 "" V 2190 3390 50  0001 C CNN
+F 3 "~" H 2150 3400 50  0001 C CNN
+	1    2150 3400
+	1    0    0    -1
+$EndComp
+$Comp
+L power:+12V #PWR?
+U 1 1 5E3405B3
+P 2250 3250
+F 0 "#PWR?" H 2250 3100 50  0001 C CNN
+F 1 "+12V" V 2265 3378 50  0000 L CNN
+F 2 "" H 2250 3250 50  0001 C CNN
+F 3 "" H 2250 3250 50  0001 C CNN
+	1    2250 3250
+	0    1    1    0
+$EndComp
+Wire Wire Line
+	2250 3200 2250 3250
+Wire Wire Line
+	2150 3250 2250 3250
+Connection ~ 2150 3250
+Connection ~ 2250 3250
+$Comp
+L power:GND #PWR?
+U 1 1 5E3445CE
+P 2150 3550
+F 0 "#PWR?" H 2150 3300 50  0001 C CNN
+F 1 "GND" H 2155 3377 50  0000 C CNN
+F 2 "" H 2150 3550 50  0001 C CNN
+F 3 "" H 2150 3550 50  0001 C CNN
+	1    2150 3550
+	1    0    0    -1
+$EndComp
+Text Label 2150 3050 0    50   ~ 0
+GLV+
 $EndSCHEMATC

Commit message: fix the fixes
Parts:
- C1: value 0.1uF -> 2u
- R1: value 28.7k -> 100k
- R2: value 7.19M -> 235k
Changed lines of the file:
@@
 EESchema Schematic File Version 4
-LIBS:TSAL-cache
 EELAYER 30 0
 EELAYER END
@@
 P 6425 1925
 F 0 "R1" H 6495 1971 50  0000 L CNN
-F 1 "28.7k" H 6495 1880 50  0000 L CNN
+F 1 "100k" H 6495 1880 50  0000 L CNN
 F 2 "" V 6355 1925 50  0001 C CNN
 F 3 "~" H 6425 1925 50  0001 C CNN
@@
 P 6425 2475
 F 0 "R2" H 6495 2521 50  0000 L CNN
-F 1 "7.19M" H 6495 2430 50  0000 L CNN
+F 1 "235k" H 6495 2430 50  0000 L CNN
 F 2 "" V 6355 2475 50  0001 C CNN
 F 3 "~" H 6425 2475 50  0001 C CNN
@@
 P 6425 2925
 F 0 "C1" H 6310 2879 50  0000 R CNN
-F 1 "0.1uF" H 6310 2970 50  0000 R CNN
+F 1 "2u" H 6310 2970 50  0000 R CNN
 F 2 "" H 6463 2775 50  0001 C CNN
 F 3 "~" H 6425 2925 50  0001 C CNN
@@
 	-1   0    0    1
 $EndComp
-Text Label 10300 3550 0    50   ~ 0
-LED_GREEN+
 Wire Wire Line
 	10100 2700 10200 2700
@@
 Text Label 2150 3050 0    50   ~ 0
 GLV+
+Text Label 10300 3550 0    50   ~ 0
+LED_GREEN+
 $EndSCHEMATC

Commit message: schem ready for review
Parts:
- removed J4, J5, J?: Conn_01x02, symbol Connector_Generic:Conn_01x02
- removed Q?: BSS84, Package_TO_SOT_SMD:SOT-23, symbol Transistor_FET:BSS84
- removed R?: R_US, symbol Device:R_US
- added J6: Conn_02x03_Counter_Clockwise, Connector_TE-Connectivity:TE_MATE-N-LOK_1-770875-x_2x03_P4.14mm_Vertical, symbol Connector_Generic:Conn_02x03_Counter_Clockwise
- added Q2: FDD8447L, Package_TO_SOT_SMD:TO-252-2, symbol Transistor_FET:2N7000
- added R8: 1k, symbol Device:R
- R6: renamed from R?; value R -> 10k
- gave numbers to parts that had none: 5
Connections:
- net +12V: now also Q2.2 (G)
- net GLV+: now also J3.1 (Pin_1), J6.1 (Pin_1), R8.1
- net GND: now also R6.2, J6.2 (Pin_2), J6.3 (Pin_3), J6.4 (Pin_4), Q2.1 (S); no longer J3.1 (Pin_1), J3.2 (Pin_2)
- net LED_GREEN+: now also J3.2 (Pin_2), J6.5 (Pin_5)
- net LED_RED+: now also J6.6 (Pin_6)
- net CAP renamed THR
- new net: Q2.3 (D), R8.2
Other:
- note added: "Green LED Jumper\n"
- note removed: "Better connector; Figure out how will interface with HV int board, or consider HV connector board\n"
- note removed: "Please check this, something seems wrong\n"
- note removed: "Spice sim?\n"
- note removed: "Why this opto? weird weird choice\n"
- note removed: "name your nets better plz"
- moved on the sheet: C1, J3, Q1, R1, R2, R6, R7, U2, U3

Commit message: Ready for Review
Parts:
- added C1: 1u, Capacitor_SMD:C_0603_1608Metric_Pad1.05x0.95mm_HandSolder, symbol Device:C
- C2: renamed from C1; value 2u -> 1u; footprint (none) -> Capacitor_SMD:C_0603_1608Metric_Pad1.05x0.95mm_HandSolder
- J1, J2: footprint (none) -> Connector_TE-Connectivity:TE_MATE-N-LOK_1-770866-x_1x02_P4.14mm_Vertical
- J3: value Conn_01x02 -> Green_LED_Jp; footprint (none) -> Connector_TE-Connectivity:TE_MATE-N-LOK_1-770866-x_1x02_P4.14mm_Vertical
- R1: renamed from R3; footprint (none) -> Resistor_SMD:R_0603_1608Metric_Pad1.05x0.95mm_HandSolder
- R2: renamed from R4; footprint (none) -> Resistor_SMD:R_0603_1608Metric_Pad1.05x0.95mm_HandSolder
- R3: renamed from R5; footprint (none) -> Resistor_SMD:R_0603_1608Metric_Pad1.05x0.95mm_HandSolder
- R4: renamed from R1; footprint (none) -> Resistor_SMD:R_0603_1608Metric_Pad1.05x0.95mm_HandSolder
- R5: renamed from R2; footprint (none) -> Resistor_SMD:R_0603_1608Metric_Pad1.05x0.95mm_HandSolder
- R6: renamed from R7; footprint (none) -> Resistor_SMD:R_0603_1608Metric_Pad1.05x0.95mm_HandSolder
- R7: renamed from R6; footprint (none) -> Resistor_SMD:R_0603_1608Metric_Pad1.05x0.95mm_HandSolder
- R8: footprint (none) -> Resistor_SMD:R_0603_1608Metric_Pad1.05x0.95mm_HandSolder
- U3: renamed from U2; footprint (none) -> Package_SO:SOIC-8_3.9x4.9mm_P1.27mm
- U4: renamed from U3; footprint (none) -> aero_footprint:LDB-_L
- renumbered J6 to J4, U4 to U1, U1 to U2
Connections:
- net +24V: now also J3.1 (Pin_1), R8.1
- net GLV+: now also J4.6 (Pin_6); no longer J3.1 (Pin_1), J4.1 (Pin_1), R8.1
- net GND: now also J4.1 (Pin_1), C1.2; no longer J4.4 (Pin_4)
- net LED_RED+: now also J4.4 (Pin_4); no longer J4.6 (Pin_6)
- net THR: now also C1.1
