File: TSAL_NEW/KiCad/TSAL/TSAL.sch (KiCad schematic (older format))
At the start: 39 parts, among them J1 HV INPUT, J2 HV GND, J3 Conn_01x03, J4 B4B-PH-K, J5 Conn_01x02, Q1 BSS84, Q2 BSS84, U1 LTV-817S, U2 LR8K4-G, U4 LM555

Commit message: Changed HVInput to Optoisolator and added HV sense pin
Parts:
- removed C1: C2012X7S2A105K125AB, Capacitor_SMD:C_0805_2012Metric, symbol Device:C
- removed R4: 20k, Resistor_SMD:R_0603_1608Metric_Pad1.05x0.95mm_HandSolder, symbol Device:R_US
- removed U2: LR8K4-G, Package_TO_SOT_SMD:TO-252-2, symbol Regulator_Linear:LR8K4-G
- added Q3: 2N7002, Package_TO_SOT_SMD:SOT-23, symbol Transistor_FET:2N7002
- added R4: 10k, Resistor_SMD:R_0603_1608Metric_Pad1.05x0.95mm_HandSolder, symbol Device:R
- J5: footprint Connector_JST:JST_PH_B2B-PH-K_1x02_P2.00mm_Vertical -> Connector_JST:JST_PH_B3B-PH-K_1x03_P2.00mm_Vertical; symbol Connector_Generic:Conn_01x02 -> Connector_Generic:Conn_01x03
- R1: value 549 -> 33k axial; footprint Resistor_SMD:R_1210_3225Metric_Pad1.42x2.65mm_HandSolder -> Resistor_THT:R_Axial_DIN0309_L9.0mm_D3.2mm_P12.70mm_Horizontal
- R3: value 180k -> 100
Connections:
- net labels added: HV_PRES_TRUE
- net labels removed: +12VA
- wire segments 73 -> 77
Other:
- note added: "HV_PRES Low when off\n+12V when on"
- note added: "Pulled Low When HV\nis Present"
- note removed: "Decap for LDO, see datasheet\n"
- moved on the sheet: D3, Q1, R13, R14, R15, R8, R9

Commit message: change resistor
Parts:
- R1: footprint Resistor_THT:R_Axial_DIN0309_L9.0mm_D3.2mm_P12.70mm_Horizontal -> Resistor_THT:R_Axial_DIN0309_L9.0mm_D3.2mm_P20.32mm_Horizontal
Changed lines of the file:
@@
 F 0 "R1" H 1418 2946 50  0000 L CNN
 F 1 "33k axial" V 1250 2775 50  0000 L CNN
-F 2 "Resistor_THT:R_Axial_DIN0309_L9.0mm_D3.2mm_P12.70mm_Horizontal" V 1390 2890 50  0001 C CNN
+F 2 "Resistor_THT:R_Axial_DIN0309_L9.0mm_D3.2mm_P20.32mm_Horizontal" V 1390 2890 50  0001 C CNN
 F 3 "~" H 1350 2900 50  0001 C CNN
 	1    1350 2900

Commit message: Updated PCB Layout
Parts:
- R1: footprint Resistor_THT:R_Axial_DIN0309_L9.0mm_D3.2mm_P20.32mm_Horizontal -> Resistor_THT:R_Axial_DIN0516_L15.5mm_D5.0mm_P25.40mm_Horizontal
- R4: value 10k -> 100
Changed lines of the file:
@@
 F 0 "R1" H 1418 2946 50  0000 L CNN
 F 1 "33k axial" V 1250 2775 50  0000 L CNN
-F 2 "Resistor_THT:R_Axial_DIN0309_L9.0mm_D3.2mm_P20.32mm_Horizontal" V 1390 2890 50  0001 C CNN
+F 2 "Resistor_THT:R_Axial_DIN0516_L15.5mm_D5.0mm_P25.40mm_Horizontal" V 1390 2890 50  0001 C CNN
 F 3 "~" H 1350 2900 50  0001 C CNN
 	1    1350 2900
@@
 P 6800 6150
 F 0 "R4" H 6870 6196 50  0000 L CNN
-F 1 "10k" H 6870 6105 50  0000 L CNN
+F 1 "100" H 6870 6105 50  0000 L CNN
 F 2 "Resistor_SMD:R_0603_1608Metric_Pad1.05x0.95mm_HandSolder" V 6730 6150 50  0001 C CNN
 F 3 "~" H 6800 6150 50  0001 C CNN

Commit message: Minor Layout Changes
Parts:
- removed D3: 1N4148WT, Diode_SMD:D_SOD-523, symbol Diode:1N4148WT
- removed R12: 10k, Resistor_SMD:R_0603_1608Metric_Pad1.05x0.95mm_HandSolder, symbol Device:R
- removed R13, R14: R, Resistor_SMD:R_0603_1608Metric_Pad1.05x0.95mm_HandSolder, symbol Device:R
- J3: value Conn_01x03 -> B3B-PH-K
- R1: value 33k axial -> ROX3SJ39K
Connections:
- wire segments 77 -> 71
Changed lines of the file:
@@
 P 1350 2900
 F 0 "R1" H 1418 2946 50  0000 L CNN
-F 1 "33k axial" V 1250 2775 50  0000 L CNN
+F 1 "ROX3SJ39K" V 1250 2775 50  0000 L CNN
 F 2 "Resistor_THT:R_Axial_DIN0516_L15.5mm_D5.0mm_P25.40mm_Horizontal" V 1390 2890 50  0001 C CNN
 F 3 "~" H 1350 2900 50  0001 C CNN
@@
 	1    0    0    -1
 $EndComp
-Text Label 5125 4100 0    50   ~ 0
+Text Label 5425 4100 0    50   ~ 0
 HV_PRES
 Wire Wire Line
@@
 NoConn ~ 6250 1950
 $Comp
-L Diode:1N4148WT D3
-U 1 1 5E368EB7
-P 5850 4100
-F 0 "D3" H 5850 3883 50  0000 C CNN
-F 1 "1N4148WT" H 5850 3974 50  0000 C CNN
-F 2 "Diode_SMD:D_SOD-523" H 5850 3925 50  0001 C CNN
-F 3 "https://www.diodes.com/assets/Datasheets/ds30396.pdf" H 5850 4100 50  0001 C CNN
-	1    5850 4100
-	-1   0    0    1
-$EndComp
-Wire Wire Line
-	5125 4100 5700 4100
-Wire Wire Line
-	6000 4100 6100 4100
-$Comp
 L Transistor_FET:BSS84 Q1
 U 1 1 5E373EFD
@@
 P 9175 3850
 F 0 "J3" H 9093 3525 50  0000 C CNN
-F 1 "Conn_01x03" H 9093 3616 50  0000 C CNN
+F 1 "B3B-PH-K" H 9093 3616 50  0000 C CNN
 F 2 "Connector_PinHeader_2.54mm:PinHeader_1x03_P2.54mm_Vertical" H 9175 3850 50  0001 C CNN
 F 3 "~" H 9175 3850 50  0001 C CNN
@@
 $EndComp
 $Comp
-L Device:R R12
-U 1 1 5E3F1C34
-P 9450 5875
-F 0 "R12" V 9243 5875 50  0000 C CNN
-F 1 "10k" V 9334 5875 50  0000 C CNN
-F 2 "Resistor_SMD:R_0603_1608Metric_Pad1.05x0.95mm_HandSolder" V 9380 5875 50  0001 C CNN
-F 3 "~" H 9450 5875 50  0001 C CNN
-	1    9450 5875
-	0    1    1    0
-$EndComp
-$Comp
-L power:GND #PWR0103
-U 1 1 5E3F3BC4
-P 9725 5875
-F 0 "#PWR0103" H 9725 5625 50  0001 C CNN
-F 1 "GND" H 9730 5702 50  0000 C CNN
-F 2 "" H 9725 5875 50  0001 C CNN
-F 3 "" H 9725 5875 50  0001 C CNN
-	1    9725 5875
-	1    0    0    -1
-$EndComp
-Wire Wire Line
-	9725 5875 9600 5875
-Wire Wire Line
-	9300 5875 9250 5875
-$Comp
 L Connector_Generic:Conn_01x03 J5
 U 1 1 5E3FC548
@@
 Wire Wire Line
 	9250 6200 9500 6200
-Connection ~ 9250 5875
 Wire Wire Line
 	9250 5875 9225 5875
@@
 Wire Wire Line
 	8825 5875 8775 5875
-$Comp
-L Device:R R13
-U 1 1 5E41840C
-P 8525 5600
-F 0 "R13" H 8595 5646 50  0000 L CNN
-F 1 "R" H 8595 5555 50  0000 L CNN
-F 2 "Resistor_SMD:R_0603_1608Metric_Pad1.05x0.95mm_HandSolder" V 8455 5600 50  0001 C CNN
-F 3 "~" H 8525 5600 50  0001 C CNN
-	1    8525 5600
-	1    0    0    -1
-$EndComp
-$Comp
-L Device:R R14
-U 1 1 5E418CB6
-P 8525 6100
-F 0 "R14" H 8595 6146 50  0000 L CNN
-F 1 "R" H 8595 6055 50  0000 L CNN
-F 2 "Resistor_SMD:R_0603_1608Metric_Pad1.05x0.95mm_HandSolder" V 8455 6100 50  0001 C CNN
-F 3 "~" H 8525 6100 50  0001 C CNN
-	1    8525 6100
-	1    0    0    -1
-$EndComp
-$Comp
-L power:+12V #PWR0104
-U 1 1 5E419279
-P 8525 5450
-F 0 "#PWR0104" H 8525 5300 50  0001 C CNN
-F 1 "+12V" H 8540 5623 50  0000 C CNN
-F 2 "" H 8525 5450 50  0001 C CNN
-F 3 "" H 8525 5450 50  0001 C CNN
-	1    8525 5450
-	1    0    0    -1
-$EndComp
-$Comp
-L power:GND #PWR0106
-U 1 1 5E41982E
-P 8525 6250
-F 0 "#PWR0106" H 8525 6000 50  0001 C CNN
-F 1 "GND" H 8530 6077 50  0000 C CNN
-F 2 "" H 8525 6250 50  0001 C CNN
-F 3 "" H 8525 6250 50  0001 C CNN
-	1    8525 6250
-	1    0    0    -1
-$EndComp
-Wire Wire Line
-	8525 5750 8525 5875
-Wire Wire Line
-	8525 5875 8525 5950
-Connection ~ 8525 5875
 $Comp
 L Device:R R16
@@
 Wire Wire Line
 	8775 6300 8775 5875
-Connection ~ 8775 5875
-Wire Wire Line
-	8775 5875 8525 5875
 $Comp
 L Transistor_FET:2N7002 Q3
@@
 Text Notes 5275 5975 0    50   ~ 0
 HV_PRES Low when off\n+12V when on
+Wire Wire Line
+	5425 4100 6100 4100
 $EndSCHEMATC
