File: TSAL_NEW/KiCad/TSAL/TSAL.kicad_pcb (KiCad board)
At the start: 2 copper layers, 74.8 x 40.6 mm, 34 parts, among them J1 HV INPUT, J2 HV GND, J3 B3B-PH-K, J4 B4B-PH-K, J5 Conn_01x02, Q1 BSS84, Q2 BSS84, Q3 2N7002, U1 LTV-817S, U4 LM555

Commit message: init review
Parts:
- added REF**: JUMPER_BLUE, AERO_FOOT:JUMPER_BLUE, F.Cu at (156.8, 96.6)
- F1: footprint Fuse:Fuse_1812_4532Metric_Pad1.30x3.40mm_HandSolder -> AERO_FOOT:Fuse_1812_4532Metric_Pad1.30x3.40mm_HandSolder
- J1, J2: footprint AERO_FOOT:TE_MATE-N-LOK_1-770866-x_1x02_P4.14mm_Vertical -> AERO_FOOT:TE_MATE-N-LOK_1-770866-x_1x02_P4.14mm_Vertical_ASM
Changed lines of the file:
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@@
     (tracks 153)
     (zones 0)
-    (modules 34)
+    (modules 35)
     (nets 25)
   )
@@
   )
   (setup
-    (last_trace_width 0.65)
+    (last_trace_width 0.25)
     (user_trace_width 0.24)
     (user_trace_width 0.36)
@@
     (pad_to_mask_clearance 0.051)
     (solder_mask_min_width 0.25)
-    (aux_axis_origin 0 0)
+    (aux_axis_origin 106.68 127)
+    (grid_origin 106.68 127)
     (visible_elements 7FFFFFFF)
     (pcbplotparams
@@
     (add_net GND)
     (add_net "Net-(D1-Pad2)")
-    (add_net "Net-(J3-Pad1)")
     (add_net "Net-(J5-Pad2)")
     (add_net "Net-(Q1-Pad1)")
@@
     (add_net "Net-(Q3-Pad2)")
     (add_net "Net-(R1-Pad2)")
-    (add_net "Net-(U4-Pad5)")
   )
   (net_class HV ""
@@
     (add_net GNDA)
   )
-  (module AERO_FOOT:TE_MATE-N-LOK_1-770866-x_1x02_P4.14mm_Vertical (layer F.Cu)
+  (module AERO_FOOT:Fuse_1812_4532Metric_Pad1.30x3.40mm_HandSolder (layer F.Cu)
+    (at 170.688 90 180)
+    (descr "Fuse SMD 1812 (4532 Metric), square (rectangular) end terminal, IPC_7351 nominal with elongated pad for handsoldering. (Body size source: https://www.nikhef.nl/pub/departments/mt/projects/detectorR_D/dtddice/ERJ2G.pdf), generated with kicad-footprint-generator")
+    (tags "resistor handsolder")
+    (attr smd)
+    (fp_text reference F1 (at 0.312 2.624) (layer F.SilkS)
+      (effects (font (size 1 1) (thickness 0.15)))
+    )
+    (fp_text value 1812L075/24 (at 0 2.65) (layer F.Fab)
+      (effects (font (size 1 1) (thickness 0.15)))
+    )
+    (fp_text user "Do not have copper under fuse on any layer" (at -0.2 -4.1) (layer Cmts.User)
+      (effects (font (size 1 1) (thickness 0.15)))
+    )
+    (fp_text user %R (at 0 0) (layer F.Fab)
+      (effects (font (size 1 1) (thickness 0.15)))
+    )
+    (fp_line (start 3.12 1.95) (end -3.12 1.95) (layer F.CrtYd) (width 0.05))
+    (fp_line (start 3.12 -1.95) (end 3.12 1.95) (layer F.CrtYd) (width 0.05))
+    (fp_line (start -3.12 -1.95) (end 3.12 -1.95) (layer F.CrtYd) (width 0.05))
+    (fp_line (start -3.12 1.95) (end -3.12 -1.95) (layer F.CrtYd) (width 0.05))
+    (fp_line (start -1.386252 1.71) (end 1.386252 1.71) (layer F.SilkS) (width 0.12))
+    (fp_line (start -1.386252 -1.71) (end 1.386252 -1.71) (layer F.SilkS) (width 0.12))
+    (fp_line (start 2.25 1.6) (end -2.25 1.6) (layer F.Fab) (width 0.1))
+    (fp_line (start 2.25 -1.6) (end 2.25 1.6) (layer F.Fab) (width 0.1))
+    (fp_line (start -2.25 -1.6) (end 2.25 -1.6) (layer F.Fab) (width 0.1))
+    (fp_line (start -2.25 1.6) (end -2.25 -1.6) (layer F.Fab) (width 0.1))
+    (pad 2 smd roundrect (at 2.225 0 180) (size 1.3 3.4) (layers F.Cu F.Paste F.Mask) (roundrect_rratio 0.192308)
+      (net 7 /GLV+))
+    (pad 1 smd roundrect (at -2.225 0 180) (size 1.3 3.4) (layers F.Cu F.Paste F.Mask) (roundrect_rratio 0.192308)
+      (net 12 "Net-(D1-Pad2)"))
+    (model ${AERO_3D}/1812L110-16DR--3DModel-STEP-56544.STEP
+      (at (xyz 0 0 0))
+      (scale (xyz 1 1 1))
+      (rotate (xyz -90 0 0))
+    )
+  )
+  (module AERO_FOOT:TE_MATE-N-LOK_1-770866-x_1x02_P4.14mm_Vertical_ASM (layer F.Cu)
     (at 119.761 120.904 270)
     (descr "Molex Mini-Universal MATE-N-LOK, old mpn/engineering number: 1-770866-x, 2 Pins per row (http://www.te.com/commerce/DocumentDelivery/DDEController?Action=srchrtrv&DocNm=82181_SOFTSHELL_HIGH_DENSITY&DocType=CS&DocLang=EN), generated with kicad-footprint-generator")
@@
       (net 4 GNDA))
     (pad "" np_thru_hole circle (at 0 8.58 270) (size 3.18 3.18) (drill 3.18) (layers *.Cu *.Mask))
-    (model ${AERO_3D}/c-1-770166-0-n-3d.stp
-      (offset (xyz 0.0254 -2.032 14.3002))
-      (scale (xyz 1 1 1))
-      (rotate (xyz 0 0 90))
-    )
-  )
-  (module AERO_FOOT:TE_MATE-N-LOK_1-770866-x_1x02_P4.14mm_Vertical (layer F.Cu)
+    (model ${AERO_3D}/2p-mate-n-lok-asm.STEP
+      (offset (xyz -27.813 2.8448 0))
+      (scale (xyz 1 1 1))
+      (rotate (xyz 90 0 -90))
+    )
+  )
+  (module AERO_FOOT:TE_MATE-N-LOK_1-770866-x_1x02_P4.14mm_Vertical_ASM (layer F.Cu)
     (at 120.34 93.98 270)
     (descr "Molex Mini-Universal MATE-N-LOK, old mpn/engineering number: 1-770866-x, 2 Pins per row (http://www.te.com/commerce/DocumentDelivery/DDEController?Action=srchrtrv&DocNm=82181_SOFTSHELL_HIGH_DENSITY&DocType=CS&DocLang=EN), generated with kicad-footprint-generator")
@@
       (net 3 /HV+))
     (pad "" np_thru_hole circle (at 0 8.58 270) (size 3.18 3.18) (drill 3.18) (layers *.Cu *.Mask))
-    (model ${AERO_3D}/c-1-770166-0-n-3d.stp
-      (offset (xyz 0.0254 -2.032 14.3002))
-      (scale (xyz 1 1 1))
-      (rotate (xyz 0 0 90))
+    (model ${AERO_3D}/2p-mate-n-lok-asm.STEP
+      (offset (xyz -27.813 2.8448 0))
+      (scale (xyz 1 1 1))
+      (rotate (xyz 90 0 -90))
+    )
+  )
+  (module AERO_FOOT:JUMPER_BLUE (layer F.Cu)
+    (at 156.7688 96.5708)
+    (descr "Through hole straight pin header, 1x03, 2.54mm pitch, single row")
+    (tags "Through hole pin header THT 1x03 2.54mm single row")
+    (fp_text reference REF** (at 0 -2.33) (layer F.SilkS) hide
+      (effects (font (size 1 1) (thickness 0.15)))
+    )
+    (fp_text value JUMPER_BLUE (at 0.1 4.8) (layer F.Fab)
+      (effects (font (size 1 1) (thickness 0.15)))
+    )
+    (fp_line (start -1.33 -1.33) (end 1.33 -1.33) (layer F.CrtYd) (width 0.12))
+    (fp_line (start 1.33 -1.33) (end 1.33 3.81) (layer F.CrtYd) (width 0.12))
+    (fp_line (start -1.33 -1.33) (end -1.33 3.81) (layer F.CrtYd) (width 0.12))
+    (fp_line (start -1.33 3.81) (end 1.33 3.81) (layer F.CrtYd) (width 0.12))
+    (model ${AERO_3D}/M7583-46_asm.STEP
+      (offset (xyz -1.0668 -1.2192 5.5372))
+      (scale (xyz 1 1 1))
+      (rotate (xyz -90 0 90))
     )
   )
@@
       (at (xyz 0 0 0))
       (scale (xyz 1 1 1))
-      (rotate (xyz 0 0 0))
-    )
-  )
-  (module Fuse:Fuse_1812_4532Metric_Pad1.30x3.40mm_HandSolder (layer F.Cu)
-    (at 170.688 90 180)
-    (descr "Fuse SMD 1812 (4532 Metric), square (rectangular) end terminal, IPC_7351 nominal with elongated pad for handsoldering. (Body size source: https://www.nikhef.nl/pub/departments/mt/projects/detectorR_D/dtddice/ERJ2G.pdf), generated with kicad-footprint-generator")
-    (tags "resistor handsolder")
-    (attr smd)
-    (fp_text reference F1 (at 0.312 2.624) (layer F.SilkS)
-      (effects (font (size 1 1) (thickness 0.15)))
-    )
-    (fp_text value 1812L075/24 (at 0 2.65) (layer F.Fab)
-      (effects (font (size 1 1) (thickness 0.15)))
-    )
-    (fp_text user %R (at 0 0) (layer F.Fab)
-      (effects (font (size 1 1) (thickness 0.15)))
-    )
-    (fp_line (start 3.12 1.95) (end -3.12 1.95) (layer F.CrtYd) (width 0.05))
-    (fp_line (start 3.12 -1.95) (end 3.12 1.95) (layer F.CrtYd) (width 0.05))
-    (fp_line (start -3.12 -1.95) (end 3.12 -1.95) (layer F.CrtYd) (width 0.05))
-    (fp_line (start -3.12 1.95) (end -3.12 -1.95) (layer F.CrtYd) (width 0.05))
-    (fp_line (start -1.386252 1.71) (end 1.386252 1.71) (layer F.SilkS) (width 0.12))
-    (fp_line (start -1.386252 -1.71) (end 1.386252 -1.71) (layer F.SilkS) (width 0.12))
-    (fp_line (start 2.25 1.6) (end -2.25 1.6) (layer F.Fab) (width 0.1))
-    (fp_line (start 2.25 -1.6) (end 2.25 1.6) (layer F.Fab) (width 0.1))
-    (fp_line (start -2.25 -1.6) (end 2.25 -1.6) (layer F.Fab) (width 0.1))
-    (fp_line (start -2.25 1.6) (end -2.25 -1.6) (layer F.Fab) (width 0.1))
-    (pad 2 smd roundrect (at 2.225 0 180) (size 1.3 3.4) (layers F.Cu F.Paste F.Mask) (roundrect_rratio 0.192308)
-      (net 7 /GLV+))
-    (pad 1 smd roundrect (at -2.225 0 180) (size 1.3 3.4) (layers F.Cu F.Paste F.Mask) (roundrect_rratio 0.192308)
-      (net 12 "Net-(D1-Pad2)"))
-    (model ${KISYS3DMOD}/Fuse.3dshapes/Fuse_1812_4532Metric.wrl
-      (at (xyz 0 0 0))
-      (scale (xyz 1 1 1))
