File: fault-latcher/KiCad/Formula_Hybrid/FH_fault-latch.kicad_pcb (KiCad board)
At the start: 2 copper layers, 35 parts, among them J1 Conn_02x03_Odd_Even, J2 Conn_01x14, K1 G5V-2, K2 G5V-2, K3 G5V-2, K4 G5V-2, Q1 2N7002, Q2 2N7002, Q3 2N7002, Q4 2N7002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

Commit message: PCB ready
Parts:
- removed SW3: SW_Push, Connector_JST:JST_PH_B2B-PH-K_1x02_P2.00mm_Vertical
- added G***: LOGO, aero_footprint:AERO_Logo_15x6mm, B.Cu at (110.5, 77.5)
- added TMS2: SW_Push, Connector_JST:JST_PH_B2B-PH-K_1x02_P2.00mm_Vertical, F.Cu at (124.9, 111.3)
- C1, C2, C3, C4, C5, C6, D1, D2, D3, D4, Q1, Q2, Q3, Q4, Q5, R1, R2, R3, R4, R5, Y1: moved to B.Cu
- moved Q4 73.2 mm to (111.8, 95.0)
- moved C4 60.1 mm to (146.8, 117.9), turned to 90 degrees
- moved R4 59.6 mm to (114.7, 123.0), turned to 180 degrees
- moved D4 59.6 mm to (111.6, 89.8)
- moved R1 58.1 mm to (114.7, 116.0), turned to 180 degrees
- moved U1 57.8 mm to (150.5, 124.0), turned to 90 degrees
- moved Q3 55.3 mm to (124.1, 104.9), turned to 270 degrees
- moved R5 53.9 mm to (111.8, 98.0)
- moved R3 53.6 mm to (114.6, 121.3), turned to 180 degrees
- moved D3 53.3 mm to (124.0, 89.8), turned to 180 degrees
- moved Q5 52.8 mm to (111.9, 103.5)
- moved R2 49.9 mm to (114.7, 118.6), turned to 180 degrees
- moved D2 46.9 mm to (136.5, 89.8), turned to 180 degrees
- moved C5 43.9 mm to (131.6, 117.3), turned to 270 degrees
- moved Y1 43.6 mm to (136.5, 118.3), turned to 90 degrees
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- renumbered SW1 to BMS, SW4 to IMD, SW2 to TMS1
Connections:
- net Net-(K1-Pad13) renamed /l1
- net Net-(K2-Pad13) renamed /l2
- net Net-(K3-Pad13) renamed /l3
- BMS pad 1: +12V -> GND
- C1 pad 2: +12V -> GND
- C2 pad 2: +12V -> GND
- C3 pad 2: +12V -> GND
- C4 pad 2: +12V -> GND
- C5 pad 2: +12V -> GND
- C6 pad 2: +12V -> GND
- D4 pad 2: +12V -> GND
- J1 pad 2: +12V -> +5V
- J1 pad 6: +12V -> GND
- J2 pad 14: Net-(J2-Pad14) -> GND
- J2 pad 2: /LOOP_OUT -> +12V
- J2 pad 3: +12V -> /CAN+
- J2 pad 4: Net-(J2-Pad4) -> /CAN-
- J2 pad 5: +12V -> /LOOP_OUT
- J2 pad 6: /CAN_H -> (no net)
- J2 pad 7: /CAN_H -> (no net)
- J2 pad 8: /CAN_L -> /CAN+
- J2 pad 9: /CAN_L -> /CAN-
- K1 pad 11: Net-(K1-Pad11) -> (no net)
- K1 pad 6: Net-(K1-Pad6) -> (no net)
- K2 pad 11: Net-(K2-Pad11) -> (no net)
- K2 pad 6: Net-(K2-Pad6) -> (no net)
- K3 pad 11: Net-(K3-Pad11) -> (no net)
- K3 pad 6: Net-(K3-Pad6) -> (no net)
- K4 pad 11: Net-(K4-Pad11) -> (no net)
- K4 pad 16: +12V -> GND
- K4 pad 4: /IMD_IND -> /IMD_FAULT
- K4 pad 6: Net-(K4-Pad6) -> (no net)
- Q1 pad 3: +12V -> GND
- Q2 pad 3: +12V -> GND
- Q3 pad 3: +12V -> GND
- Q4 pad 3: +12V -> GND
- Q5 pad 3: +12V -> GND
- TMS1 pad 1: +12V -> GND
- U1 pad 2: +12V -> GND
- U2 pad 10: Net-(U2-Pad10) -> (no net)
- U2 pad 11: Net-(U2-Pad11) -> (no net)
- U2 pad 12: Net-(U2-Pad12) -> (no net)
- U2 pad 14: Net-(U2-Pad14) -> (no net)
- U2 pad 19: Net-(U2-Pad19) -> (no net)
- U2 pad 21: Net-(U2-Pad21) -> GND
- U2 pad 22: Net-(U2-Pad22) -> (no net)
- U2 pad 23: Net-(U2-Pad23) -> (no net)
- U2 pad 24: Net-(U2-Pad24) -> (no net)
- U2 pad 25: Net-(U2-Pad25) -> (no net)
- U2 pad 26: Net-(U2-Pad26) -> (no net)
- U2 pad 27: Net-(U2-Pad27) -> (no net)
- U2 pad 28: Net-(U2-Pad28) -> (no net)
- U2 pad 29: Net-(U2-Pad29) -> /RESET
- U2 pad 3: Net-(U2-Pad21) -> GND
- U2 pad 30: Net-(U2-Pad30) -> (no net)
- U2 pad 31: Net-(U2-Pad31) -> (no net)
- U2 pad 5: Net-(U2-Pad21) -> GND
- U2 pad 7: Net-(U2-Pad7) -> (no net)
- U2 pad 8: Net-(U2-Pad8) -> (no net)
- U3 pad 10: Net-(U3-Pad10) -> (no net)
- U3 pad 11: Net-(U3-Pad11) -> (no net)
- U3 pad 12: Net-(U3-Pad12) -> (no net)
- U3 pad 17: Net-(U3-Pad17) -> (no net)
- U3 pad 3: Net-(U3-Pad3) -> (no net)
- U3 pad 4: Net-(U3-Pad4) -> (no net)
- U3 pad 5: Net-(U3-Pad5) -> (no net)
- U3 pad 6: Net-(U3-Pad6) -> (no net)
- U3 pad 9: +12V -> GND
- U4 pad 2: +12V -> GND
- U4 pad 5: Net-(U4-Pad5) -> (no net)
- U4 pad 6: /CAN_L -> /CAN-
- U4 pad 7: /CAN_H -> /CAN+
- U4 pad 8: Net-(U4-Pad8) -> (no net)
- Y1 pad 2: Net-(Y1-Pad2) -> GND
Routing:
- net +12V: track 0.00 -> 150.9 mm, vias 0 -> 1
- net +5V: track 0.00 -> 91.6 mm, vias 0 -> 5
- net /CAN+: track 0.00 -> 46.5 mm
- net /BMS_IND: track 0.00 -> 46.3 mm, vias 0 -> 1
- net /CAN-: track 0.00 -> 45.1 mm
- net /TMS1_IND: track 0.00 -> 42.5 mm, vias 0 -> 1
- net /IMD_IND: track 0.00 -> 41.3 mm, vias 0 -> 1
- net /LOOP_IN: track 0.00 -> 37.2 mm
- net /TMS2_IND: track 0.00 -> 32.3 mm, vias 0 -> 2
- net Net-(D4-Pad1): track 0.00 -> 31.9 mm
- net /IMD_FAULT: track 0.00 -> 29.3 mm
- net Net-(D1-Pad2): track 0.00 -> 28.4 mm
- net Net-(D3-Pad2): track 0.00 -> 28.3 mm
- net Net-(D2-Pad2): track 0.00 -> 28.2 mm
- net /TMS2_FAULT: track 0.00 -> 25.9 mm
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- added copper zone on B.Cu, net GND
- added copper zone on F.Cu, net GND
Other:
- board outline added: 49.5 x 61 mm
- net class POWER: trace_width 0.508 -> 1.2
- board text added: "Fault Latcher Rev1 C.Jemison Rev2 G.Spearing 20.0206"
