File: fault-latcher/KiCad/Formula_Hybrid/FH_fault-latch.kicad_pcb (KiCad board)
At the start: 2 copper layers, 49.5 x 61 mm, 36 parts, among them J1 Conn_02x03_Odd_Even, J2 Conn_01x14, K1 G5V-2, K2 G5V-2, K3 G5V-2, K4 G5V-2, Q1 2N7002, Q2 2N7002, Q3 2N7002, Q4 2N7002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

Commit message: minor FH Chnage look at FN
Parts:
- removed G***: LOGO, aero_footprint:AERO_Logo_15x6mm
- renumbered BMS to SW1, TMS1 to SW2, TMS2 to SW3, IMD to SW4
Connections:
- J2 pad 6: (no net) -> +12V
- J2 pad 7: (no net) -> GND
Routing:
- net +12V: track 150.9 -> 156.0 mm
