File: fault-latcher/KiCad/Formula_Hybrid/FH_fault-latch.sch (KiCad schematic (older format))
At the start: 10 parts

Commit message: Create PCB
Parts:
- added C1, C2, C3, C5, C6: 0.1u, Capacitor_SMD:C_0603_1608Metric_Pad1.05x0.95mm_HandSolder, symbol Device:C
- added C4: 10u, Capacitor_SMD:C_0603_1608Metric_Pad1.05x0.95mm_HandSolder, symbol Device:C
- added D1, D2, D3, D4: 1N4148, Diode_SMD:D_SOD-123, symbol Diode:1N4148
- added Q1, Q2, Q3, Q4, Q5: 2N7002, Package_TO_SOT_SMD:SOT-23, symbol Transistor_FET:2N7002
- added R1, R2, R3, R4: 10K, Resistor_SMD:R_0603_1608Metric_Pad1.05x0.95mm_HandSolder, symbol Device:R
- added R5: 1K, Resistor_SMD:R_0603_1608Metric_Pad1.05x0.95mm_HandSolder, symbol Device:R
- added SW1, SW2, SW3, SW4: SW_Push, Connector_JST:JST_PH_B2B-PH-K_1x02_P2.00mm_Vertical, symbol Switch:SW_Push
- added Y1: Resonator, Crystal:Resonator_SMD_muRata_CSTxExxV-3Pin_3.0x1.1mm_HandSoldering, symbol Device:Resonator
- J1: renamed from J?; footprint (none) -> Connector_PinSocket_2.54mm:PinSocket_2x03_P2.54mm_Vertical
- J2: renamed from J?; footprint (none) -> AERO-footprints:TE_1-776266-1_14pin_Horizontal
- gave numbers to parts that had none: 8
Connections:
- net CAN-H is gone; now on net CAN_H: J2.6 (Pin_6), J2.7 (Pin_7)
- net CAN-L is gone; now on net CAN_L: J2.8 (Pin_8), J2.9 (Pin_9)
- net GND is gone; now on net +12V: J1.6 (Pin_6), J2.5 (Pin_5)
- net +12V: now also K1.16, K2.16, K3.16, K4.16, U1.1 (IN), U1.2 (GND), U3.9 (VSS), U4.2 (VSS), C1.1, C1.2, C2.2, C3.2, C4.2, C5.2, C6.2, D1.1 (K), D2.1 (K), D3.1 (K), D4.2 (A), Q1.3 (D), Q2.3 (D), Q3.3 (D), Q4.3 (D), Q5.3 (D), R1.1, R2.1, R3.1, R4.1, R5.2, SW1.1, SW2.1, SW3.1, SW4.1
- net BMS_FAULT: now also K1.4
- net LOOP_IN: now also K1.9
- net LOOP_OUT: now also K4.13
- net MISO: now also U2.16 (PB4), U3.15 (SO)
- net MOSI: now also U2.15 (PB3), U3.14 (SI)
- net SCK: now also U2.17 (PB5), U3.13 (SCK)
- net TMS1_FAULT: now also K2.4
- net TMS2_FAULT: now also K3.4
- net TMS1_IND: now reaches U2.1 (PD3)
- net TMS1_IND: now also Q2.2 (S), R2.2
- net CS: now reaches U2.13 (PB1)
- net CS: now also U3.16 (~CS)
- net +5V: now reaches U2.18 (AVCC)
- net +5V: now also U1.3 (OUT), U2.4 (VCC), U2.6 (VCC), U3.18 (VDD), U4.3 (VDD), C2.1, C4.1, C5.1, C6.1
- net TMS2_IND: now reaches U2.2 (PD4)
- net TMS2_IND: now also Q3.2 (S), R3.2
- net at U2.20 (AREF): now also C3.1
- net BMS_IND: now reaches U2.32 (PD2)
- net BMS_IND: now also Q1.2 (S), R1.2
- net IMD_IND: now reaches U2.9 (PD5)
- net IMD_IND: now also K4.4, Q4.2 (S), R4.2
- net TX: now reaches U4.1 (TXD)
- net TX: now also U3.1 (TXCAN)
- net RX: now reaches U4.4 (RXD)
- net RX: now also U3.2 (RXCAN)
- net CAN_L: now reaches U4.6 (CANL)
- net CAN_H: now reaches U4.7 (CANH)
- net at U3.7 (OSC2): now also Y1.1
- net at U3.8 (OSC1): now also Y1.3
- net at K1.1: now also K1.8, D1.2 (A), Q1.1 (G), SW1.2
- net at K1.13: now also K2.9
- net at K2.1: now also K2.8, D2.2 (A), Q2.1 (G), SW2.2
- net at K2.13: now also K3.9
- net at K3.1: now also K3.8, D3.2 (A), Q3.1 (G), SW3.2
- net at K3.13: now also K4.9
- net at K4.1: now also K4.8, D4.1 (K), Q5.1 (G), SW4.2
- new net: Q4.1 (G), Q5.2 (S), R5.1
Other:
- moved on the sheet: J1, K1, K2, K3, K4, U1, U2, U3, U4

Commit message: PCB ready
Connections:
- net +12V: now also J2.2 (Pin_2); no longer C1.2, C2.2, C3.2, C4.2, C5.2, C6.2, D4.2 (A), J1.2 (Pin_2), J1.6 (Pin_6), J2.3 (Pin_3), J2.5 (Pin_5), K4.16, Q1.3 (D), Q2.3 (D), Q3.3 (D), Q4.3 (D), Q5.3 (D), SW1.1, SW2.1, SW3.1, U1.2 (GND), U3.9 (VSS), U4.2 (VSS)
- net +5V: now also J1.2 (Pin_2)
- net IMD_FAULT: now also K4.4
- net IMD_IND: no longer K4.4
- net LOOP_OUT: now also J2.5 (Pin_5); no longer J2.2 (Pin_2)
- net RESET: now also U2.29 (~RESET~/PC6)
- net GND: now reaches U2.21 (GND), U2.3 (GND), U2.5 (GND)
- net GND: now also C1.2, C2.2, C3.2, C4.2, C5.2, C6.2, D4.2 (A), J1.6 (Pin_6), J2.14 (Pin_14), K4.16, Q1.3 (D), Q2.3 (D), Q3.3 (D), Q4.3 (D), Q5.3 (D), SW1.1, SW2.1, SW3.1, U1.2 (GND), U3.9 (VSS), U4.2 (VSS), Y1.2
- net l1: now reaches K1.13, K2.9
- net l2: now reaches K2.13, K3.9
- net l3: now reaches K3.13, K4.9
- net CAN-: now reaches J2.4 (Pin_4)
- net CAN-: now also J2.9 (Pin_9), U4.6 (CANL)
- removed net CAN_H: J2.6 (Pin_6), J2.7 (Pin_7), U4.7 (CANH)
- removed net CAN_L: J2.8 (Pin_8), J2.9 (Pin_9), U4.6 (CANL)
- new net CAN+: J2.3 (Pin_3), J2.8 (Pin_8), U4.7 (CANH)
Changed lines of the file:
@@
 U 1 1 5E3AC359
 P 2250 5400
-F 0 "U2" H 2250 3811 50  0000 C CNN
-F 1 "ATmega328P-AU" H 2250 3720 50  0000 C CNN
+F 0 "U2" H 1625 3800 50  0000 C CNN
+F 1 "ATmega328P-AU" H 1650 3900 50  0000 C CNN
 F 2 "Package_QFP:TQFP-32_7x7mm_P0.8mm" H 2250 5400 50  0001 C CIN
 F 3 "http://ww1.microchip.com/downloads/en/DeviceDoc/ATmega328_P%20AVR%20MCU%20with%20picoPower%20Technology%20Data%20Sheet%2040001984A.pdf" H 2250 5400 50  0001 C CNN
@@
 Text Label 9450 4400 0    50   ~ 0
 LOOP_IN
-Text Label 9450 4900 0    50   ~ 0
-CAN_H
+Text Label 9450 4600 0    50   ~ 0
+CAN+
+Text Label 9450 4700 0    50   ~ 0
+CAN-
+Text Label 9450 5200 0    50   ~ 0
+CAN-
 Text Label 9450 5100 0    50   ~ 0
-CAN_L
-Text Label 9450 5200 0    50   ~ 0
-CAN_L
-Text Label 9450 5000 0    50   ~ 0
-CAN_H
-Text Label 9450 4500 0    50   ~ 0
+CAN+
+Text Label 9450 4800 0    50   ~ 0
 LOOP_OUT
 Text Label 9450 5300 0    50   ~ 0
@@
 L power:+12V #PWR0101
 U 1 1 5E3D3477
-P 9275 4600
-F 0 "#PWR0101" H 9275 4450 50  0001 C CNN
-F 1 "+12V" H 9290 4773 50  0000 C CNN
-F 2 "" H 9275 4600 50  0001 C CNN
-F 3 "" H 9275 4600 50  0001 C CNN
-	1    9275 4600
+P 9275 4500
+F 0 "#PWR0101" H 9275 4350 50  0001 C CNN
+F 1 "+12V" H 9290 4673 50  0000 C CNN
+F 2 "" H 9275 4500 50  0001 C CNN
+F 3 "" H 9275 4500 50  0001 C CNN
+	1    9275 4500
 	1    0    0    -1
 $EndComp
@@
 L power:GND #PWR0102
 U 1 1 5E3D3A82
-P 9275 4800
-F 0 "#PWR0102" H 9275 4550 50  0001 C CNN
-F 1 "GND" H 9280 4627 50  0000 C CNN
-F 2 "" H 9275 4800 50  0001 C CNN
-F 3 "" H 9275 4800 50  0001 C CNN
-	1    9275 4800
+P 9275 5700
+F 0 "#PWR0102" H 9275 5450 50  0001 C CNN
+F 1 "GND" H 9280 5527 50  0000 C CNN
+F 2 "" H 9275 5700 50  0001 C CNN
+F 3 "" H 9275 5700 50  0001 C CNN
+	1    9275 5700
 	1    0    0    -1
 $EndComp
@@
 	9450 4400 9950 4400
 Wire Wire Line
-	9450 4500 9950 4500
-Wire Wire Line
-	9450 4900 9950 4900
-Wire Wire Line
-	9450 5000 9950 5000
+	9450 4800 9950 4800
+Wire Wire Line
+	9450 4600 9950 4600
 Wire Wire Line
 	9450 5100 9950 5100
 Wire Wire Line
+	9450 4700 9950 4700
+Wire Wire Line
 	9450 5200 9950 5200
 Wire Wire Line
@@
 	9450 5600 9950 5600
 Wire Wire Line
-	9275 4600 9950 4600
-Wire Wire Line
-	9275 4800 9950 4800
+	9275 4500 9950 4500
+Wire Wire Line
+	9275 5700 9950 5700
 Text Label 2075 1275 2    50   ~ 0
 MOSI
@@
 Text Label 900  1375 0    50   ~ 0
 RESET
-$Comp
-L power:+12V #PWR0103
-U 1 1 5E3D8F61
-P 2075 1175
-F 0 "#PWR0103" H 2075 1025 50  0001 C CNN
-F 1 "+12V" H 2090 1348 50  0000 C CNN
-F 2 "" H 2075 1175 50  0001 C CNN
-F 3 "" H 2075 1175 50  0001 C CNN
-	1    2075 1175
-	1    0    0    -1
-$EndComp
 $Comp
 L power:GND #PWR0104
@@
 	5700 2950 6275 2950
 Connection ~ 5700 2950
-Wire Wire Line
-	7375 2950 8150 2950
 Connection ~ 7375 2950
 $Comp
@@
 	1    0    0    -1
 $EndComp
-$Comp
-L power:GND #PWR0117
-U 1 1 5E4FD88C
-P 1475 2600
-F 0 "#PWR0117" H 1475 2350 50  0001 C CNN
-F 1 "GND" H 1480 2427 50  0000 C CNN
-F 2 "" H 1475 2600 50  0001 C CNN
-F 3 "" H 1475 2600 50  0001 C CNN
-	1    1475 2600
-	1    0    0    -1
-$EndComp
-Wire Wire Line
-	2100 2600 1475 2600
-Connection ~ 1475 2600
-Wire Wire Line
-	900  2600 1475 2600
 Wire Wire Line
 	900  2200 900  2300
@@
 Wire Wire Line
 	7075 2950 7375 2950
-Wire Wire Line
-	8150 2400 8150 2950
-Connection ~ 8150 2400
-Connection ~ 8150 2950
 Text Label 3625 2175 2    50   ~ 0
 BMS_IND
@@
 	8550 1625 8075 1625
 Text Label 10875 1625 2    50   ~ 0
-IMD_IND
+IMD_FAULT
 Wire Wire Line
 	10875 1625 10550 1625
@@
 Wire Wire Line
 	9050 2025 9850 2025
-Wire Wire Line
-	8150 2950 8925 2950
 $Comp
 L Transistor_FET:2N7002 Q1
@@
 	8150 2200 8150 2025
 Text Label 7400 4725 2    50   ~ 0
-CAN_H
+CAN+
 Wire Wire Line
 	7400 4725 7050 4725
 Text Label 7375 4925 2    50   ~ 0
-CAN_L
+CAN-
 Wire Wire Line
 	7375 4925 7050 4925
+Text Label 5400 1225 2    50   ~ 0
+l1
+Text Label 7175 1225 2    50   ~ 0
+l2
+Text Label 9600 1225 2    50   ~ 0
+l3
+$Comp
+L power:+5V #PWR0103
+U 1 1 5E3F41A7
+P 2075 1175
+F 0 "#PWR0103" H 2075 1025 50  0001 C CNN
+F 1 "+5V" H 2090 1348 50  0000 C CNN
+F 2 "" H 2075 1175 50  0001 C CNN
+F 3 "" H 2075 1175 50  0001 C CNN
+	1    2075 1175
+	1    0    0    -1
+$EndComp
+Wire Wire Line
+	1475 2650 1475 2600
+Wire Wire Line
+	1475 2650 2100 2650
+Wire Wire Line
+	2100 2650 2100 2600
+Connection ~ 1475 2650
+Wire Wire Line
+	1475 2650 900  2650
+Wire Wire Line
+	900  2650 900  2600
+$Comp
+L power:GND #PWR0117
+U 1 1 5E4FD88C
+P 1475 2650
+F 0 "#PWR0117" H 1475 2400 50  0001 C CNN
+F 1 "GND" H 1480 2477 50  0000 C CNN
+F 2 "" H 1475 2650 50  0001 C CNN
+F 3 "" H 1475 2650 50  0001 C CNN
+	1    1475 2650
+	1    0    0    -1
+$EndComp
+Text Label 3200 5700 2    50   ~ 0
+RESET
+Wire Wire Line
+	3200 5700 2850 5700
+Wire Wire Line
+	7375 2950 8925 2950
+$Comp
+L power:GND #PWR0122
+U 1 1 5E4B4375
+P 4025 6150
+F 0 "#PWR0122" H 4025 5900 50  0001 C CNN
+F 1 "GND" H 4030 5977 50  0000 C CNN
+F 2 "" H 4025 6150 50  0001 C CNN
+F 3 "" H 4025 6150 50  0001 C CNN
+	1    4025 6150
+	1    0    0    -1
+$EndComp
+$Comp
+L power:GND #PWR0123
+U 1 1 5E4CD70F
+P 2250 6900
+F 0 "#PWR0123" H 2250 6650 50  0001 C CNN
+F 1 "GND" H 2250 6725 50  0000 C CNN
+F 2 "" H 2250 6900 50  0001 C CNN
+F 3 "" H 2250 6900 50  0001 C CNN
+	1    2250 6900
+	1    0    0    -1
+$EndComp
 $EndSCHEMATC

Commit message: minor FH Chnage look at FN
Connections:
- net +12V: now also J2.6 (Pin_6)
- net GND: now also J2.7 (Pin_7)
Changed lines of the file:
@@
 	1    0    0    -1
 $EndComp
+$Comp
+L power:+12V #PWR?
+U 1 1 5E4DAE11
+P 9300 4900
+F 0 "#PWR?" H 9300 4750 50  0001 C CNN
+F 1 "+12V" H 9315 5073 50  0000 C CNN
+F 2 "" H 9300 4900 50  0001 C CNN
+F 3 "" H 9300 4900 50  0001 C CNN
+	1    9300 4900
+	1    0    0    -1
+$EndComp
+Wire Wire Line
+	9300 4900 9950 4900
+$Comp
+L power:GND #PWR?
+U 1 1 5E4E15DD
+P 9300 5000
+F 0 "#PWR?" H 9300 4750 50  0001 C CNN
+F 1 "GND" H 9305 4827 50  0000 C CNN
+F 2 "" H 9300 5000 50  0001 C CNN
+F 3 "" H 9300 5000 50  0001 C CNN
+	1    9300 5000
+	1    0    0    -1
+$EndComp
+Wire Wire Line
+	9300 5000 9950 5000
 $EndSCHEMATC

Commit message: "update old library"
Parts:
- added R6: 10k, symbol Device:R
Connections:
- net +5V: now also R6.1
- net BMS_IND: now also Q1.3 (D); no longer Q1.2 (S)
- net GND: now also Q1.2 (S), Q2.2 (S), Q3.2 (S), Q4.2 (S), Q5.2 (S), U4.8 (Rs); no longer Q1.3 (D), Q2.3 (D), Q3.3 (D), Q4.3 (D), Q5.3 (D)
- net IMD_IND: now also Q4.3 (D); no longer Q4.2 (S)
- net TMS1_IND: now also Q2.3 (D); no longer Q2.2 (S)
- net TMS2_IND: now also Q3.3 (D); no longer Q3.2 (S)
- net at U3.17 (~RESET): now also R6.2
- net at Q4.1 (G), R5.1: now also Q5.3 (D); no longer Q5.2 (S)
Other:
- note added: "Fault Directions:\nBMS: Driven low when OK, floating during fault\nTMS: Driven low during when OK, floating during fault\nIMD: Driven high when OK, driven low during fault"
Changed lines of the file:
@@
 F 3 "https://www.fairchildsemi.com/datasheets/2N/2N7002.pdf" H 3725 2375 50  0001 L CNN
 	1    3725 2375
-	-1   0    0    1
+	-1   0    0    -1
 $EndComp
 $Comp
@@
 F 3 "https://www.fairchildsemi.com/datasheets/2N/2N7002.pdf" H 5500 2400 50  0001 L CNN
 	1    5500 2400
-	-1   0    0    1
+	-1   0    0    -1
 $EndComp
 $Comp
@@
 F 3 "https://www.fairchildsemi.com/datasheets/2N/2N7002.pdf" H 7175 2400 50  0001 L CNN
 	1    7175 2400
-	-1   0    0    1
+	-1   0    0    -1
 $EndComp
 $Comp
@@
 F 3 "https://www.fairchildsemi.com/datasheets/2N/2N7002.pdf" H 9025 2750 50  0001 L CNN
 	1    9025 2750
-	-1   0    0    1
+	-1   0    0    -1
 $EndComp
 Connection ~ 8925 2950
@@
 F 3 "https://www.fairchildsemi.com/datasheets/2N/2N7002.pdf" H 9650 2400 50  0001 L CNN
 	1    9650 2400
-	-1   0    0    1
+	-1   0    0    -1
 $EndComp
 Connection ~ 9850 2400
@@
 $EndComp
 $Comp
-L power:+12V #PWR?
+L power:+12V #PWR0124
 U 1 1 5E4DAE11
 P 9300 4900
-F 0 "#PWR?" H 9300 4750 50  0001 C CNN
+F 0 "#PWR0124" H 9300 4750 50  0001 C CNN
 F 1 "+12V" H 9315 5073 50  0000 C CNN
 F 2 "" H 9300 4900 50  0001 C CNN
@@
 	9300 4900 9950 4900
 $Comp
-L power:GND #PWR?
+L power:GND #PWR0125
 U 1 1 5E4E15DD
 P 9300 5000
-F 0 "#PWR?" H 9300 4750 50  0001 C CNN
+F 0 "#PWR0125" H 9300 4750 50  0001 C CNN
 F 1 "GND" H 9305 4827 50  0000 C CNN
 F 2 "" H 9300 5000 50  0001 C CNN
@@
 Wire Wire Line
 	9300 5000 9950 5000
+Wire Wire Line
+	6050 5025 6050 5225
+Wire Wire Line
+	6050 5225 6550 5225
+Connection ~ 6550 5225
+$Comp
+L Device:R R6
+U 1 1 5EA1FD37
+P 5775 5675
+F 0 "R6" H 5845 5721 50  0000 L CNN
+F 1 "10k" H 5845 5630 50  0000 L CNN
+F 2 "" V 5705 5675 50  0001 C CNN
+F 3 "~" H 5775 5675 50  0001 C CNN
+	1    5775 5675
+	1    0    0    -1
+$EndComp
+$Comp
+L power:+5V #PWR0126
+U 1 1 5EA204D9
+P 5775 5525
+F 0 "#PWR0126" H 5775 5375 50  0001 C CNN
+F 1 "+5V" H 5790 5698 50  0000 C CNN
+F 2 "" H 5775 5525 50  0001 C CNN
+F 3 "" H 5775 5525 50  0001 C CNN
+	1    5775 5525
+	1    0    0    -1
+$EndComp
+Wire Wire Line
+	5775 5825 5500 5825
+Text Notes 3300 3425 0    50   ~ 0
+Fault Directions:\nBMS: Driven low when OK, floating during fault\nTMS: Driven low during when OK, floating during fault\nIMD: Driven high when OK, driven low during fault
 $EndSCHEMATC
