File: LED_Indicator/led_indicator/led_indicator.kicad_pcb (KiCad board)
At the start: 2 copper layers, 7 parts

Commit message: PCB Design ready to ship
Parts:
- removed TP1, TP2, TP3, TP4: TestPoint, TestPoint:TestPoint_Pad_2.5x2.5mm
- added D4: LED_PAD, aero_footprint:LXML-PM01, F.Cu at (181.7, 102.2)
- added G: TestPoint, TestPoint:TestPoint_Pad_2.5x2.5mm, F.Cu at (185.5, 96.8)
- added G: TestPoint, TestPoint:TestPoint_Pad_2.5x2.5mm, F.Cu at (173.8, 97.0)
- added R: TestPoint, TestPoint:TestPoint_Pad_2.5x2.5mm, F.Cu at (186.5, 91.8)
- added R: TestPoint, TestPoint:TestPoint_Pad_2.5x2.5mm, F.Cu at (173.2, 90.2)
- D1, D2, D3: footprint aero_footprint:luxeon-pm01 -> aero_footprint:LXML-PM01
- moved D3 34.5 mm to (181.9, 95.8)
- moved D1 33.9 mm to (176.7, 95.8)
- moved D2 33.8 mm to (177.2, 102.2), turned to 180 degrees
Connections:
- D1 pad 2: Net-(D1-Pad2) -> /R_IN
- D1 pad 3: (no net) -> /THM
- D2 pad 2: Net-(D2-Pad2) -> /G_IN
- D2 pad 3: (no net) -> /THM
- D3 pad 1: Net-(D3-Pad1) -> /R_OUT
- D3 pad 3: (no net) -> /THM
Routing:
- net Net-(D2-Pad2): track 12.8 -> 0.00 mm
- net Net-(D1-Pad2): track 4.77 -> 0.00 mm
- net Net-(D3-Pad1): track 4.64 -> 0.00 mm
- net /R_IN: track 0.00 -> 4.01 mm
- net /G_IN: track 0.00 -> 3.94 mm
- net /R_OUT: track 0.00 -> 3.85 mm
- net /G_OUT: track 0.00 -> 3.68 mm
- net Net-(D2-Pad1): track 5.29 -> 2.77 mm
- net Net-(D1-Pad1): track 2.79 -> 3.46 mm
- net /THM: vias 0 -> 33
- net (no net): vias 31 -> 0
- added copper zone on B.Cu, net /THM
- added copper zone on F.Cu, net /THM
Other:
- board outline added: 17.9 x 12.5 mm
- board text added: "LED Board 20.0206"
