File: PedalBoard2020/pedal-board-2020/pedal-board-2020.kicad_pcb (KiCad board)
At the start: 2 copper layers, 30.5 x 61.7 mm, 17 parts, among them J1 Conn_02x03_Odd_Even, J2 Conn_01x23, U1 ATmega328P-AU, U2 MCP2515-xSO, U3 MCP2551-I-SN, U4 R-785.0-1.0, Y1 16MHz

Commit message: add extra sensor
Connections:
- J2 pad 13: (no net) -> /SENSOR_2
- J2 pad 6: (no net) -> /SENSOR_1
- U1 pad 1: (no net) -> /SENSOR_1
- U1 pad 2: (no net) -> /SENSOR_2
Routing:
- net /SENSOR_2: track 0.00 -> 19.6 mm, vias 0 -> 1
- net /SENSOR_1: track 0.00 -> 9.14 mm
- net /RESET: track 39.1 -> 42.4 mm
Changed lines of the file:
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@@
     (thickness 1.6)
     (drawings 6)
-    (tracks 236)
+    (tracks 253)
     (zones 0)
     (modules 17)
-    (nets 23)
+    (nets 25)
   )
   (page A4)
@@
   (net 21 /STEER)
   (net 22 /BRAKE0)
+  (net 23 /SENSOR_2)
+  (net 24 /SENSOR_1)
   (net_class Default "This is the default net class."
     (clearance 0.2)
@@
     (add_net /RXCAN)
     (add_net /SCK)
+    (add_net /SENSOR_1)
+    (add_net /SENSOR_2)
     (add_net /STEER)
     (add_net /TXCAN)
     (add_net GND)
     (add_net "Net-(C2-Pad1)")
-    (add_net "Net-(J2-Pad13)")
-    (add_net "Net-(J2-Pad6)")
     (add_net "Net-(R3-Pad2)")
-    (add_net "Net-(U1-Pad1)")
     (add_net "Net-(U1-Pad10)")
     (add_net "Net-(U1-Pad11)")
@@
     (add_net "Net-(U1-Pad14)")
     (add_net "Net-(U1-Pad19)")
-    (add_net "Net-(U1-Pad2)")
     (add_net "Net-(U1-Pad22)")
     (add_net "Net-(U1-Pad28)")
@@
     (pad 14 thru_hole circle (at 22 4 270) (size 3 3) (drill 1.75) (layers *.Cu *.Mask)
       (net 19 /CANL))
-    (pad 13 thru_hole circle (at 18 4 270) (size 3 3) (drill 1.75) (layers *.Cu *.Mask))
+    (pad 13 thru_hole circle (at 18 4 270) (size 3 3) (drill 1.75) (layers *.Cu *.Mask)
+      (net 23 /SENSOR_2))
     (pad 12 thru_hole circle (at 14 4 270) (size 3 3) (drill 1.75) (layers *.Cu *.Mask)
       (net 3 +5V))
@@
     (pad 7 thru_hole circle (at 24 0 270) (size 3 3) (drill 1.75) (layers *.Cu *.Mask)
       (net 18 /CANH))
-    (pad 6 thru_hole circle (at 20 0 270) (size 3 3) (drill 1.75) (layers *.Cu *.Mask))
+    (pad 6 thru_hole circle (at 20 0 270) (size 3 3) (drill 1.75) (layers *.Cu *.Mask)
+      (net 24 /SENSOR_1))
     (pad 5 thru_hole circle (at 16 0 270) (size 3 3) (drill 1.75) (layers *.Cu *.Mask)
       (net 9 /ACC0))
@@
     (pad 3 smd rect (at -4.25 -1.2 90) (size 1.6 0.55) (layers F.Cu F.Paste F.Mask)
       (net 1 GND))
-    (pad 2 smd rect (at -4.25 -2 90) (size 1.6 0.55) (layers F.Cu F.Paste F.Mask))
-    (pad 1 smd rect (at -4.25 -2.8 90) (size 1.6 0.55) (layers F.Cu F.Paste F.Mask))
+    (pad 2 smd rect (at -4.25 -2 90) (size 1.6 0.55) (layers F.Cu F.Paste F.Mask)
+      (net 23 /SENSOR_2))
+    (pad 1 smd rect (at -4.25 -2.8 90) (size 1.6 0.55) (layers F.Cu F.Paste F.Mask)
+      (net 24 /SENSOR_1))
     (model ${KISYS3DMOD}/Package_QFP.3dshapes/TQFP-32_7x7mm_P0.8mm.wrl
       (at (xyz 0 0 0))
@@
   (segment (start 102.856 65.532) (end 104.535 63.853) (width 0.36) (layer F.Cu) (net 1))
   (segment (start 101.713 58.166) (end 104.535 58.166) (width 0.36) (layer F.Cu) (net 1))
+  (segment (start 109.474 65.758) (end 109.474 66.283) (width 0.36) (layer F.Cu) (net 1))
+  (segment (start 109.474 65.758) (end 109.474 68.213) (width 0.36) (layer F.Cu) (net 1))
+  (segment (start 108.839 101.411) (end 108.839 102.386) (width 0.36) (layer F.Cu) (net 1))
+  (segment (start 110.109 103.656) (end 110.109 106.361) (width 0.36) (layer F.Cu) (net 1))
+  (segment (start 108.839 102.386) (end 110.109 103.656) (width 0.36) (layer F.Cu) (net 1))
   (segment (start 105.048 72.314) (end 105.048 73.474) (width 0.36) (layer F.Cu) (net 2))
   (segment (start 105.048 70.709) (end 105.048 72.314) (width 0.36) (layer F.Cu) (net 2))
-  (segment (start 109.474 65.758) (end 109.474 66.283) (width 0.36) (layer F.Cu) (net 1))
-  (segment (start 109.474 65.758) (end 109.474 68.213) (width 0.36) (layer F.Cu) (net 1))
   (segment (start 105.048 68.434) (end 105.048 73.474) (width 0.36) (layer F.Cu) (net 2))
   (segment (start 109.474 64.008) (end 105.048 68.434) (width 0.36) (layer F.Cu) (net 2))
@@
   (segment (start 100.506 78.232) (end 100.398 78.124) (width 0.36) (layer F.Cu) (net 5))
   (segment (start 102.108 78.232) (end 100.506 78.232) (width 0.36) (layer F.Cu) (net 5))
-  (segment (start 102.108 81.788) (end 102.108 78.232) (width 0.36) (layer B.Cu) (net 5))
+  (segment (start 107.632 78.232) (end 102.108 78.232) (width 0.36) (layer B.Cu) (net 5))
+  (segment (start 108.712 79.312) (end 107.632 78.232) (width 0.36) (layer B.Cu) (net 5))
   (segment (start 102.87 110.49) (end 108.712 104.648) (width 0.36) (layer B.Cu) (net 5))
-  (segment (start 108.712 88.646) (end 102.108 81.788) (width 0.36) (layer B.Cu) (net 5))
-  (segment (start 108.712 104.648) (end 108.712 88.646) (width 0.36) (layer B.Cu) (net 5))
+  (segment (start 108.712 104.648) (end 108.712 79.312) (width 0.36) (layer B.Cu) (net 5))
   (segment (start 110.744 76.41) (end 110.744 79.756) (width 0.36) (layer F.Cu) (net 6))
   (via (at 110.744 79.756) (size 0.8) (drill 0.4) (layers F.Cu B.Cu) (net 6))
@@
   (segment (start 101.375973 87.376) (end 103.43001 89.430037) (width 0.36) (layer F.Cu) (net 17))
   (segment (start 108.712 98.552) (end 110.109 99.949) (width 0.36) (layer F.Cu) (net 17))
-  (segment (start 108.839 101.411) (end 108.839 102.386) (width 0.36) (layer F.Cu) (net 1))
-  (segment (start 110.109 103.656) (end 110.109 106.361) (width 0.36) (layer F.Cu) (net 1))
-  (segment (start 108.839 102.386) (end 110.109 103.656) (width 0.36) (layer F.Cu) (net 1))
   (segment (start 96.012 96.326) (end 96.012 98.806) (width 0.36) (layer F.Cu) (net 18))
   (segment (start 98.919 101.713) (end 98.919 103.632) (width 0.36) (layer F.Cu) (net 18))
@@
   (segment (start 100.7 72.326) (end 100.712 72.314) (width 0.36) (layer F.Cu) (net 22))
   (segment (start 96.012 72.326) (end 100.7 72.326) (width 0.36) (layer F.Cu) (net 22))
+  (segment (start 96.794402 86.326) (end 98.1 85.020402) (width 0.36) (layer B.Cu) (net 23))
+  (segment (start 92.012 86.326) (end 96.794402 86.326) (width 0.36) (layer B.Cu) (net 23))
+  (segment (start 98.1 85.020402) (end 98.1 79.7) (width 0.36) (layer B.Cu) (net 23))
+  (segment (start 98.1 79.7) (end 98.9 78.9) (width 0.36) (layer B.Cu) (net 23))
+  (segment (start 98.9 78.9) (end 101.5 78.9) (width 0.36) (layer B.Cu) (net 23))
+  (via (at 102.5 79.35) (size 0.8) (drill 0.4) (layers F.Cu B.Cu) (net 23))
+  (segment (start 101.5 78.9) (end 101.95 79.35) (width 0.36) (layer B.Cu) (net 23))
+  (segment (start 101.95 79.35) (end 102.5 79.35) (width 0.36) (layer B.Cu) (net 23))
+  (segment (start 102.503001 80.669001) (end 102.648 80.814) (width 0.36) (layer F.Cu) (net 23))
+  (segment (start 102.648 80.814) (end 102.648 81.974) (width 0.36) (layer F.Cu) (net 23))
+  (segment (start 102.503001 79.918686) (end 102.503001 80.669001) (width 0.36) (layer F.Cu) (net 23))
+  (segment (start 102.5 79.915685) (end 102.503001 79.918686) (width 0.36) (layer F.Cu) (net 23))
+  (segment (start 102.5 79.35) (end 102.5 79.915685) (width 0.36) (layer F.Cu) (net 23))
+  (segment (start 96.012 88.326) (end 98.85 85.488) (width 0.36) (layer F.Cu) (net 24))
+  (segment (start 101.213 81.974) (end 101.848 81.974) (width 0.36) (layer F.Cu) (net 24))
+  (segment (start 98.85 84.337) (end 101.213 81.974) (width 0.36) (layer F.Cu) (net 24))
+  (segment (start 98.85 85.488) (end 98.85 84.337) (width 0.36) (layer F.Cu) (net 24))
   (zone (net 1) (net_name GND) (layer F.Cu) (hatch edge 0.508)
     (connect_pads (clearance 0.508))
