File: PedalBoard2020/pedal-board-2020/pedal-board-2020.kicad_pcb (KiCad board)
At the start: 2 copper layers, 30.5 x 61.7 mm, 17 parts, among them J1 Conn_02x03_Odd_Even, J2 Conn_01x23, U1 ATmega328P-AU, U2 MCP2515-xSO, U3 MCP2551-I-SN, U4 R-785.0-1.0, Y1 16MHz

Commit message: small updates
Parts:
- moved R4 0.51 mm to (98.5, 103.8), turned to 270 degrees
Connections:
- net /CANH renamed /CAN+
- net /CANL renamed /CAN-
Routing:
- net /CAN+: track 24.1 -> 24.9 mm

Commit message: Altium work on HV stuff
Parts:
- J2: footprint Connector_TE-Connectivity:TE_AMPSEAL_1-776087-x_3Rows_23_P0.4mm_Horizontal -> AERO-footprints:TE_1-776087-1

Commit message: Minor changes / updates
Routing:
- net GND: track 40.6 -> 43.1 mm, vias 2 -> 5
Changed lines of the file:
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@@
-(kicad_pcb (version 20171130) (host pcbnew "(5.1.4)-1")
+(kicad_pcb (version 20171130) (host pcbnew 5.1.5-52549c5~84~ubuntu18.04.1)
   (general
     (thickness 1.6)
     (drawings 6)
-    (tracks 258)
+    (tracks 263)
     (zones 0)
     (modules 17)
@@
   (segment (start 110.109 103.656) (end 110.109 106.361) (width 0.36) (layer F.Cu) (net 1))
   (segment (start 108.839 102.386) (end 110.109 103.656) (width 0.36) (layer F.Cu) (net 1))
+  (via (at 102.7684 98.4504) (size 0.8) (drill 0.4) (layers F.Cu B.Cu) (net 1))
+  (segment (start 102.362 98.8568) (end 102.362 100.838) (width 0.25) (layer F.Cu) (net 1))
+  (segment (start 102.7684 98.4504) (end 102.362 98.8568) (width 0.25) (layer F.Cu) (net 1))
+  (via (at 98.3996 99.568) (size 0.8) (drill 0.4) (layers F.Cu B.Cu) (net 1))
+  (via (at 104.521 88.392) (size 0.8) (drill 0.4) (layers F.Cu B.Cu) (net 1))
   (segment (start 105.048 72.314) (end 105.048 73.474) (width 0.36) (layer F.Cu) (net 2))
   (segment (start 105.048 70.709) (end 105.048 72.314) (width 0.36) (layer F.Cu) (net 2))
