File: PedalBoard2020/pedal-board-2020/pedal-board-2020.sch (KiCad schematic (older format))
At the start: 17 parts, among them J1 Conn_02x03_Odd_Even, J2 Conn_01x23, U1 ATmega328P-AU, U2 MCP2515-xSO, U3 MCP2551-I-SN, U4 R-785.0-1.0, Y1 16MHz

Commit message: add extra sensor
Connections:
- net labels added: SENSOR_1, SENSOR_2
- wire segments 109 -> 114
Changed lines of the file:
@@
 $EndComp
 Connection ~ 7950 3900
+Text Label 10300 3100 0    50   ~ 0
+SENSOR_1
+Wire Wire Line
+	10300 3100 10650 3100
+Text Label 10300 3775 0    50   ~ 0
+SENSOR_2
+Wire Wire Line
+	10300 3775 10650 3775
+Wire Wire Line
+	10650 3775 10650 3800
+Text Label 3750 5000 2    50   ~ 0
+SENSOR_1
+Wire Wire Line
+	3750 5000 3350 5000
+Text Label 3750 5100 2    50   ~ 0
+SENSOR_2
+Wire Wire Line
+	3750 5100 3350 5100
 $EndSCHEMATC
