File: PedalBoard2020/pedal-board-2020/pedal-board-2020.sch (KiCad schematic (older format))
At the start: 17 parts, among them J1 Conn_02x03_Odd_Even, J2 Conn_01x23, U1 ATmega328P-AU, U2 MCP2515-xSO, U3 MCP2551-I-SN, U4 R-785.0-1.0, Y1 16MHz

Commit message: small updates
Connections:
- net labels added: CAN+, CAN-
- net labels removed: CANH, CANL
Changed lines of the file:
@@
 $EndComp
 Text Label 8775 3400 2    50   ~ 0
-CANH
+CAN+
 Text Label 8775 3600 2    50   ~ 0
-CANL
+CAN-
 $Comp
 L Device:R R4
@@
 	5050 4200 5050 4600
 Text Label 10325 3200 0    50   ~ 0
-CANH
+CAN+
 Text Label 10350 3900 0    50   ~ 0
-CANL
+CAN-
 $Comp
 L power:+5V #PWR0118

Commit message: Altium work on HV stuff
Parts:
- U1: symbol MCU_Microchip_ATmega:ATmega328P-AU -> pedal-board-2020-rescue:ATmega328P-AU-MCU_Microchip_ATmega
Changed lines of the file:
@@
 EESchema Schematic File Version 4
+LIBS:pedal-board-2020-cache
 EELAYER 30 0
 EELAYER END
@@
 $EndDescr
 $Comp
-L MCU_Microchip_ATmega:ATmega328P-AU U1
+L pedal-board-2020-rescue:ATmega328P-AU-MCU_Microchip_ATmega U1
 U 1 1 5E386332
 P 2750 4200

Commit message: Minor changes / updates
Other:
- note added: "Front DAQ board\nG.Spearing\n20.0303"
- moved on the sheet: C5, C6, J1, J2, U4
