File: LV_Breakout/GLV_COMB.sch (KiCad schematic (older format))
At the start: 19 parts, among them Q1 CSD18563Q5A, U2 LM74700QDBVTQ1, U3 INA219AIDR, U4 INA219AIDR

Commit message: LVPDU schem and pcb
Parts:
- C10, C6, C8: footprint Capacitor_SMD:C_0603_1608Metric -> Capacitor_SMD:C_0603_1608Metric_Pad1.05x0.95mm_HandSolder
- C11, C9: footprint Resistor_SMD:R_0603_1608Metric -> Capacitor_SMD:C_0603_1608Metric_Pad1.05x0.95mm_HandSolder
- D1: footprint Diode_SMD:D_SMB_Handsoldering -> AERO_FOOT:DO-214AA
- R10, R4, R5, R9: footprint Resistor_SMD:R_0603_1608Metric -> Resistor_SMD:R_0805_2012Metric_Pad1.15x1.40mm_HandSolder
- R3, R8: footprint AERO-footprints:KRL6432E-M-R003-F-T1 -> Resistor_SMD:R_2512_6332Metric_Pad1.52x3.35mm_HandSolder
- R6, R7: footprint Resistor_SMD:R_2512_6332Metric -> Resistor_SMD:R_2512_6332Metric_Pad1.52x3.35mm_HandSolder
- U2: footprint Package_TO_SOT_SMD:SOT-23-6 -> Package_TO_SOT_SMD:SOT-23-6_Handsoldering
Changed lines of the file:
@@
 EESchema Schematic File Version 4
-LIBS:LV_Breakout-cache
 EELAYER 30 0
 EELAYER END
@@
 F 0 "U2" H 3900 4637 60  0000 C CNN
 F 1 "LM74700QDBVTQ1" H 3900 4531 60  0000 C CNN
-F 2 "Package_TO_SOT_SMD:SOT-23-6" H 3900 4490 60  0001 C CNN
+F 2 "Package_TO_SOT_SMD:SOT-23-6_Handsoldering" H 3900 4490 60  0001 C CNN
 F 3 "" H 3000 4250 60  0000 C CNN
 	1    3000 4250
@@
 Connection ~ 2350 3300
 $Comp
-L power:GND #PWR08
+L power:GND #PWR013
 U 1 1 5E550712
 P 3000 4350
-F 0 "#PWR08" H 3000 4100 50  0001 C CNN
+F 0 "#PWR013" H 3000 4100 50  0001 C CNN
 F 1 "GND" V 3005 4222 50  0000 R CNN
 F 2 "" H 3000 4350 50  0001 C CNN
@@
 F 0 "D1" V 2396 3071 50  0000 R CNN
 F 1 "SMBJ15CA" V 2305 3071 50  0000 R CNN
-F 2 "Diode_SMD:D_SMB_Handsoldering" H 2350 3150 50  0001 C CNN
+F 2 "AERO_FOOT:DO-214AA" H 2350 3150 50  0001 C CNN
 F 3 "https://www.littelfuse.com/~/media/electronics/datasheets/tvs_diodes/littelfuse_tvs_diode_smbj_datasheet.pdf.pdf" H 2350 3150 50  0001 C CNN
 	1    2350 3150
@@
 $EndComp
 $Comp
-L power:GND #PWR07
+L power:GND #PWR012
 U 1 1 5E55169F
 P 2350 3000
-F 0 "#PWR07" H 2350 2750 50  0001 C CNN
+F 0 "#PWR012" H 2350 2750 50  0001 C CNN
 F 1 "GND" H 2355 2827 50  0000 C CNN
 F 2 "" H 2350 3000 50  0001 C CNN
@@
 F 0 "C6" H 2865 3196 50  0000 L CNN
 F 1 "22nF" H 2865 3105 50  0000 L CNN
-F 2 "Capacitor_SMD:C_0603_1608Metric" H 2788 3000 50  0001 C CNN
+F 2 "Capacitor_SMD:C_0603_1608Metric_Pad1.05x0.95mm_HandSolder" H 2788 3000 50  0001 C CNN
 F 3 "~" H 2750 3150 50  0001 C CNN
 	1    2750 3150
@@
 F 0 "R8" H 6318 3900 50  0000 L CNN
 F 1 "KRL6432E-M-R003-F-T1" H 6318 3855 50  0001 L CNN
-F 2 "AERO-footprints:KRL6432E-M-R003-F-T1" V 6290 3890 50  0001 C CNN
+F 2 "Resistor_SMD:R_2512_6332Metric_Pad1.52x3.35mm_HandSolder" V 6290 3890 50  0001 C CNN
 F 3 "https://www.susumu.co.jp/common/pdf/n_catalog_partition19_en.pdf" H 6250 3900 50  0001 C CNN
 	1    6250 3900
@@
 F 0 "R9" V 7195 3750 50  0000 C CNN
 F 1 "10" V 7286 3750 50  0000 C CNN
-F 2 "Resistor_SMD:R_0603_1608Metric" V 7440 3740 50  0001 C CNN
+F 2 "Resistor_SMD:R_0805_2012Metric_Pad1.15x1.40mm_HandSolder" V 7440 3740 50  0001 C CNN
 F 3 "~" H 7400 3750 50  0001 C CNN
 	1    7400 3750
@@
 F 0 "R10" V 7195 4050 50  0000 C CNN
 F 1 "10" V 7286 4050 50  0000 C CNN
-F 2 "Resistor_SMD:R_0603_1608Metric" V 7440 4040 50  0001 C CNN
+F 2 "Resistor_SMD:R_0805_2012Metric_Pad1.15x1.40mm_HandSolder" V 7440 4040 50  0001 C CNN
 F 3 "~" H 7400 4050 50  0001 C CNN
 	1    7400 4050
@@
 F 0 "C10" H 7965 3946 50  0000 L CNN
 F 1 "1uF" H 7965 3855 50  0000 L CNN
-F 2 "Capacitor_SMD:C_0603_1608Metric" H 7888 3750 50  0001 C CNN
+F 2 "Capacitor_SMD:C_0603_1608Metric_Pad1.05x0.95mm_HandSolder" H 7888 3750 50  0001 C CNN
 F 3 "~" H 7850 3900 50  0001 C CNN
 	1    7850 3900
@@
 	7850 3750 7550 3750
 $Comp
-L power:+5V #PWR015
+L power:+5V #PWR020
 U 1 1 5E567AD4
 P 8750 3450
-F 0 "#PWR015" H 8750 3300 50  0001 C CNN
+F 0 "#PWR020" H 8750 3300 50  0001 C CNN
 F 1 "+5V" H 8765 3623 50  0000 C CNN
 F 2 "" H 8750 3450 50  0001 C CNN
@@
 $EndComp
 $Comp
-L power:GND #PWR016
+L power:GND #PWR021
 U 1 1 5E56862C
 P 8750 4250
-F 0 "#PWR016" H 8750 4000 50  0001 C CNN
+F 0 "#PWR021" H 8750 4000 50  0001 C CNN
 F 1 "GND" H 8755 4077 50  0000 C CNN
 F 2 "" H 8750 4250 50  0001 C CNN
@@
 $EndComp
 $Comp
-L power:GND #PWR018
+L power:GND #PWR023
 U 1 1 5E568A9C
 P 9100 4700
-F 0 "#PWR018" H 9100 4450 50  0001 C CNN
+F 0 "#PWR023" H 9100 4450 50  0001 C CNN
 F 1 "GND" H 9105 4527 50  0000 C CNN
 F 2 "" H 9100 4700 50  0001 C CNN
@@
 F 0 "C11" H 9215 4596 50  0000 L CNN
 F 1 "0.1uF" H 9215 4505 50  0000 L CNN
-F 2 "Resistor_SMD:R_0603_1608Metric" H 9138 4400 50  0001 C CNN
+F 2 "Capacitor_SMD:C_0603_1608Metric_Pad1.05x0.95mm_HandSolder" H 9138 4400 50  0001 C CNN
 F 3 "~" H 9100 4550 50  0001 C CNN
 	1    9100 4550
@@
 $EndComp
 $Comp
-L power:+5V #PWR017
+L power:+5V #PWR022
 U 1 1 5E569379
 P 9100 4400
-F 0 "#PWR017" H 9100 4250 50  0001 C CNN
+F 0 "#PWR022" H 9100 4250 50  0001 C CNN
 F 1 "+5V" H 9115 4573 50  0000 C CNN
 F 2 "" H 9100 4400 50  0001 C CNN
@@
 SCL
 $Comp
-L power:GND #PWR019
+L power:GND #PWR024
 U 1 1 5E569C73
 P 9450 4050
-F 0 "#PWR019" H 9450 3800 50  0001 C CNN
+F 0 "#PWR024" H 9450 3800 50  0001 C CNN
 F 1 "GND" V 9455 3922 50  0000 R CNN
 F 2 "" H 9450 4050 50  0001 C CNN
@@
 F 0 "R3" H 2368 2200 50  0000 L CNN
 F 1 "KRL6432E-M-R003-F-T1" H 2368 2155 50  0001 L CNN
-F 2 "AERO-footprints:KRL6432E-M-R003-F-T1" V 2340 2190 50  0001 C CNN
+F 2 "Resistor_SMD:R_2512_6332Metric_Pad1.52x3.35mm_HandSolder" V 2340 2190 50  0001 C CNN
 F 3 "https://www.susumu.co.jp/common/pdf/n_catalog_partition19_en.pdf" H 2300 2200 50  0001 C CNN
 	1    2300 2200
@@
 F 0 "R4" V 3245 2050 50  0000 C CNN
 F 1 "10" V 3336 2050 50  0000 C CNN
-F 2 "Resistor_SMD:R_0603_1608Metric" V 3490 2040 50  0001 C CNN
+F 2 "Resistor_SMD:R_0805_2012Metric_Pad1.15x1.40mm_HandSolder" V 3490 2040 50  0001 C CNN
 F 3 "~" H 3450 2050 50  0001 C CNN
 	1    3450 2050
@@
 F 0 "R5" V 3245 2350 50  0000 C CNN
 F 1 "10" V 3336 2350 50  0000 C CNN
-F 2 "Resistor_SMD:R_0603_1608Metric" V 3490 2340 50  0001 C CNN
+F 2 "Resistor_SMD:R_0805_2012Metric_Pad1.15x1.40mm_HandSolder" V 3490 2340 50  0001 C CNN
 F 3 "~" H 3450 2350 50  0001 C CNN
 	1    3450 2350
@@
 F 0 "C8" H 4015 2246 50  0000 L CNN
 F 1 "1uF" H 4015 2155 50  0000 L CNN
-F 2 "Capacitor_SMD:C_0603_1608Metric" H 3938 2050 50  0001 C CNN
+F 2 "Capacitor_SMD:C_0603_1608Metric_Pad1.05x0.95mm_HandSolder" H 3938 2050 50  0001 C CNN
 F 3 "~" H 3900 2200 50  0001 C CNN
 	1    3900 2200
@@
 	3900 2050 3600 2050
 $Comp
-L power:+5V #PWR09
+L power:+5V #PWR014
 U 1 1 5E5743E7
 P 4800 1750
-F 0 "#PWR09" H 4800 1600 50  0001 C CNN
+F 0 "#PWR014" H 4800 1600 50  0001 C CNN
 F 1 "+5V" H 4815 1923 50  0000 C CNN
 F 2 "" H 4800 1750 50  0001 C CNN
@@
 $EndComp
 $Comp
-L power:GND #PWR010
+L power:GND #PWR015
 U 1 1 5E5743ED
 P 4800 2550
-F 0 "#PWR010" H 4800 2300 50  0001 C CNN
+F 0 "#PWR015" H 4800 2300 50  0001 C CNN
 F 1 "GND" H 4805 2377 50  0000 C CNN
 F 2 "" H 4800 2550 50  0001 C CNN
@@
 $EndComp
 $Comp
-L power:GND #PWR012
+L power:GND #PWR017
 U 1 1 5E5743F3
 P 5150 3000
-F 0 "#PWR012" H 5150 2750 50  0001 C CNN
+F 0 "#PWR017" H 5150 2750 50  0001 C CNN
 F 1 "GND" H 5155 2827 50  0000 C CNN
 F 2 "" H 5150 3000 50  0001 C CNN
@@
 F 0 "C9" H 5265 2896 50  0000 L CNN
 F 1 "0.1uF" H 5265 2805 50  0000 L CNN
-F 2 "Resistor_SMD:R_0603_1608Metric" H 5188 2700 50  0001 C CNN
+F 2 "Capacitor_SMD:C_0603_1608Metric_Pad1.05x0.95mm_HandSolder" H 5188 2700 50  0001 C CNN
 F 3 "~" H 5150 2850 50  0001 C CNN
 	1    5150 2850
@@
 $EndComp
 $Comp
-L power:+5V #PWR011
+L power:+5V #PWR016
 U 1 1 5E5743FF
 P 5150 2700
-F 0 "#PWR011" H 5150 2550 50  0001 C CNN
+F 0 "#PWR016" H 5150 2550 50  0001 C CNN
 F 1 "+5V" H 5165 2873 50  0000 C CNN
 F 2 "" H 5150 2700 50  0001 C CNN
@@
 F 0 "R6" V 3595 3000 50  0000 C CNN
 F 1 "20" V 3686 3000 50  0000 C CNN
-F 2 "Resistor_SMD:R_2512_6332Metric" V 3840 2990 50  0001 C CNN
+F 2 "Resistor_SMD:R_2512_6332Metric_Pad1.52x3.35mm_HandSolder" V 3840 2990 50  0001 C CNN
 F 3 "~" H 3800 3000 50  0001 C CNN
 	1    3800 3000
@@
 $EndComp
 $Comp
-L power:GND #PWR014
+L power:GND #PWR019
 U 1 1 5E57A93E
 P 5500 2350
-F 0 "#PWR014" H 5500 2100 50  0001 C CNN
+F 0 "#PWR019" H 5500 2100 50  0001 C CNN
 F 1 "GND" V 5505 2222 50  0000 R CNN
 F 2 "" H 5500 2350 50  0001 C CNN
@@
 $EndComp
 $Comp
-L power:+5V #PWR013
+L power:+5V #PWR018
 U 1 1 5E57B003
 P 5200 2250
-F 0 "#PWR013" H 5200 2100 50  0001 C CNN
+F 0 "#PWR018" H 5200 2100 50  0001 C CNN
 F 1 "+5V" V 5215 2378 50  0000 L CNN
 F 2 "" H 5200 2250 50  0001 C CNN
@@
 F 0 "R7" V 3895 2850 50  0000 C CNN
 F 1 "20" V 3986 2850 50  0000 C CNN
-F 2 "Resistor_SMD:R_2512_6332Metric" V 4140 2840 50  0001 C CNN
+F 2 "Resistor_SMD:R_2512_6332Metric_Pad1.52x3.35mm_HandSolder" V 4140 2840 50  0001 C CNN
 F 3 "~" H 4100 2850 50  0001 C CNN
 	1    4100 2850
