File: LV_Breakout/_autosave-Port_Panel.sch (KiCad schematic (older format))
At the start: 24 parts, among them J1 DB9_Male_MountingHoles, J10 TE 776228-1, J2 B3B-PH-K-S(LF)(SN), J3 Conn_02x03_Odd_Even, J4 LD09S13A4GX00LF, J5 USB_B, J6 RJ45, J7 B6B-XH-A(LF)(SN), J8 B10B-PHDSS(LF)(SN), J9 RJ45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

Commit message: second revision
Parts:
- J5: footprint Connector_USB:USB_B_OST_USB-B1HSxx_Horizontal -> Connector_USB:USB_B_TE_5787834_Vertical
Changed lines of the file:
@@
 F 0 "J5" H 6132 3617 50  0000 C CNN
 F 1 "USB_B" H 6132 3526 50  0000 C CNN
-F 2 "Connector_USB:USB_B_OST_USB-B1HSxx_Horizontal" H 6225 3100 50  0001 C CNN
+F 2 "Connector_USB:USB_B_TE_5787834_Vertical" H 6225 3100 50  0001 C CNN
 F 3 " ~" H 6225 3100 50  0001 C CNN
 	1    6075 3150
