File: LV_Breakout/LV_Breakout.sch (KiCad schematic (older format))
At the start: 18 parts

Commit message: finish sch and ready for review
Parts:
- removed J?: TO_BRB, symbol Connector_Generic:Conn_01x02
- removed J? (x4): Conn_01x02, symbol Connector_Generic:Conn_01x02
- removed K?: RT314A03, Relay_THT:Relay_SPDT_Schrack-RT1-16A-FormC_RM5mm, symbol Relay:DIPxx-1Axx-11x
- added F4: COOL, Fuse:Fuseholder_Blade_Mini_Keystone_3568, symbol Device:Fuse
- added F6: LV PWR, Fuse:Fuseholder_Blade_Mini_Keystone_3568, symbol Device:Fuse
- added J5: DAQ, Connector_JST:JST_PHD_B12B-PHDSS_2x06_P2.00mm_Vertical, symbol Connector_Generic:Conn_02x06_Counter_Clockwise
- added J7: PWR_AMPSEAL, aero_footprint:TE_1-776200-1_23pin_Vertical, symbol Connector_Generic:Conn_01x23
- added K1: RAYEX-L90B, Relay_THT:Relay_SPST_RAYEX-L90B, symbol Relay:RAYEX-L90A
- F1, F2, F3: renamed from F?; footprint (none) -> Fuse:Fuseholder_Blade_Mini_Keystone_3568
- F10: renamed from F?; value Fuse -> DCDC; footprint (none) -> Fuse:Fuseholder_Blade_Mini_Keystone_3568
- F5: renamed from F?; value Fuse -> LOGIC; footprint (none) -> Fuse:Fuseholder_Blade_Mini_Keystone_3568
- F7: renamed from F?; value DAQ -> FAN; footprint (none) -> Fuse:Fuseholder_Blade_Mini_Keystone_3568
- F8: renamed from F?; value Fuse -> BRB; footprint (none) -> Fuse:Fuseholder_Blade_Mini_Keystone_3568
- F9: renamed from F?; value Fuse -> Main GLV; footprint (none) -> Fuse:Fuseholder_Blade_Mini_Keystone_3568
- J1: renamed from J?; value Conn_01x02 -> LOGIC_PWR; footprint (none) -> aero_footprint:TE_MATE-N-LOK_1-770866-x_1x02_P4.14mm_Vertical
- J2: renamed from J?; footprint (none) -> aero_footprint:TE_MATE-N-LOK_1-770866-x_1x02_P4.14mm_Vertical
- J4: renamed from J?; footprint (none) -> Connector_JST:JST_PHD_B10B-PHDSS_2x05_P2.00mm_Vertical
- J6: renamed from J?; value Conn_01x23 -> DAQ_AMPSEAL; footprint (none) -> aero_footprint:TE_1-776200-1_23pin_Vertical; symbol Connector_Generic:Conn_01x35 -> Connector_Generic:Conn_01x23
Connections:
- net labels added: +5V, BMS+DAQ_PWR, COOL_PWR, FAN_PWR, LV_PWR, RINE_PWR
- net labels removed: BMS_PWR
- wire segments 87 -> 118
Other:
- note added: "DAQ Ampseal"
- note added: "Power Ampseal"
- note removed: "Main Ampseal"
- moved on the sheet: F1, F10, F3, F7, F8, F9, J1, J2

Commit message: Footprint updates of GLV board, pull the libraries repo please!
Parts:
- removed K1: RAYEX-L90B, Relay_THT:Relay_SPST_RAYEX-L90B, symbol Relay:RAYEX-L90A
- added K1: T9VV1K15-12S, AERO-footprints:RELAY_T9VV1K15-12S, symbol AERO_custom_symbols:T9VV1K15-12S
- F1, F10, F2, F3, F4, F5, F6, F7, F8, F9: footprint Fuse:Fuseholder_Blade_Mini_Keystone_3568 -> AERO-footprints:Fuseholder_Blade_Mini_Keystone_3568
- J1, J2: footprint aero_footprint:TE_MATE-N-LOK_1-770866-x_1x02_P4.14mm_Vertical -> AERO-footprints:TE_MATE-N-LOK_1-770866-x_1x02_P4.14mm_Vertical
- J4: footprint Connector_JST:JST_PHD_B10B-PHDSS_2x05_P2.00mm_Vertical -> AERO-footprints:JST_PHD_B10B-PHDSS_2x05_P2.00mm_Vertical
- J5: footprint Connector_JST:JST_PHD_B12B-PHDSS_2x06_P2.00mm_Vertical -> AERO-footprints:JST_PHD_B12B-PHDSS_2x06_P2.00mm_Vertical
- J6, J7: footprint aero_footprint:TE_1-776200-1_23pin_Vertical -> AERO-footprints:TE_1-776200-1_23pin_Vertical
Connections:
- wire segments 118 -> 119
Changed lines of the file:
@@
 EESchema Schematic File Version 4
+LIBS:LV_Breakout-cache
 EELAYER 30 0
 EELAYER END
@@
 Text Label 5450 4775 2    50   ~ 0
 FROM_BRB
-Wire Wire Line
-	5450 4775 4950 4775
-$Comp
-L Relay:RAYEX-L90A K1
-U 1 1 5E6B6E51
-P 4550 4975
-F 0 "K1" V 3983 4975 50  0000 C CNN
-F 1 "RAYEX-L90B" V 4074 4975 50  0000 C CNN
-F 2 "Relay_THT:Relay_SPST_RAYEX-L90B" H 4900 4925 50  0001 L CNN
-F 3 "https://a3.sofastcdn.com/attachment/7jioKBjnRiiSrjrjknRiwS77gwbf3zmp/L90-SERIES.pdf" H 5050 4825 50  0001 L CNN
-	1    4550 4975
-	0    1    1    0
-$EndComp
 Text Label 3100 5025 0    50   ~ 0
 DCDC_IN
@@
 F 0 "F10" V 3525 5025 50  0000 C CNN
 F 1 "DCDC" V 3675 5050 50  0000 C CNN
-F 2 "Fuse:Fuseholder_Blade_Mini_Keystone_3568" V 3530 5025 50  0001 C CNN
+F 2 "AERO-footprints:Fuseholder_Blade_Mini_Keystone_3568" V 3530 5025 50  0001 C CNN
 F 3 "~" H 3600 5025 50  0001 C CNN
 	1    3600 5025
@@
 F 0 "F9" V 3403 5250 50  0000 C CNN
 F 1 "Main GLV" V 3494 5250 50  0000 C CNN
-F 2 "Fuse:Fuseholder_Blade_Mini_Keystone_3568" V 3530 5250 50  0001 C CNN
+F 2 "AERO-footprints:Fuseholder_Blade_Mini_Keystone_3568" V 3530 5250 50  0001 C CNN
 F 3 "~" H 3600 5250 50  0001 C CNN
 	1    3600 5250
@@
 Wire Wire Line
 	3900 5250 3900 5175
-Wire Wire Line
-	4150 5175 3900 5175
 Wire Wire Line
 	3900 5025 3900 5175
@@
 F 0 "F4" V 2278 5200 50  0000 C CNN
 F 1 "COOL" V 2369 5200 50  0000 C CNN
-F 2 "Fuse:Fuseholder_Blade_Mini_Keystone_3568" V 2405 5200 50  0001 C CNN
+F 2 "AERO-footprints:Fuseholder_Blade_Mini_Keystone_3568" V 2405 5200 50  0001 C CNN
 F 3 "~" H 2475 5200 50  0001 C CNN
 	1    2475 5200
@@
 F 0 "F6" V 2278 5800 50  0000 C CNN
 F 1 "LV PWR" V 2369 5800 50  0000 C CNN
-F 2 "Fuse:Fuseholder_Blade_Mini_Keystone_3568" V 2405 5800 50  0001 C CNN
+F 2 "AERO-footprints:Fuseholder_Blade_Mini_Keystone_3568" V 2405 5800 50  0001 C CNN
 F 3 "~" H 2475 5800 50  0001 C CNN
 	1    2475 5800
@@
 F 0 "J1" V 1625 5450 50  0000 C CNN
 F 1 "LOGIC_PWR" V 1725 5350 50  0000 C CNN
-F 2 "aero_footprint:TE_MATE-N-LOK_1-770866-x_1x02_P4.14mm_Vertical" H 1625 5300 50  0001 C CNN
+F 2 "AERO-footprints:TE_MATE-N-LOK_1-770866-x_1x02_P4.14mm_Vertical" H 1625 5300 50  0001 C CNN
 F 3 "~" H 1625 5300 50  0001 C CNN
 	1    1625 5300
@@
 F 0 "F5" V 2278 5500 50  0000 C CNN
 F 1 "LOGIC" V 2369 5500 50  0000 C CNN
-F 2 "Fuse:Fuseholder_Blade_Mini_Keystone_3568" V 2405 5500 50  0001 C CNN
+F 2 "AERO-footprints:Fuseholder_Blade_Mini_Keystone_3568" V 2405 5500 50  0001 C CNN
 F 3 "~" H 2475 5500 50  0001 C CNN
 	1    2475 5500
@@
 F 0 "F7" V 2278 6100 50  0000 C CNN
 F 1 "FAN" V 2369 6100 50  0000 C CNN
-F 2 "Fuse:Fuseholder_Blade_Mini_Keystone_3568" V 2405 6100 50  0001 C CNN
+F 2 "AERO-footprints:Fuseholder_Blade_Mini_Keystone_3568" V 2405 6100 50  0001 C CNN
 F 3 "~" H 2475 6100 50  0001 C CNN
 	1    2475 6100
@@
 F 0 "F1" V 2278 4300 50  0000 C CNN
 F 1 "SHUTDOWN" V 2369 4300 50  0000 C CNN
-F 2 "Fuse:Fuseholder_Blade_Mini_Keystone_3568" V 2405 4300 50  0001 C CNN
+F 2 "AERO-footprints:Fuseholder_Blade_Mini_Keystone_3568" V 2405 4300 50  0001 C CNN
 F 3 "~" H 2475 4300 50  0001 C CNN
 	1    2475 4300
@@
 F 0 "F2" V 2278 4600 50  0000 C CNN
 F 1 "BMS" V 2369 4600 50  0000 C CNN
-F 2 "Fuse:Fuseholder_Blade_Mini_Keystone_3568" V 2405 4600 50  0001 C CNN
+F 2 "AERO-footprints:Fuseholder_Blade_Mini_Keystone_3568" V 2405 4600 50  0001 C CNN
 F 3 "~" H 2475 4600 50  0001 C CNN
 	1    2475 4600
@@
 F 0 "F3" V 2278 4900 50  0000 C CNN
 F 1 "RINEHART" V 2369 4900 50  0000 C CNN
-F 2 "Fuse:Fuseholder_Blade_Mini_Keystone_3568" V 2405 4900 50  0001 C CNN
+F 2 "AERO-footprints:Fuseholder_Blade_Mini_Keystone_3568" V 2405 4900 50  0001 C CNN
 F 3 "~" H 2475 4900 50  0001 C CNN
 	1    2475 4900
@@
 F 0 "F8" V 4375 5900 50  0000 L CNN
 F 1 "BRB" V 4525 5850 50  0000 L CNN
-F 2 "Fuse:Fuseholder_Blade_Mini_Keystone_3568" V 4380 5950 50  0001 C CNN
+F 2 "AERO-footprints:Fuseholder_Blade_Mini_Keystone_3568" V 4380 5950 50  0001 C CNN
 F 3 "~" H 4450 5950 50  0001 C CNN
 	1    4450 5950
@@
 F 0 "J2" H 3655 5942 50  0000 L CNN
 F 1 "GLV_IN" H 3525 6075 50  0000 L CNN
-F 2 "aero_footprint:TE_MATE-N-LOK_1-770866-x_1x02_P4.14mm_Vertical" H 3575 5950 50  0001 C CNN
+F 2 "AERO-footprints:TE_MATE-N-LOK_1-770866-x_1x02_P4.14mm_Vertical" H 3575 5950 50  0001 C CNN
 F 3 "~" H 3575 5950 50  0001 C CNN
 	1    3575 5950
@@
 $EndComp
 Wire Wire Line
-	5175 5275 4950 5275
+	5050 5175 4825 5175
 $Comp
 L power:+12V #PWR0101
 U 1 1 5E50D205
-P 5175 5275
-F 0 "#PWR0101" H 5175 5125 50  0001 C CNN
-F 1 "+12V" H 5190 5448 50  0000 C CNN
-F 2 "" H 5175 5275 50  0001 C CNN
-F 3 "" H 5175 5275 50  0001 C CNN
-	1    5175 5275
+P 5050 5175
+F 0 "#PWR0101" H 5050 5025 50  0001 C CNN
+F 1 "+12V" H 5065 5348 50  0000 C CNN
+F 2 "" H 5050 5175 50  0001 C CNN
+F 3 "" H 5050 5175 50  0001 C CNN
+	1    5050 5175
 	-1   0    0    -1
 $EndComp
@@
 F 0 "J7" H 8930 4392 50  0000 L CNN
 F 1 "PWR_AMPSEAL" V 8975 3250 50  0000 L CNN
-F 2 "aero_footprint:TE_1-776200-1_23pin_Vertical" H 8850 4350 50  0001 C CNN
+F 2 "AERO-footprints:TE_1-776200-1_23pin_Vertical" H 8850 4350 50  0001 C CNN
 F 3 "~" H 8850 4350 50  0001 C CNN
 	1    8850 4350
@@
 F 0 "J6" H 8205 4367 50  0000 L CNN
 F 1 "DAQ_AMPSEAL" V 8225 3450 50  0000 L CNN
-F 2 "aero_footprint:TE_1-776200-1_23pin_Vertical" H 8125 4325 50  0001 C CNN
+F 2 "AERO-footprints:TE_1-776200-1_23pin_Vertical" H 8125 4325 50  0001 C CNN
 F 3 "~" H 8125 4325 50  0001 C CNN
 	1    8125 4325
@@
 F 0 "J4" H 4625 2292 50  0000 C CNN
 F 1 "BMS" H 4625 2201 50  0000 C CNN
-F 2 "Connector_JST:JST_PHD_B10B-PHDSS_2x05_P2.00mm_Vertical" H 4575 1875 50  0001 C CNN
+F 2 "AERO-footprints:JST_PHD_B10B-PHDSS_2x05_P2.00mm_Vertical" H 4575 1875 50  0001 C CNN
 F 3 "~" H 4575 1875 50  0001 C CNN
 	1    4575 1875
@@
 Wire Wire Line
 	3800 2800 4375 2800
-$Comp
-L Connector_Generic:Conn_02x06_Counter_Clockwise J5
-U 1 1 5E5073C8
-P 4575 3000
-F 0 "J5" H 4625 3417 50  0000 C CNN
-F 1 "DAQ" H 4625 3326 50  0000 C CNN
-F 2 "Connector_JST:JST_PHD_B12B-PHDSS_2x06_P2.00mm_Vertical" H 4575 3000 50  0001 C CNN
-F 3 "~" H 4575 3000 50  0001 C CNN
-	1    4575 3000
-	1    0    0    -1
-$EndComp
 Text Notes 4275 4275 0    50   ~ 0
 RELAY\nGLV OR DCDC
@@
 	7075 4925 7075 4825
 Connection ~ 7075 4825
+$Comp
+L Connector_Generic:Conn_02x06_Counter_Clockwise J5
+U 1 1 5E5073C8
+P 4575 3000
+F 0 "J5" H 4625 3417 50  0000 C CNN
+F 1 "DAQ" H 4625 3326 50  0000 C CNN
+F 2 "AERO-footprints:JST_PHD_B12B-PHDSS_2x06_P2.00mm_Vertical" H 4575 3000 50  0001 C CNN
+F 3 "~" H 4575 3000 50  0001 C CNN
+	1    4575 3000
+	1    0    0    -1
+$EndComp
+$Comp
+L AERO_custom_symbols:T9VV1K15-12S K1
+U 1 1 5E50EFF5
+P 4525 4975
+F 0 "K1" V 3958 4975 50  0000 C CNN
+F 1 "T9VV1K15-12S" V 4049 4975 50  0000 C CNN
+F 2 "AERO-footprints:RELAY_T9VV1K15-12S" H 4875 4925 50  0001 L CNN
+F 3 "https://www.te.com/commerce/DocumentDelivery/DDEController?Action=srchrtrv&DocNm=Power_PCB_Relay_T9V_Solar&DocType=DS&DocLang=English" H 4525 4975 50  0001 C CNN
+	1    4525 4975
+	0    1    1    0
+$EndComp
+Wire Wire Line
+	4150 4775 4225 4775
+Wire Wire Line
+	4825 4775 5450 4775
+Wire Wire Line
+	3900 5175 4225 5175
 $EndSCHEMATC

Commit message: Final fixes to GLV board so it works with HV board
Parts:
- removed F10: DCDC, AERO-footprints:Fuseholder_Blade_Mini_Keystone_3568, symbol Device:Fuse
- added C1, C5: C, Capacitor_SMD:C_0603_1608Metric_Pad1.05x0.95mm_HandSolder, symbol Device:C
- added C2, C3, C4: URS1E472MHD, AERO-footprints:CAP_18x25_NICH, symbol Device:CP1
- added R1: RR01J2R0TB, AERO-footprints:NeOhm_RR01_Vert, symbol Device:R_US
- added R2: 50M, Resistor_SMD:R_0603_1608Metric_Pad1.05x0.95mm_HandSolder, symbol Device:R_US
- added U1: R-78E5.0-0.5, Converter_DCDC:Converter_DCDC_RECOM_R-78E-0.5_THT, symbol Regulator_Switching:R-78E5.0-0.5
- F8: value BRB -> BRB, 2A
- J2: value GLV_IN -> BATT_IN
Connections:
- net labels added: BATT_IN, SCL, SDA, VCAP_AB
- wire segments 119 -> 127
Other:
- note added: "Consider filter on input, see datasheet"
- note added: "Fuses for each source are upstream"
- note added: "Not sure how battery is actually conneting to this but I'm leaving that to you"
- note added: "Still needs DAQ, Other ampseal/molex/whatever, MCU, etc\n\nHas ideal diode and current monitor built in now, along with bulk storage caps"
- note added: "This part exists and works!"
- moved on the sheet: F1, F2, F3, F4, F5, F6, F7, F9, J1

Commit message: LVPDU schem and pcb
Parts:
- removed F4: COOL, AERO-footprints:Fuseholder_Blade_Mini_Keystone_3568, symbol Device:Fuse
- removed J5: DAQ, AERO-footprints:JST_PHD_B12B-PHDSS_2x06_P2.00mm_Vertical, symbol Connector_Generic:Conn_02x06_Counter_Clockwise
- removed J6: DAQ_AMPSEAL, AERO-footprints:TE_1-776200-1_23pin_Vertical, symbol Connector_Generic:Conn_01x23
- added F1, F10: 3568 Mini Blade, AERO_FOOT:Fuseholder_Blade_Mini_Keystone_3568, symbol Device:Fuse
- C1: value C -> 1u
- C2, C3, C4: footprint AERO-footprints:CAP_18x25_NICH -> Capacitor_THT:CP_Radial_D18.0mm_P7.50mm
- C5: value C -> 10u
- F2: value BMS -> 3568 Mini Blade; footprint AERO-footprints:Fuseholder_Blade_Mini_Keystone_3568 -> AERO_FOOT:Fuseholder_Blade_Mini_Keystone_3568
- F3: value RINEHART -> 3568 Mini Blade; footprint AERO-footprints:Fuseholder_Blade_Mini_Keystone_3568 -> AERO_FOOT:Fuseholder_Blade_Mini_Keystone_3568
- F4: renamed from F1; value SHUTDOWN -> 3568 Mini Blade; footprint AERO-footprints:Fuseholder_Blade_Mini_Keystone_3568 -> AERO_FOOT:Fuseholder_Blade_Mini_Keystone_3568
- F5: value LOGIC -> 3568 Mini Blade; footprint AERO-footprints:Fuseholder_Blade_Mini_Keystone_3568 -> AERO_FOOT:Fuseholder_Blade_Mini_Keystone_3568
- F6: value LV PWR -> 3568 Mini Blade; footprint AERO-footprints:Fuseholder_Blade_Mini_Keystone_3568 -> AERO_FOOT:Fuseholder_Blade_Mini_Keystone_3568
- F7: value FAN -> 3568 Mini Blade; footprint AERO-footprints:Fuseholder_Blade_Mini_Keystone_3568 -> AERO_FOOT:Fuseholder_Blade_Mini_Keystone_3568
- F8: value BRB, 2A -> 3568 Mini Blade; footprint AERO-footprints:Fuseholder_Blade_Mini_Keystone_3568 -> AERO_FOOT:Fuseholder_Blade_Mini_Keystone_3568
- F9: value Main GLV -> 3568 Mini Blade; footprint AERO-footprints:Fuseholder_Blade_Mini_Keystone_3568 -> AERO_FOOT:Fuseholder_Blade_Mini_Keystone_3568
- J1: renamed from J4; value BMS -> B10B-PHDSS(LF)(SN); footprint AERO-footprints:JST_PHD_B10B-PHDSS_2x05_P2.00mm_Vertical -> Connector_JST:JST_PHD_B8B-PHDSS_2x04_P2.00mm_Vertical; symbol Connector_Generic:Conn_02x05_Counter_Clockwise -> Connector_Generic:Conn_02x04_Counter_Clockwise
- J2: value BATT_IN -> DF22-2P-7.92DSA(05); footprint AERO-footprints:TE_MATE-N-LOK_1-770866-x_1x02_P4.14mm_Vertical -> Connector_JST:JST_VH_B2P3-VH_1x02_P7.92mm_Vertical
- J3: renamed from J1; value LOGIC_PWR -> TE 1-770872-0; footprint AERO-footprints:TE_MATE-N-LOK_1-770866-x_1x02_P4.14mm_Vertical -> AERO_CUSTOM:TE_MATE-N-LOK_1-770866-x_1x02_P4.14mm_Vertical
- J4: renamed from J7; value PWR_AMPSEAL -> TE 776228-1; footprint AERO-footprints:TE_1-776200-1_23pin_Vertical -> AERO_CUSTOM:TE_1-776200-1_23pin_Vertical
- K1: footprint AERO-footprints:RELAY_T9VV1K15-12S -> AERO_FOOT:RELAY_T9VV1K15-12S
- R1: footprint AERO-footprints:NeOhm_RR01_Vert -> Resistor_THT:R_Axial_DIN0207_L6.3mm_D2.5mm_P10.16mm_Horizontal
- R2: footprint Resistor_SMD:R_0603_1608Metric_Pad1.05x0.95mm_HandSolder -> Resistor_SMD:R_2512_6332Metric_Pad1.52x3.35mm_HandSolder
Connections:
- net labels added: DAQ_PWR, LOGIC
- net labels removed: BMS+DAQ_PWR, BMS_FAULT, CAN+, CAN-, SENSOR_1, SENSOR_2, SENSOR_3, SENSOR_4, SENSOR_5, SENSOR_6, SENSOR_7, USB+, USB-, USB_5V, USB_GND
- wire segments 127 -> 93
Other:
- note added: "12V to 5V for DAQ"
- note added: "Conn for DAQ\nand Port Pannel Board"
- note added: "Fuse Bank"
- note removed: "Consider filter on input, see datasheet"
- note removed: "DAQ Ampseal"
- note removed: "Fuses for each source are upstream"
- note removed: "Not sure how battery is actually conneting to this but I'm leaving that to you"
- note removed: "Still needs DAQ, Other ampseal/molex/whatever, MCU, etc\n\nHas ideal diode and current monitor built in now, along with bulk storage caps"
- note removed: "This part exists and works!"
- moved on the sheet: C2, C3, C4, F4, J2, J3, J4, K1, R1, R2

Commit message: second revision
Parts:
- J3: footprint AERO_CUSTOM:TE_MATE-N-LOK_1-770866-x_1x02_P4.14mm_Vertical -> AERO_CUSTOM:TE_MATE-N-LOK_1-770870-x_1x03_P4.14mm_Vertical; symbol Connector_Generic:Conn_01x02 -> Connector_Generic:Conn_01x03
Connections:
- wire segments 93 -> 98
Changed lines of the file:
@@
 	9775 2525 10075 2525
 Wire Wire Line
-	9475 1025 8875 1025
-Wire Wire Line
 	9475 1625 9100 1625
 Wire Wire Line
 	9475 1925 9100 1925
 $Comp
-L Connector_Generic:Conn_01x02 J3
+L Connector_Generic:Conn_01x03 J3
 U 1 1 5E5F0877
-P 8575 2025
-F 0 "J3" V 8575 2175 50  0000 C CNN
-F 1 "TE 1-770872-0" V 8675 2075 50  0000 C CNN
-F 2 "AERO_CUSTOM:TE_MATE-N-LOK_1-770866-x_1x02_P4.14mm_Vertical" H 8575 2025 50  0001 C CNN
-F 3 "~" H 8575 2025 50  0001 C CNN
-	1    8575 2025
-	0    -1   -1   0
+P 8600 2575
+F 0 "J3" V 8925 2550 50  0000 C CNN
+F 1 "TE 1-770872-0" V 8775 2550 50  0000 C CNN
+F 2 "AERO_CUSTOM:TE_MATE-N-LOK_1-770870-x_1x03_P4.14mm_Vertical" H 8600 2575 50  0001 C CNN
+F 3 "~" H 8600 2575 50  0001 C CNN
+	1    8600 2575
+	1    0    0    1
 $EndComp
 Connection ~ 10075 1925
@@
 	1    0    0    -1
 $EndComp
-Wire Wire Line
-	8675 2225 9475 2225
 $Comp
 L power:GND #PWR08
 U 1 1 5E7F9F43
-P 8575 2225
-F 0 "#PWR08" H 8575 1975 50  0001 C CNN
-F 1 "GND" H 8580 2052 50  0000 C CNN
-F 2 "" H 8575 2225 50  0001 C CNN
-F 3 "" H 8575 2225 50  0001 C CNN
-	1    8575 2225
-	1    0    0    -1
+P 8400 2925
+F 0 "#PWR08" H 8400 2675 50  0001 C CNN
+F 1 "GND" H 8405 2752 50  0000 C CNN
+F 2 "" H 8400 2925 50  0001 C CNN
+F 3 "" H 8400 2925 50  0001 C CNN
+	1    8400 2925
+	0    -1   -1   0
 $EndComp
 Text Label 9900 6100 2    50   ~ 0
@@
 Text Label 6275 3500 0    50   ~ 0
 FROM_BRB
-Wire Wire Line
-	6675 3500 6225 3500
 Wire Wire Line
 	5525 3900 5625 3900
@@
 	6550 6100 6550 6000
 Connection ~ 6550 6100
+Wire Wire Line
+	8400 2675 8400 2925
+Wire Wire Line
+	8700 1025 9475 1025
+Wire Wire Line
+	8200 2225 8200 2475
+Wire Wire Line
+	8200 2225 9475 2225
+Wire Wire Line
+	6225 3500 7400 3500
+Wire Wire Line
+	7400 3500 7400 2575
+Wire Wire Line
+	7400 2575 8400 2575
+Wire Wire Line
+	8200 2475 8400 2475
 $EndSCHEMATC

Commit message: Updated PCB Layout
Parts:
- added F11: 1812L075/24, Fuse:Fuse_1812_4532Metric_Pad1.30x3.40mm_HandSolder, symbol Device:Polyfuse
Connections:
- wire segments 98 -> 99
Changed lines of the file:
@@
 	0    1    1    0
 $EndComp
-Text Label 4425 6125 2    50   ~ 0
+Text Label 3725 6125 0    50   ~ 0
 DAQ_PWR
 Text Label 9125 2225 0    50   ~ 0
@@
 Wire Wire Line
 	8200 2475 8400 2475
+$Comp
+L Device:Polyfuse F11
+U 1 1 5E5ACD10
+P 4275 6125
+F 0 "F11" V 4050 6125 50  0000 C CNN
+F 1 "1812L075/24" V 4141 6125 50  0000 C CNN
+F 2 "Fuse:Fuse_1812_4532Metric_Pad1.30x3.40mm_HandSolder" H 4325 5925 50  0001 L CNN
+F 3 "~" H 4275 6125 50  0001 C CNN
+	1    4275 6125
+	0    1    1    0
+$EndComp
+Wire Wire Line
+	3725 6125 4125 6125
 $EndSCHEMATC
