File: LV_Breakout/LV_Breakout.sch (KiCad schematic (older format))
At the start: 23 parts, among them J1 B10B-PHDSS(LF)(SN), J2 DF22-2P-7.92DSA(05), J3 TE 1-770872-0, J4 TE 776228-1, K1 T9VV1K15-12S, U1 R-78E5.0-0.5

Commit message: Change trace and create Gerber
Changed lines of the file:
@@
 Wire Wire Line
 	9100 6200 9900 6200
-Text Label 9900 4700 2    50   ~ 0
+Text Label 9900 6200 2    50   ~ 0
 FROM_BRB
 Wire Wire Line
@@
 	10050 4200 9900 4200
 Connection ~ 9900 4200
-Text Label 9900 6200 2    50   ~ 0
+Text Label 9900 4700 2    50   ~ 0
 LV_PWR
 Wire Wire Line
