File: LV_Breakout/LV_Breakout.kicad_pcb (KiCad board)
At the start: 2 copper layers, 101.6 x 90.8 mm, 42 parts, among them J1 B10B-PHDSS(LF)(SN), J2 DF22-2P-7.92DSA(05), J3 TE 1-770872-0, J4 TE 776228-1, K1 T9VV1K15-12S, Q1 CSD18563Q5A, U1 R-78E5.0-0.5, U2 LM74700QDBVTQ1, U3 INA219AIDR, U4 INA219AIDR

Commit message: Minor changes / updates
Parts:
- added G***: LOGO, AERO_CUSTOM:AERO_Logo_15x6mm, B.Cu at (194.1, 32.0)
Changed lines of the file:
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@@
     (tracks 207)
     (zones 0)
-    (modules 42)
+    (modules 43)
     (nets 28)
   )
@@
     (add_net "Net-(C8-Pad1)")
     (add_net "Net-(C8-Pad2)")
-    (add_net "Net-(J3-Pad2)")
     (add_net "Net-(Q1-Pad2)")
   )
@@
     (uvia_drill 0.1)
   )
+  (module AERO_CUSTOM:AERO_Logo_15x6mm (layer B.Cu)
+    (at 194.056 32.004 180)
+    (fp_text reference G*** (at 0 0) (layer B.SilkS) hide
+      (effects (font (size 1.524 1.524) (thickness 0.3)) (justify mirror))
+    )
+    (fp_text value LOGO (at 0.75 0) (layer B.SilkS) hide
+      (effects (font (size 1.524 1.524) (thickness 0.3)) (justify mirror))
+    )
+    (fp_poly (pts (xy 6.892292 2.256606) (xy 7.522038 1.627588) (xy 7.522038 -1.522592) (xy 6.209332 -2.833934)
+      (xy 5.038016 -1.661096) (xy 5.038016 -1.378625) (xy 5.912672 -1.378625) (xy 6.024987 -1.494504)
+      (xy 6.137301 -1.610384) (xy 6.374849 -1.374656) (xy 6.612397 -1.138929) (xy 6.612397 1.208337)
+      (xy 6.262534 1.556887) (xy 5.912672 1.905436) (xy 5.912672 -1.378625) (xy 5.038016 -1.378625)
+      (xy 5.038016 1.662595) (xy 5.650281 2.27411) (xy 6.262545 2.885624) (xy 6.892292 2.256606)) (layer B.SilkS) (width 0.01))
+    (fp_poly (pts (xy 4.085094 2.369879) (xy 4.583195 1.870887) (xy 4.583195 0.963505) (xy 3.972357 0.349823)
+      (xy 4.295269 0.025563) (xy 4.618182 -0.298698) (xy 4.618182 -1.659646) (xy 4.801166 -1.844931)
+      (xy 4.984149 -2.030217) (xy 4.180096 -2.83427) (xy 3.395312 -2.046694) (xy 3.567904 -1.85427)
+      (xy 3.740497 -1.661846) (xy 3.742011 -1.206428) (xy 3.743526 -0.751011) (xy 3.358678 -0.367356)
+      (xy 2.973829 0.0163) (xy 2.973829 -1.699463) (xy 3.149146 -1.872144) (xy 3.324464 -2.044825)
+      (xy 2.931053 -2.439355) (xy 2.796179 -2.57326) (xy 2.678343 -2.687693) (xy 2.586396 -2.774262)
+      (xy 2.529184 -2.824577) (xy 2.515023 -2.833884) (xy 2.484378 -2.809858) (xy 2.414426 -2.743504)
+      (xy 2.313856 -2.643412) (xy 2.191358 -2.518171) (xy 2.10951 -2.433024) (xy 1.726618 -2.032164)
+      (xy 1.912896 -1.8482) (xy 2.099173 -1.664236) (xy 2.099173 0.472657) (xy 2.903857 0.472657)
+      (xy 3.349759 0.91856) (xy 3.795662 1.364463) (xy 2.903857 2.256268) (xy 2.903857 0.472657)
+      (xy 2.099173 0.472657) (xy 2.099173 1.764775) (xy 1.898879 1.967182) (xy 1.698585 2.169588)
+      (xy 2.046914 2.519229) (xy 2.395244 2.86887) (xy 3.586993 2.86887) (xy 4.085094 2.369879)) (layer B.SilkS) (width 0.01))
+    (fp_poly (pts (xy -2.126864 2.214321) (xy -1.487961 1.574717) (xy -1.819235 1.24206) (xy -2.150508 0.909403)
+      (xy -2.632141 1.390114) (xy -3.113774 1.870826) (xy -3.113774 0.416909) (xy -2.449463 0.427118)
+      (xy -1.785151 0.437328) (xy -2.212781 0.008746) (xy -2.64041 -0.419835) (xy -3.113774 -0.419835)
+      (xy -3.113774 -1.430874) (xy -2.989067 -1.525994) (xy -2.864359 -1.621113) (xy -2.507589 -1.265558)
+      (xy -2.15082 -0.910002) (xy -1.835197 -1.225625) (xy -1.519575 -1.541248) (xy -2.169155 -2.187566)
+      (xy -2.34366 -2.360587) (xy -2.501708 -2.516125) (xy -2.636615 -2.647697) (xy -2.741696 -2.748821)
+      (xy -2.810268 -2.813012) (xy -2.835454 -2.833884) (xy -2.863865 -2.810205) (xy -2.934415 -2.7438)
+      (xy -3.039961 -2.641616) (xy -3.173361 -2.510602) (xy -3.327474 -2.357704) (xy -3.420301 -2.264972)
+      (xy -3.98843 -1.69606) (xy -3.98843 1.624396) (xy -3.377098 2.23916) (xy -2.765766 2.853925)
+      (xy -2.126864 2.214321)) (layer B.SilkS) (width 0.01))
+    (fp_poly (pts (xy -5.221339 2.265012) (xy -4.618182 1.661116) (xy -4.618182 -1.659646) (xy -4.435198 -1.844931)
+      (xy -4.252214 -2.030217) (xy -4.654241 -2.432243) (xy -5.056267 -2.83427) (xy -5.457346 -2.43205)
+      (xy -5.858424 -2.02983) (xy -5.492838 -1.659646) (xy -5.492838 -0.944628) (xy -6.262535 -0.944628)
+      (xy -6.262535 -1.659646) (xy -6.079551 -1.844931) (xy -5.896567 -2.030217) (xy -6.70062 -2.83427)
+      (xy -7.502776 -2.02983) (xy -7.319984 -1.844738) (xy -7.13719 -1.659646) (xy -7.13719 -0.034986)
+      (xy -6.262535 -0.034986) (xy -5.492838 -0.034986) (xy -5.492838 1.10401) (xy -5.875913 1.50538)
+      (xy -6.258989 1.906749) (xy -6.260762 0.935881) (xy -6.262535 -0.034986) (xy -7.13719 -0.034986)
+      (xy -7.13719 1.557578) (xy -6.480843 2.213243) (xy -5.824495 2.868909) (xy -5.221339 2.265012)) (layer B.SilkS) (width 0.01))
+    (fp_poly (pts (xy 0.892149 2.064187) (xy 0.53294 1.084573) (xy 1.076576 1.084573) (xy 1.281642 1.084154)
+      (xy 1.425832 1.082139) (xy 1.518241 1.077389) (xy 1.567965 1.068766) (xy 1.5841 1.055131)
+      (xy 1.575739 1.035346) (xy 1.565711 1.023347) (xy 1.537708 0.986527) (xy 1.472995 0.898463)
+      (xy 1.375622 0.764785) (xy 1.24964 0.591123) (xy 1.0991 0.383107) (xy 0.928052 0.146367)
+      (xy 0.740547 -0.113466) (xy 0.540636 -0.390763) (xy 0.33237 -0.679893) (xy 0.1198 -0.975227)
+      (xy -0.093025 -1.271134) (xy -0.302053 -1.561985) (xy -0.503233 -1.842148) (xy -0.692515 -2.105995)
+      (xy -0.865847 -2.347895) (xy -1.019181 -2.562217) (xy -1.148463 -2.743333) (xy -1.249645 -2.885611)
+      (xy -1.318674 -2.983422) (xy -1.351501 -3.031136) (xy -1.35222 -3.032265) (xy -1.349457 -3.013674)
+      (xy -1.325691 -2.935209) (xy -1.282989 -2.803056) (xy -1.223417 -2.623402) (xy -1.149041 -2.402431)
+      (xy -1.061928 -2.146332) (xy -0.964145 -1.861288) (xy -0.871159 -1.592142) (xy -0.764276 -1.283551)
+      (xy -0.664769 -0.995885) (xy -0.574915 -0.735757) (xy -0.496994 -0.509778) (xy -0.433282 -0.32456)
+      (xy -0.386058 -0.186716) (xy -0.357599 -0.102858) (xy -0.349862 -0.078987) (xy -0.382823 -0.075836)
+      (xy -0.473606 -0.073166) (xy -0.610059 -0.071186) (xy -0.780034 -0.070108) (xy -0.869786 -0.069973)
+      (xy -1.389709 -0.069973) (xy -0.998949 0.81343) (xy -0.875406 1.092997) (xy -0.742067 1.395195)
+      (xy -0.60729 1.701053) (xy -0.479431 1.9916) (xy -0.366846 2.247865) (xy -0.313152 2.370317)
+      (xy -0.018117 3.043801) (xy 1.251357 3.043801) (xy 0.892149 2.064187)) (layer B.SilkS) (width 0.01))
+  )
   (module AERO_FOOT:DF22-2P-7.92DSA05 (layer F.Cu)
     (at 201.93 58.166 90)
@@
   (segment (start 169.545 73.66) (end 169.545 78.597801) (width 1.2) (layer F.Cu) (net 8))
   (via (at 155.448 48.768) (size 2.8) (drill 1.8) (layers F.Cu B.Cu) (net 9))
-  (via (at 179.832 79.248) (size 2.8) (drill 1.8) (layers F.Cu B.Cu) (net 9))
+  (via (at 177.8 77.47) (size 2.8) (drill 1.8) (layers F.Cu B.Cu) (net 9))
   (segment (start 174.78 71.915) (end 173.54501 70.68001) (width 0.625) (layer F.Cu) (net 10))
   (segment (start 174.78 72.39) (end 174.78 71.915) (width 0.625) (layer F.Cu) (net 10))
@@
     (polygon
       (pts
-        (xy 158.496 92.964) (xy 151.384 92.964) (xy 137.668 111.252) (xy 122.936 111.252) (xy 122.936 97.028)
-        (xy 129.54 97.028) (xy 141.732 84.328) (xy 158.496 83.82)
+        (xy 159.004 92.964) (xy 151.384 92.964) (xy 137.668 111.252) (xy 122.936 111.252) (xy 122.936 97.028)
+        (xy 129.54 97.028) (xy 141.732 84.328) (xy 159.004 83.82)
       )
     )
@@
     (min_thickness 0.05)
     (keepout (tracks allowed) (vias allowed) (copperpour not_allowed))
-    (fill (arc_segments 32) (thermal_gap 0.5) (thermal_bridge_width 1) (smoothing chamfer))
+    (fill (arc_segments 32) (thermal_gap 0.5) (thermal_bridge_width 1))
     (polygon
       (pts

Commit message: Update 3d of lv breakout
Parts:
- C2, C3, C4: footprint Capacitor_THT:CP_Radial_D18.0mm_P7.50mm -> AERO_FOOT:CAP_18x25_NICH
- J1: value B10B-PHDSS(LF)(SN) -> B8B-PHDSS(LF)(SN)
- J3: value TE 1-770872-0 -> 1-770873-0; footprint AERO_CUSTOM:TE_MATE-N-LOK_1-770870-x_1x03_P4.14mm_Vertical -> AERO_FOOT:TE_MATE-N-LOK_1-770870-x_1x03_P4.14mm_Vertical
- J4: footprint AERO_CUSTOM:TE_1-776200-1_23pin_Vertical -> AERO_FOOT:TE_1-776228-1_23P_VERT_ASM
