File: dash-2019-2020/Left_rev2/left-board_rev2.kicad_pcb (KiCad board)
At the start: 2 copper layers, 43.2 x 19.7 mm, 8 parts, among them J1 B5B-PH-SM4-TB(LF)(SN)

Commit message: layout changes
Parts:
- removed the G*** at (135.3, 43.8)
- removed the G*** at (119.4, 39.4)
