File: dash-2019-2020/Right_rev2/_autosave-right.sch (KiCad schematic (older format))
At the start: 34 parts, among them J1 JST-XH, J11 Conn_01x03, J12 Conn_02x03_Odd_Even, J13 JST-XH, J2 JST-XH, J3 AMPSEAL, J5 B5B-PH-SM4-TB(LF)(SN), J8 JST-XH, Q1 MMBT2222ALT1G, U1 R-78E5.0-1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

Commit message: layout changes
Parts:
- added J4: 1-770966-0, AERO_FOOT:TE_MATE-N-LOK_1-770866-x_1x02_P4.14mm_Vertical, symbol Connector_Generic:Conn_01x02
Connections:
- net SHUTDOWN_IN: now also J4.2 (Pin_2)
- net SHUTDOWN_OUT: now also J4.1 (Pin_1)
Changed lines of the file:
@@
 	3050 7000 2650 7000
 $Comp
-L power:+12V #PWR?
+L power:+12V #PWR0113
 U 1 1 5E6A8867
 P 2650 5200
-F 0 "#PWR?" H 2650 5050 50  0001 C CNN
+F 0 "#PWR0113" H 2650 5050 50  0001 C CNN
 F 1 "+12V" V 2665 5328 50  0000 L CNN
 F 2 "" H 2650 5200 50  0001 C CNN
@@
 $EndComp
 $Comp
-L power:+12V #PWR?
+L power:+12V #PWR0120
 U 1 1 5E6A8871
 P 2650 5300
-F 0 "#PWR?" H 2650 5150 50  0001 C CNN
+F 0 "#PWR0120" H 2650 5150 50  0001 C CNN
 F 1 "+12V" V 2665 5428 50  0000 L CNN
 F 2 "" H 2650 5300 50  0001 C CNN
@@
 Wire Wire Line
 	3225 5000 2650 5000
+$Comp
+L Connector_Generic:Conn_01x02 J4
+U 1 1 5E6CAAE9
+P 3575 1475
+F 0 "J4" H 3493 1150 50  0000 C CNN
+F 1 "1-770966-0" H 3493 1241 50  0000 C CNN
+F 2 "AERO_FOOT:TE_MATE-N-LOK_1-770866-x_1x02_P4.14mm_Vertical" H 3575 1475 50  0001 C CNN
+F 3 "~" H 3575 1475 50  0001 C CNN
+	1    3575 1475
+	-1   0    0    1
+$EndComp
+Text Label 4350 1375 2    50   ~ 0
+SHUTDOWN_IN
+Wire Wire Line
+	4350 1375 3775 1375
+Text Label 4350 1475 2    50   ~ 0
+SHUTDOWN_OUT
+Wire Wire Line
+	4350 1475 3775 1475
 $EndSCHEMATC
