File: dash-2019-2020/Right_rev2/right.sch (KiCad schematic (older format))
At the start: 33 parts, among them J1 JST-XH, J11 Conn_01x03, J12 Conn_02x03_Odd_Even, J13 JST-XH, J2 JST-XH, J3 AMPSEAL, J5 B5B-PH-SM4-TB(LF)(SN), J8 JST-XH, Q1 MMBT2222ALT1G, U1 R-78E5.0-0.5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

Commit message: Minor Layout Changes
Parts:
- added J4: JST-XH, Connector_JST:JST_XH_S3B-XH-A_1x03_P2.50mm_Horizontal, symbol Connector_Generic:Conn_01x03
- added Q2: PSMN5R2-60YL, Package_TO_SOT_SMD:LFPAK56, symbol Transistor_FET:PSMN5R2-60YL
- added R8: 100, Resistor_SMD:R_0603_1608Metric_Pad1.05x0.95mm_HandSolder, symbol Device:R
- added R9: 1k, Resistor_SMD:R_0603_1608Metric_Pad1.05x0.95mm_HandSolder, symbol Device:R
- U1: value R-78E5.0-0.5 -> R-78E5.0-1
Connections:
- net +12V: now also J4.1 (Pin_1)
- net GND: now also J4.3 (Pin_3), Q2.1 (S), Q2.2 (S), Q2.3 (S), R8.2; no longer J3.20 (Pin_20)
- new net: Q2.5 (D), R9.2
- new net Horn_In: J3.20 (Pin_20), Q2.4 (G), R8.1
- new net Horn_Out: J4.2 (Pin_2), R9.1
Other:
- note added: "Hall Effect have\n+5V"
- note added: "String Pots have \n+12V in"
Changed lines of the file:
@@
 Wire Wire Line
 	10050 2550 10450 2550
-Wire Wire Line
-	2650 5400 3150 5400
-Wire Wire Line
-	2650 5500 3150 5500
 Text Label 3150 5400 2    50   ~ 0
 SPEED_R
@@
 P 5950 5550
 F 0 "U1" H 5950 5792 50  0000 C CNN
-F 1 "R-78E5.0-0.5" H 5950 5701 50  0000 C CNN
+F 1 "R-78E5.0-1" H 5950 5701 50  0000 C CNN
 F 2 "Converter_DCDC:Converter_DCDC_RECOM_R-78E-0.5_THT" H 5950 5750 50  0001 C CNN
 F 3 "" H 6050 5300 50  0001 C CNN
@@
 $EndComp
 $Comp
-L power:GND #PWR0111
-U 1 1 5E4B1527
-P 2650 6000
-F 0 "#PWR0111" H 2650 5750 50  0001 C CNN
-F 1 "GND" V 2655 5872 50  0000 R CNN
-F 2 "" H 2650 6000 50  0001 C CNN
-F 3 "" H 2650 6000 50  0001 C CNN
-	1    2650 6000
-	0    -1   1    0
-$EndComp
-$Comp
 L power:GND #PWR0112
 U 1 1 5E4B187E
@@
 Wire Wire Line
 	10050 3250 10400 3250
-$Comp
-L power:GND #PWR0115
-U 1 1 5E5E7040
-P 2650 6700
-F 0 "#PWR0115" H 2650 6450 50  0001 C CNN
-F 1 "GND" V 2655 6572 50  0000 R CNN
-F 2 "" H 2650 6700 50  0001 C CNN
-F 3 "" H 2650 6700 50  0001 C CNN
-	1    2650 6700
-	0    -1   1    0
-$EndComp
 $Comp
 L Mechanical:MountingHole H1
@@
 	0    1    -1   0
 $EndComp
+Text Notes 3325 5275 0    50   ~ 0
+String Pots have \n+12V in
+Text Notes 3325 5475 0    50   ~ 0
+Hall Effect have\n+5V
+Wire Wire Line
+	2650 5500 3150 5500
+Wire Wire Line
+	2650 5400 3150 5400
+Text Label 3025 6700 2    50   ~ 0
+Horn_In
+Wire Wire Line
+	3025 6700 2650 6700
+Text Label 2775 2575 2    50   ~ 0
+Horn_Out
+$Comp
+L Transistor_FET:PSMN5R2-60YL Q2
+U 1 1 5E61F43C
+P 4375 5800
+F 0 "Q2" H 4580 5846 50  0000 L CNN
+F 1 "PSMN5R2-60YL" H 4580 5755 50  0000 L CNN
+F 2 "Package_TO_SOT_SMD:LFPAK56" H 4525 5800 50  0001 C CNN
+F 3 "https://assets.nexperia.com/documents/data-sheet/PSMN5R2-60YL.pdf" H 4375 5800 50  0001 C CNN
+	1    4375 5800
+	1    0    0    -1
+$EndComp
+$Comp
+L Device:R R8
+U 1 1 5E62062E
+P 4100 5950
+F 0 "R8" H 4170 5996 50  0000 L CNN
+F 1 "100" H 4170 5905 50  0000 L CNN
+F 2 "Resistor_SMD:R_0603_1608Metric_Pad1.05x0.95mm_HandSolder" V 4030 5950 50  0001 C CNN
+F 3 "~" H 4100 5950 50  0001 C CNN
+	1    4100 5950
+	1    0    0    -1
+$EndComp
+$Comp
+L power:GND #PWR0111
+U 1 1 5E6210B2
+P 4475 6150
+F 0 "#PWR0111" H 4475 5900 50  0001 C CNN
+F 1 "GND" H 4480 5977 50  0000 C CNN
+F 2 "" H 4475 6150 50  0001 C CNN
+F 3 "" H 4475 6150 50  0001 C CNN
+	1    4475 6150
+	1    0    0    -1
+$EndComp
+Text Label 4475 5200 0    50   ~ 0
+Horn_Out
+Wire Wire Line
+	4475 5500 4475 5600
+Text Label 3725 5800 0    50   ~ 0
+Horn_In
+Wire Wire Line
+	3725 5800 4100 5800
+Connection ~ 4100 5800
+Wire Wire Line
+	4100 5800 4175 5800
+Wire Wire Line
+	4100 6100 4100 6150
+Wire Wire Line
+	4100 6150 4475 6150
+Wire Wire Line
+	4475 6150 4475 6000
+Connection ~ 4475 6150
+$Comp
+L Device:R R9
+U 1 1 5E64A6EA
+P 4475 5350
+F 0 "R9" H 4545 5396 50  0000 L CNN
+F 1 "1k" H 4545 5305 50  0000 L CNN
+F 2 "Resistor_SMD:R_0603_1608Metric_Pad1.05x0.95mm_HandSolder" V 4405 5350 50  0001 C CNN
+F 3 "~" H 4475 5350 50  0001 C CNN
+	1    4475 5350
+	1    0    0    -1
+$EndComp
+$Comp
+L power:GND #PWR0115
+U 1 1 5E672C3D
+P 2650 6000
+F 0 "#PWR0115" H 2650 5750 50  0001 C CNN
+F 1 "GND" V 2655 5872 50  0000 R CNN
+F 2 "" H 2650 6000 50  0001 C CNN
+F 3 "" H 2650 6000 50  0001 C CNN
+	1    2650 6000
+	0    -1   -1   0
+$EndComp
+$Comp
+L power:GND #PWR0121
+U 1 1 5E68FCBD
+P 2475 2475
+F 0 "#PWR0121" H 2475 2225 50  0001 C CNN
+F 1 "GND" V 2480 2347 50  0000 R CNN
+F 2 "" H 2475 2475 50  0001 C CNN
+F 3 "" H 2475 2475 50  0001 C CNN
+	1    2475 2475
+	0    -1   -1   0
+$EndComp
+Wire Wire Line
+	2475 2475 2375 2475
+Wire Wire Line
+	2375 2575 2775 2575
+Wire Wire Line
+	2475 2675 2375 2675
+$Comp
+L Connector_Generic:Conn_01x03 J4
+U 1 1 5E68FCCB
+P 2175 2575
+F 0 "J4" H 2093 2250 50  0000 C CNN
+F 1 "JST-XH" H 2093 2341 50  0000 C CNN
+F 2 "Connector_JST:JST_XH_S3B-XH-A_1x03_P2.50mm_Horizontal" H 2175 2575 50  0001 C CNN
+F 3 "~" H 2175 2575 50  0001 C CNN
+	1    2175 2575
+	-1   0    0    1
+$EndComp
+$Comp
+L power:+12V #PWR0120
+U 1 1 5E6B3597
+P 2475 2675
+F 0 "#PWR0120" H 2475 2525 50  0001 C CNN
+F 1 "+12V" V 2490 2803 50  0000 L CNN
+F 2 "" H 2475 2675 50  0001 C CNN
+F 3 "" H 2475 2675 50  0001 C CNN
+	1    2475 2675
+	0    1    1    0
+$EndComp
 $EndSCHEMATC

Commit message: layout changes
Parts:
- removed J4: JST-XH, Connector_JST:JST_XH_S3B-XH-A_1x03_P2.50mm_Horizontal, symbol Connector_Generic:Conn_01x03
- removed Q2: PSMN5R2-60YL, Package_TO_SOT_SMD:LFPAK56, symbol Transistor_FET:PSMN5R2-60YL
- removed R9: 1k, Resistor_SMD:R_0603_1608Metric_Pad1.05x0.95mm_HandSolder, symbol Device:R
- R8: value 100 -> 1k
Connections:
- net +12V: now also J8.2 (Pin_2)
- net +5V: no longer J8.2 (Pin_2)
- net GND: now also J3.20 (Pin_20); no longer R8.2
- net at Q1.3 (C): now also R8.1; no longer J8.1 (Pin_1)
- removed net Horn_In: J3.20 (Pin_20), R8.1
- new net: J8.1 (Pin_1), R8.2
Other:
- moved on the sheet: Q1
Changed lines of the file:
@@
 Text Label 1650 3850 2    50   ~ 0
 BRAKE
-Text Label 1750 2550 2    50   ~ 0
+Text Label 2200 2550 2    50   ~ 0
 RTD_IND
 Wire Wire Line
-	1750 2550 1450 2550
+	2200 2550 1900 2550
 Wire Wire Line
 	1250 3250 1350 3250
@@
 L Transistor_BJT:MMBT5550L Q1
 U 1 1 5DFCE072
-P 1250 2550
-F 0 "Q1" H 1100 2350 60  0000 L CNN
-F 1 "MMBT2222ALT1G" H 600 2750 60  0000 L CNN
-F 2 "Package_TO_SOT_SMD:SOT-23" H 1450 2750 60  0001 L CNN
-F 3 "http://www.onsemi.com/pub/Collateral/MMBT2222LT1-D.PDF" H 1450 2850 60  0001 L CNN
-F 4 "MMBT2222ALT1GOSCT-ND" H 1450 2950 60  0001 L CNN "Digi-Key_PN"
-F 5 "MMBT2222ALT1G" H 1450 3050 60  0001 L CNN "MPN"
-F 6 "Discrete Semiconductor Products" H 1450 3150 60  0001 L CNN "Category"
-F 7 "Transistors - Bipolar (BJT) - Single" H 1450 3250 60  0001 L CNN "Family"
-F 8 "http://www.onsemi.com/pub/Collateral/MMBT2222LT1-D.PDF" H 1450 3350 60  0001 L CNN "DK_Datasheet_Link"
-F 9 "/product-detail/en/on-semiconductor/MMBT2222ALT1G/MMBT2222ALT1GOSCT-ND/1139806" H 1450 3450 60  0001 L CNN "DK_Detail_Page"
-F 10 "TRANS NPN 40V 0.6A SOT23" H 1450 3550 60  0001 L CNN "Description"
-F 11 "ON Semiconductor" H 1450 3650 60  0001 L CNN "Manufacturer"
-F 12 "Active" H 1450 3750 60  0001 L CNN "Status"
-	1    1250 2550
+P 1700 2550
+F 0 "Q1" H 1550 2350 60  0000 L CNN
+F 1 "MMBT2222ALT1G" H 1050 2750 60  0000 L CNN
+F 2 "Package_TO_SOT_SMD:SOT-23" H 1900 2750 60  0001 L CNN
+F 3 "http://www.onsemi.com/pub/Collateral/MMBT2222LT1-D.PDF" H 1900 2850 60  0001 L CNN
+F 4 "MMBT2222ALT1GOSCT-ND" H 1900 2950 60  0001 L CNN "Digi-Key_PN"
+F 5 "MMBT2222ALT1G" H 1900 3050 60  0001 L CNN "MPN"
+F 6 "Discrete Semiconductor Products" H 1900 3150 60  0001 L CNN "Category"
+F 7 "Transistors - Bipolar (BJT) - Single" H 1900 3250 60  0001 L CNN "Family"
+F 8 "http://www.onsemi.com/pub/Collateral/MMBT2222LT1-D.PDF" H 1900 3350 60  0001 L CNN "DK_Datasheet_Link"
+F 9 "/product-detail/en/on-semiconductor/MMBT2222ALT1G/MMBT2222ALT1GOSCT-ND/1139806" H 1900 3450 60  0001 L CNN "DK_Detail_Page"
+F 10 "TRANS NPN 40V 0.6A SOT23" H 1900 3550 60  0001 L CNN "Description"
+F 11 "ON Semiconductor" H 1900 3650 60  0001 L CNN "Manufacturer"
+F 12 "Active" H 1900 3750 60  0001 L CNN "Status"
+	1    1700 2550
 	-1   0    0    -1
-$EndComp
-$Comp
-L power:+5V #PWR0117
-U 1 1 5DFE74FA
-P 1350 2200
-F 0 "#PWR0117" H 1350 2050 50  0001 C CNN
-F 1 "+5V" H 1365 2373 50  0000 C CNN
-F 2 "" H 1350 2200 50  0001 C CNN
-F 3 "" H 1350 2200 50  0001 C CNN
-	1    1350 2200
-	1    0    0    -1
 $EndComp
 Wire Wire Line
@@
 L power:GND #PWR0118
 U 1 1 5E06CBE5
-P 1150 2750
-F 0 "#PWR0118" H 1150 2500 50  0001 C CNN
-F 1 "GND" H 1155 2577 50  0000 C CNN
-F 2 "" H 1150 2750 50  0001 C CNN
-F 3 "" H 1150 2750 50  0001 C CNN
-	1    1150 2750
+P 1600 2750
+F 0 "#PWR0118" H 1600 2500 50  0001 C CNN
+F 1 "GND" H 1605 2577 50  0000 C CNN
+F 2 "" H 1600 2750 50  0001 C CNN
+F 3 "" H 1600 2750 50  0001 C CNN
+	1    1600 2750
 	1    0    0    -1
 $EndComp
@@
 Wire Wire Line
 	2650 5400 3150 5400
-Text Label 3025 6700 2    50   ~ 0
-Horn_In
-Wire Wire Line
-	3025 6700 2650 6700
-Text Label 2775 2575 2    50   ~ 0
-Horn_Out
-$Comp
-L Transistor_FET:PSMN5R2-60YL Q2
-U 1 1 5E61F43C
-P 4375 5800
-F 0 "Q2" H 4580 5846 50  0000 L CNN
-F 1 "PSMN5R2-60YL" H 4580 5755 50  0000 L CNN
-F 2 "Package_TO_SOT_SMD:LFPAK56" H 4525 5800 50  0001 C CNN
-F 3 "https://assets.nexperia.com/documents/data-sheet/PSMN5R2-60YL.pdf" H 4375 5800 50  0001 C CNN
-	1    4375 5800
-	1    0    0    -1
-$EndComp
-$Comp
-L Device:R R8
-U 1 1 5E62062E
-P 4100 5950
-F 0 "R8" H 4170 5996 50  0000 L CNN
-F 1 "100" H 4170 5905 50  0000 L CNN
-F 2 "Resistor_SMD:R_0603_1608Metric_Pad1.05x0.95mm_HandSolder" V 4030 5950 50  0001 C CNN
-F 3 "~" H 4100 5950 50  0001 C CNN
-	1    4100 5950
-	1    0    0    -1
-$EndComp
-$Comp
-L power:GND #PWR0111
-U 1 1 5E6210B2
-P 4475 6150
-F 0 "#PWR0111" H 4475 5900 50  0001 C CNN
-F 1 "GND" H 4480 5977 50  0000 C CNN
-F 2 "" H 4475 6150 50  0001 C CNN
-F 3 "" H 4475 6150 50  0001 C CNN
-	1    4475 6150
-	1    0    0    -1
-$EndComp
-Text Label 4475 5200 0    50   ~ 0
-Horn_Out
-Wire Wire Line
-	4475 5500 4475 5600
-Text Label 3725 5800 0    50   ~ 0
-Horn_In
-Wire Wire Line
-	3725 5800 4100 5800
-Connection ~ 4100 5800
-Wire Wire Line
-	4100 5800 4175 5800
-Wire Wire Line
-	4100 6100 4100 6150
-Wire Wire Line
-	4100 6150 4475 6150
-Wire Wire Line
-	4475 6150 4475 6000
-Connection ~ 4475 6150
-$Comp
-L Device:R R9
-U 1 1 5E64A6EA
-P 4475 5350
-F 0 "R9" H 4545 5396 50  0000 L CNN
-F 1 "1k" H 4545 5305 50  0000 L CNN
-F 2 "Resistor_SMD:R_0603_1608Metric_Pad1.05x0.95mm_HandSolder" V 4405 5350 50  0001 C CNN
-F 3 "~" H 4475 5350 50  0001 C CNN
-	1    4475 5350
-	1    0    0    -1
-$EndComp
 $Comp
 L power:GND #PWR0115
@@
 $EndComp
 $Comp
-L power:GND #PWR0121
-U 1 1 5E68FCBD
-P 2475 2475
-F 0 "#PWR0121" H 2475 2225 50  0001 C CNN
-F 1 "GND" V 2480 2347 50  0000 R CNN
-F 2 "" H 2475 2475 50  0001 C CNN
-F 3 "" H 2475 2475 50  0001 C CNN
-	1    2475 2475
-	0    -1   -1   0
-$EndComp
-Wire Wire Line
-	2475 2475 2375 2475
-Wire Wire Line
-	2375 2575 2775 2575
-Wire Wire Line
-	2475 2675 2375 2675
-$Comp
-L Connector_Generic:Conn_01x03 J4
-U 1 1 5E68FCCB
-P 2175 2575
-F 0 "J4" H 2093 2250 50  0000 C CNN
-F 1 "JST-XH" H 2093 2341 50  0000 C CNN
-F 2 "Connector_JST:JST_XH_S3B-XH-A_1x03_P2.50mm_Horizontal" H 2175 2575 50  0001 C CNN
-F 3 "~" H 2175 2575 50  0001 C CNN
-	1    2175 2575
-	-1   0    0    1
-$EndComp
-$Comp
-L power:+12V #PWR0120
-U 1 1 5E6B3597
-P 2475 2675
-F 0 "#PWR0120" H 2475 2525 50  0001 C CNN
-F 1 "+12V" V 2490 2803 50  0000 L CNN
-F 2 "" H 2475 2675 50  0001 C CNN
-F 3 "" H 2475 2675 50  0001 C CNN
-	1    2475 2675
-	0    1    1    0
-$EndComp
+L power:+12V #PWR0117
+U 1 1 5E6DE99C
+P 1350 2200
+F 0 "#PWR0117" H 1350 2050 50  0001 C CNN
+F 1 "+12V" H 1365 2373 50  0000 C CNN
+F 2 "" H 1350 2200 50  0001 C CNN
+F 3 "" H 1350 2200 50  0001 C CNN
+	1    1350 2200
+	1    0    0    -1
+$EndComp
+$Comp
+L power:GND #PWR0111
+U 1 1 5E6FD50F
+P 2650 6700
+F 0 "#PWR0111" H 2650 6450 50  0001 C CNN
+F 1 "GND" V 2655 6572 50  0000 R CNN
+F 2 "" H 2650 6700 50  0001 C CNN
+F 3 "" H 2650 6700 50  0001 C CNN
+	1    2650 6700
+	0    -1   1    0
+$EndComp
+$Comp
+L Device:R R8
+U 1 1 5E61F1C3
+P 1300 2350
+F 0 "R8" V 1400 2325 50  0000 C CNN
+F 1 "1k" V 1300 2350 50  0000 C CNN
+F 2 "Resistor_SMD:R_0603_1608Metric_Pad1.05x0.95mm_HandSolder" V 1230 2350 50  0001 C CNN
+F 3 "~" H 1300 2350 50  0001 C CNN
+	1    1300 2350
+	0    1    1    0
+$EndComp
+Wire Wire Line
+	1600 2350 1450 2350
 $EndSCHEMATC

Commit message: init review
Parts:
- added F?: MF-MSMF050, AERO_FOOT:Fuse_1812_4532Metric_Pad1.30x3.40mm_HandSolder, symbol Device:Polyfuse
- added JP?: Wire, AERO_FOOT:Wire_16AWG, symbol AERO_custom_symbols:Wire
- added R?: RES 0603 10k 1%, symbol Device:R
- added R?: RES 0805 2 1%, Resistor_SMD:R_0805_2012Metric, symbol Device:R_US
- added S?: 100SP1T1B4M2QE, DigiKey_Lib:Toggle_Switch_100SP1T1B4M2QE, symbol Switch:SW_SPDT
- J11: value Conn_01x03 -> Header 100Mil 1x3
- J12: value Conn_02x03_Odd_Even -> Header ICSP
Connections:
- net +5V: now also R?.1
- net GND: now also JP?.1, S?.2 (B)
- new net COOLING_MODE: R?.2, S?.1 (A)
- no-connect marks 0 -> 1
Other:
- note added: "Assuming sensor gives pulse when magnet passes. These should go to timer pins (timer IN)"
- note added: "Button needs a pulldown resistor."
- note added: "Cap for areff, additional cap for VCC (there are 2 VCC pins)"
- note added: "Consider changeing to a fet."
- note added: "Consider fusing 5V out, I will put the part in if you think you should"
- note added: "Consider the following input protection and anti brownout circuit"
- note added: "Fuse before cap"
- note added: "I put in some led partnumbers, and checked resistances for any leds driven by resistors."
- note added: "Part numbers for right angle headers? Consider PH for some of these. Make sure parts are correct for right angle."
- note added: "Simpler way to wire: See left"
- note added: "To allow for grounding of the front metal"
- note added: "Why do string pots use 12V in?\nUse opamps to buffer, or change gain.\n They should be using 5V. We can talk about this."
- note added: "fuse should be on input not output"
- note added: "label on pcb"
- note added: "should be 0805 not 0603\n"
- note added: "what is TP14 and the power led for?"
Changed lines of the file:
@@
 P 10400 1400
 F 0 "J12" H 10450 1717 50  0000 C CNN
-F 1 "Conn_02x03_Odd_Even" H 10450 1626 50  0000 C CNN
+F 1 "Header ICSP" H 10450 1626 50  0000 C CNN
 F 2 "Connector_PinHeader_2.54mm:PinHeader_2x03_P2.54mm_Vertical" H 10400 1400 50  0001 C CNN
 F 3 "~" H 10400 1400 50  0001 C CNN
@@
 P 9350 5950
 F 0 "J11" H 9268 5625 50  0000 C CNN
-F 1 "Conn_01x03" H 9268 5716 50  0000 C CNN
+F 1 "Header 100Mil 1x3" H 9268 5716 50  0000 C CNN
 F 2 "Connector_PinHeader_2.54mm:PinHeader_1x03_P2.54mm_Vertical" H 9350 5950 50  0001 C CNN
 F 3 "~" H 9350 5950 50  0001 C CNN
@@
 Wire Wire Line
 	1600 2350 1450 2350
+Text Notes 5900 5100 0    50   ~ 0
+fuse should be on input not output
+Text Notes 5900 5200 0    50   ~ 0
+Fuse before cap
+Text Notes 2250 2750 0    50   ~ 0
+Consider changeing to a fet.
+Text Notes 1550 1100 0    50   ~ 0
+Button needs a pulldown resistor.
+Text Notes 1550 1200 0    50   ~ 0
+Part numbers for right angle headers? Consider PH for some of these. Make sure parts are correct for right angle.
+Text Notes 7300 6200 0    50   ~ 0
+what is TP14 and the power led for?
+Text Notes 7200 6350 0    50   ~ 0
+I put in some led partnumbers, and checked resistances for any leds driven by resistors.
+Text Notes 10100 5850 0    50   ~ 0
+label on pcb
+$Comp
+L AERO_custom_symbols:Wire JP?
+U 1 1 5E68041A
+P 13050 2650
+F 0 "JP?" V 13050 2838 50  0000 L CNN
+F 1 "Wire" H 13050 2800 50  0001 C CNN
+F 2 "AERO_FOOT:Wire_16AWG" H 13250 2650 50  0001 C CNN
+F 3 "~" H 13250 2650 50  0001 C CNN
+	1    13050 2650
+	0    1    1    0
+$EndComp
+$Comp
+L power:GND #PWR?
+U 1 1 5E680F1E
+P 13050 2650
+F 0 "#PWR?" H 13050 2400 50  0001 C CNN
+F 1 "GND" H 13055 2477 50  0000 C CNN
+F 2 "" H 13050 2650 50  0001 C CNN
+F 3 "" H 13050 2650 50  0001 C CNN
+	1    13050 2650
+	1    0    0    -1
+$EndComp
+Text Notes 12750 2400 0    50   ~ 0
+To allow for grounding of the front metal
+Text Notes 9150 4850 0    50   ~ 0
+Cap for areff, additional cap for VCC (there are 2 VCC pins)
+Text Notes 2350 4400 0    50   ~ 0
+Simpler way to wire: See left
+$Comp
+L Switch:SW_SPDT S?
+U 1 1 5E68AE8E
+P -1300 4050
+F 0 "S?" H -1300 4353 60  0000 C CNN
+F 1 "100SP1T1B4M2QE" H -1300 4247 60  0000 C CNN
+F 2 "DigiKey_Lib:Toggle_Switch_100SP1T1B4M2QE" H -1100 4250 60  0001 L CNN
+F 3 "http://spec_sheets.e-switch.com/specs/T111597.pdf" H -1100 4350 60  0001 L CNN
+F 4 "EG2355-ND" H -1100 4450 60  0001 L CNN "Digi-Key_PN"
+F 5 "100SP1T1B4M2QE" H -1100 4550 60  0001 L CNN "MPN"
+F 6 "Switches" H -1100 4650 60  0001 L CNN "Category"
+F 7 "Toggle Switches" H -1100 4750 60  0001 L CNN "Family"
+F 8 "http://spec_sheets.e-switch.com/specs/T111597.pdf" H -1100 4850 60  0001 L CNN "DK_Datasheet_Link"
+F 9 "/product-detail/en/e-switch/100SP1T1B4M2QE/EG2355-ND/378824" H -1100 4950 60  0001 L CNN "DK_Detail_Page"
+F 10 "SWITCH TOGGLE SPDT 5A 120V" H -1100 5050 60  0001 L CNN "Description"
+F 11 "E-Switch" H -1100 5150 60  0001 L CNN "Manufacturer"
+F 12 "Active" H -1100 5250 60  0001 L CNN "Status"
+	1    -1300 4050
+	1    0    0    -1
+$EndComp
+Text Label -500 3950 2    50   ~ 0
+COOLING_MODE
+$Comp
+L power:GND #PWR?
+U 1 1 5E68AE98
+P -1600 4200
+F 0 "#PWR?" H -1600 3950 50  0001 C CNN
+F 1 "GND" H -1595 4027 50  0000 C CNN
+F 2 "" H -1600 4200 50  0001 C CNN
+F 3 "" H -1600 4200 50  0001 C CNN
+	1    -1600 4200
+	1    0    0    -1
+$EndComp
+Wire Wire Line
+	-1600 4200 -1600 4050
+Wire Wire Line
+	-1600 4050 -1500 4050
+$Comp
+L Device:R R?
+U 1 1 5E691C08
+P -400 3800
+F 0 "R?" H -330 3846 50  0000 L CNN
+F 1 "RES 0603 10k 1%" H -330 3755 50  0000 L CNN
+F 2 "" V -470 3800 50  0001 C CNN
+F 3 "~" H -400 3800 50  0001 C CNN
+	1    -400 3800
+	1    0    0    -1
+$EndComp
+$Comp
+L power:+5V #PWR?
+U 1 1 5E6925E8
+P -400 3650
+F 0 "#PWR?" H -400 3500 50  0001 C CNN
+F 1 "+5V" H -385 3823 50  0000 C CNN
+F 2 "" H -400 3650 50  0001 C CNN
+F 3 "" H -400 3650 50  0001 C CNN
+	1    -400 3650
+	1    0    0    -1
+$EndComp
+Wire Wire Line
+	-1100 3950 -400 3950
+NoConn ~ -1100 4150
+Text Notes 3050 4800 0    50   ~ 0
+Why do string pots use 12V in?\nUse opamps to buffer, or change gain.\n They should be using 5V. We can talk about this.
+Text Notes 3100 5550 0    50   ~ 0
+Assuming sensor gives pulse when magnet passes. These should go to timer pins (timer IN)
+Text Notes 2800 6400 0    50   ~ 0
+Consider fusing 5V out, I will put the part in if you think you should
+$Comp
+L Device:Polyfuse F?
+U 1 1 5E6ACF8C
+P 3900 9400
+F 0 "F?" V 3675 9400 50  0000 C CNN
+F 1 "MF-MSMF050" V 3766 9400 50  0000 C CNN
+F 2 "AERO_FOOT:Fuse_1812_4532Metric_Pad1.30x3.40mm_HandSolder" H 3950 9200 50  0001 L CNN
+F 3 "~" H 3900 9400 50  0001 C CNN
+	1    3900 9400
+	0    1    1    0
+$EndComp
+Text Notes 2500 8700 0    50   ~ 0
+Consider the following input protection and anti brownout circuit
+$Comp
+L Device:R_US R?
+U 1 1 5E6BA7FB
+P 5100 9400
+F 0 "R?" V 4895 9400 50  0000 C CNN
+F 1 "RES 0805 2 1%" V 4986 9400 50  0000 C CNN
+F 2 "Resistor_SMD:R_0805_2012Metric" V 5140 9390 50  0001 C CNN
+F 3 "~" H 5100 9400 50  0001 C CNN
+	1    5100 9400
+	0    1    1    0
+$EndComp
+Text Notes 4800 9650 0    50   ~ 0
+should be 0805 not 0603\n
 $EndSCHEMATC
