File: dash-2019-2020/Right_rev2/right.sch (KiCad schematic (older format))
At the start: 34 parts, among them J1 JST-XH, J11 Conn_01x03, J12 Conn_02x03_Odd_Even, J13 JST-XH, J2 JST-XH, J3 AMPSEAL, J5 B5B-PH-SM4-TB(LF)(SN), J8 JST-XH, Q1 MMBT2222ALT1G, U1 R-78E5.0-1, U2 ATmega328P-AU

Commit message: Review dash
Parts:
- added C1: 0.1uF, Capacitor_SMD:C_0603_1608Metric, symbol Device:C
- added C2, C9: UUD1V331MNL1GS, Capacitor_SMD:CP_Elec_10x10, symbol Device:CP1
- added D2: B340A-13-F1, Diode_SMD:D_SMA_Handsoldering, symbol Device:D_Schottky
- added D9: SZMMSZ5243BT1G, Diode_SMD:D_SOD-123, symbol Device:D_Zener
- added F2: MF-MSMF050, AERO_FOOT:Fuse_1812_4532Metric_Pad1.30x3.40mm_HandSolder, symbol Device:Polyfuse
- added FB1: 742792097, AERO_FOOT:FB_0805, symbol Device:Ferrite_Bead
- added J4: 1-770966-0, AERO_FOOT:1-770966-0, symbol Connector_Generic:Conn_01x02
- added R10: RES 0805 2 1%, Resistor_SMD:R_0805_2012Metric_Pad1.15x1.40mm_HandSolder, symbol Device:R
- added R9: 10k, Resistor_SMD:R_0603_1608Metric_Pad1.05x0.95mm_HandSolder, symbol Device:R
- added S2: 100SP1T1B4M2QE, AERO_FOOT:Toggle_Switch_100SP1T1B4M2QE, symbol Switch:SW_SPDT
- D1: value LED -> SM0805YCL
- D4: value LED -> SM0805GCL
- D5: value LED -> SM0805HCL
- F1: value 1812L075/24 -> MF-MSMF050; footprint Fuse:Fuse_1812_4532Metric_Pad1.30x3.40mm_HandSolder -> AERO_FOOT:Fuse_1812_4532Metric_Pad1.30x3.40mm_HandSolder
- J11: value Conn_01x03 -> Header 1x3 0.1in
- J12: value Conn_02x03_Odd_Even -> Header 2x3 0.1in
- R1: value R_US -> RES 0603 10k 1%
- R2, R3: value 1k -> 1.5k
- R5: value 330 -> 1.5k
- S1: footprint DigiKey_Lib:Toggle_Switch_100SP1T1B4M2QE -> AERO_FOOT:Toggle_Switch_100SP1T1B4M2QE
- TH1: value Thermistor -> NCU18XH103F60RB
Connections:
- net +5V: now also R9.1
- net GND: now also C1.2, C2.2, C9.2, D9.2 (A), S2.2 (B)
- net SHUTDOWN_IN: now also J4.2 (Pin_2)
- net SHUTDOWN_OUT: now also J4.1 (Pin_1)
- new net COOLING_MODE: C1.1, R9.2, S2.1 (A)
- new net D+: D2.1 (K), D9.1 (K), FB1.2, R10.1
- new net F+: D2.2 (A), F2.1
- new net VCAP: C2.1, C9.1, R10.2
- no-connect marks 0 -> 1
Other:
- note added: "+12 In"
- note added: "0805"
- note added: "Consider reannotating when you finish"
- note added: "Currently in pull up config."
- note added: "Fuse should go before regulator. I changed \nfootprint and PN to a 500mA, due to buck \nconverter eff.\n\nSee the suggested topology below the sheet"
- note added: "Hall effect should go to timer input pins on atmega for easy pulse decoding"
- note added: "I skipped the usual common mode choke here for space, but normally it would be here."
- note added: "Label on board"
- note added: "Make sure all full correct parts are in asap after shipping board."
- note added: "Many of the test points are not necessary"
- note added: "Reset should ahve an RC timer on it. I can send example."
- note added: "TVS should be added to DAMPER lines and speed sensors\n"
- note added: "There is a much better (and easier) \nway to do this switch. You also need\n pullups/pulldowns. See left-offsheet."
- note added: "This should be the +12 net, and one incomming +12 should be made to +12_IN"
- note added: "To recom"
- note added: "Try to route MCU CLK. See info near switch"
- note added: "Why are string pots 12V? If the whole \nrange isn't used, this should be dealt with\n via an opamp. At a minimum, there s\nhould be a clamping diode to ensure\n 12V can't reach the MCU"
- note added: "add decap for aref, and 1 more cap, there are 2 vcc, 1 avcc"
- note added: "and recom decap"
- note added: "caps are for anti brownout"

Commit message: PCB layoutchanges
Parts:
- removed C2, C9: UUD1V331MNL1GS, Capacitor_SMD:CP_Elec_10x10, symbol Device:CP1
- removed D2: B340A-13-F1, Diode_SMD:D_SMA_Handsoldering, symbol Device:D_Schottky
- removed D9: SZMMSZ5243BT1G, Diode_SMD:D_SOD-123, symbol Device:D_Zener
- removed F2: MF-MSMF050, AERO_FOOT:Fuse_1812_4532Metric_Pad1.30x3.40mm_HandSolder, symbol Device:Polyfuse
- removed FB1: 742792097, AERO_FOOT:FB_0805, symbol Device:Ferrite_Bead
- removed R10: RES 0805 2 1%, Resistor_SMD:R_0805_2012Metric_Pad1.15x1.40mm_HandSolder, symbol Device:R
- removed S1: 100SP1T1B4M2QE, AERO_FOOT:Toggle_Switch_100SP1T1B4M2QE, symbol Switch:SW_SPDT
- removed TP11, TP12, TP13, TP15: TestPoint, TestPoint:TestPoint_Pad_D1.0mm, symbol Connector:TestPoint
- added D2, D3: SP0503BAHT, Package_TO_SOT_SMD:SOT-143, symbol Power_Protection:SP0503BAHT
- renumbered C3 to C2, C4 to C3, C5 to C4, C6 to C5, D3 to D1, D1 to D4, D4 to D5, D5 to D6, J8 to J2, J2 to J3, J13 to J4, J3 to J6, J4 to J7, J11 to J8, J12 to J9, R8 to R1, R9 to R2, R1 to R3, R5 to R4, R2 to R5, R3 to R6, S2 to S1, TP14 to TP1
Connections:
- net COOLING_MODE_1 is gone; now on net COOLING_MODE: U2.27 (PC4)
- net DAMPER_L: now also D3.3 (K)
- net DAMPER_R: now also D3.2 (K)
- net GND: now also D2.1 (A), D3.1 (A)
- net SHUTDOWN_IN: now also J7.1 (Pin_1); no longer J7.2 (Pin_2)
- net SHUTDOWN_OUT: now also J7.2 (Pin_2); no longer J7.1 (Pin_1)
- net SPEED_L: now also D2.2 (K)
- net SPEED_R: now also D2.3 (K)
- net COOLING_MODE_2: no longer names the net of U2.28 (PC5)
Other:
- note added: "String Pots have \n+5V in"
- note removed: "+12 In"
- note removed: "0805"
- note removed: "Consider reannotating when you finish"
- note removed: "Currently in pull up config."
- note removed: "Fuse should go before regulator. I changed \nfootprint and PN to a 500mA, due to buck \nconverter eff.\n\nSee the suggested topology below the sheet"
- note removed: "Hall effect should go to timer input pins on atmega for easy pulse decoding"
- note removed: "I skipped the usual common mode choke here for space, but normally it would be here."
- note removed: "Make sure all full correct parts are in asap after shipping board."
- note removed: "Many of the test points are not necessary"
- note removed: "Need pull ups/downs on \nSPEED_R/SPEED_L?"
- note removed: "Reset should ahve an RC timer on it. I can send example."
- note removed: "String Pots have \n+12V in"
- note removed: "TVS should be added to DAMPER lines and speed sensors\n"
- note removed: "There is a much better (and easier) \nway to do this switch. You also need\n pullups/pulldowns. See left-offsheet."
- note removed: "This should be the +12 net, and one incomming +12 should be made to +12_IN"
- note removed: "To recom"
- note removed: "Try to route MCU CLK. See info near switch"
- note removed: "Why are string pots 12V? If the whole \nrange isn't used, this should be dealt with\n via an opamp. At a minimum, there s\nhould be a clamping diode to ensure\n 12V can't reach the MCU"
- note removed: "add decap for aref, and 1 more cap, there are 2 vcc, 1 avcc"
- note removed: "and recom decap"
- note removed: "caps are for anti brownout"
- moved on the sheet: C1, R2, S1

Commit message: add notes for future
Parts:
- J5: value B5B-PH-SM4-TB(LF)(SN) -> S5B-PH-K-S(LF)(SN)
Other:
- note added: "Notes for future:\nFuse should be before Recom\nThere should be anti brownout caps and polarity protection\nConsider the "Power Switch" thing\nLook into better MCUs\nCreate common subschematics for CAN, Power supply, etc"
Changed lines of the file:
@@
 P 2050 1800
 F 0 "J5" H 1975 2225 50  0000 C CNN
-F 1 "B5B-PH-SM4-TB(LF)(SN)" H 1950 2125 50  0000 C CNN
+F 1 "S5B-PH-K-S(LF)(SN)" H 1950 2125 50  0000 C CNN
 F 2 "Connector_JST:JST_PH_S5B-PH-K_1x05_P2.00mm_Horizontal" H 2050 1800 50  0001 C CNN
 F 3 "~" H 2050 1800 50  0001 C CNN
@@
 	1    0    0    -1
 $EndComp
+Text Notes 700  8750 0    50   ~ 0
+Notes for future:\nFuse should be before Recom\nThere should be anti brownout caps and polarity protection\nConsider the "Power Switch" thing\nLook into better MCUs\nCreate common subschematics for CAN, Power supply, etc
 $EndSCHEMATC

Commit message: start documentation
Parts:
- D4: value SM0805YCL -> SM0805UYC
- R4: value 1.5k -> 150
Changed lines of the file:
@@
 P 7075 6000
 F 0 "D4" H 7068 5745 50  0000 C CNN
-F 1 "SM0805YCL" H 7068 5836 50  0000 C CNN
+F 1 "SM0805UYC" H 7068 5836 50  0000 C CNN
 F 2 "LED_SMD:LED_0805_2012Metric_Pad1.15x1.40mm_HandSolder" H 7075 6000 50  0001 C CNN
 F 3 "~" H 7075 6000 50  0001 C CNN
@@
 P 7075 5700
 F 0 "R4" H 7145 5746 50  0000 L CNN
-F 1 "1.5k" H 7145 5655 50  0000 L CNN
+F 1 "150" H 7145 5655 50  0000 L CNN
 F 2 "Resistor_SMD:R_0603_1608Metric_Pad1.05x0.95mm_HandSolder" V 7005 5700 50  0001 C CNN
 F 3 "~" H 7075 5700 50  0001 C CNN

Commit message: minor updates
Other:
- note added: "Direction Switch"
Changed lines of the file:
@@
 Text Notes 700  8750 0    50   ~ 0
 Notes for future:\nFuse should be before Recom\nThere should be anti brownout caps and polarity protection\nConsider the "Power Switch" thing\nLook into better MCUs\nCreate common subschematics for CAN, Power supply, etc
+Text Notes 1725 7025 0    50   ~ 0
+Direction Switch
 $EndSCHEMATC
