File: dash-2019-2020/Right_rev2/CANbus-interface.sch (KiCad schematic (older format))
At the start: 13 parts, among them U4 MCP2551-I-SN, U5 MCP2515-xSO, Y1 Resonator

Commit message: Review dash
Parts:
- added L1: SRF4532, AERO_FOOT:SRF4532-220Y, symbol Device:EMI_Filter_CommonMode
Other:
- note added: "Add cann termination resistor, consider\nadding RC circuits for reset pins (add a \ncap, value of 1uf-1nf, going to other\nvoltage rail) STRONGLY consider adding \nthe common mode choke I added above."
- note added: "None of the testpoints here are (strictly) needed"
- note added: "canh_in"
- note added: "canh_out"
- note added: "canl_in"
- note added: "canl_out"
Changed lines of the file:
@@
 Wire Wire Line
 	6750 3250 7450 3250
+Text Notes 8200 3950 0    50   ~ 0
+None of the testpoints here are (strictly) needed
+Text Notes 4950 2550 0    50   ~ 0
+Add cann termination resistor, consider\nadding RC circuits for reset pins (add a \ncap, value of 1uf-1nf, going to other\nvoltage rail) STRONGLY consider adding \nthe common mode choke I added above.
+$Comp
+L Device:EMI_Filter_CommonMode L1
+U 1 1 5E6B7D9A
+P 5200 2000
+F 0 "L1" H 5200 2281 50  0000 C CNN
+F 1 "SRF4532" H 5200 2190 50  0000 C CNN
+F 2 "AERO_FOOT:SRF4532-220Y" H 5200 2040 50  0001 C CNN
+F 3 "~" H 5200 2040 50  0001 C CNN
+	1    5200 2000
+	1    0    0    -1
+$EndComp
+Text Notes 5550 1900 0    50   ~ 0
+canh_in
+Text Notes 4600 1900 0    50   ~ 0
+canh_out
+Text Notes 5550 2100 0    50   ~ 0
+canl_in
+Text Notes 4600 2100 0    50   ~ 0
+canl_out
 $EndSCHEMATC

Commit message: PCB layoutchanges
Parts:
- removed TP1, TP2, TP6, TP7, TP8, TP9: TestPoint, TestPoint:TestPoint_Pad_D1.0mm, symbol Connector:TestPoint
- renumbered C7 to C6, C8 to C7, R6 to R7, R7 to R8, U4 to U3, U5 to U4
Connections:
- net CAN+: now also L1.2; no longer U3.7 (CANH)
- net CAN-: now also L1.4; no longer U3.6 (CANL)
- net at L1.1: now also U3.7 (CANH)
- net at L1.3: now also U3.6 (CANL)
Other:
- note removed: "Add cann termination resistor, consider\nadding RC circuits for reset pins (add a \ncap, value of 1uf-1nf, going to other\nvoltage rail) STRONGLY consider adding \nthe common mode choke I added above."
- note removed: "None of the testpoints here are (strictly) needed"
- note removed: "canh_in"
- note removed: "canh_out"
- note removed: "canl_in"
- note removed: "canl_out"
- moved on the sheet: L1
