File: dash-2019-2020/Right_rev2/right.kicad_pcb (KiCad board)
At the start: 2 copper layers, 94 x 63.5 mm, 52 parts, among them J1 JST-XH, J11 Conn_01x03, J12 Conn_02x03_Odd_Even, J13 JST-XH, J2 JST-XH, J3 AMPSEAL, J5 B5B-PH-SM4-TB(LF)(SN), J8 JST-XH, Q1 MMBT2222ALT1G, U1 R-78E5.0-0.5, U2 ATmega328P-AU, U3 STP16CP05, U4 MCP2551-I-SN, U5 MCP2515-xSO, Y1 Resonator

Commit message: Minor Layout Changes
Parts:
- moved J5 2.79 mm to (180.3, 112.0)
Routing:
- net +5V: track 355.5 -> 383.8 mm
- net /BRAKE: track 66.5 -> 70.3 mm
- net ~FAULT_IND_3: track 57.7 -> 60.5 mm
- net ~FAULT_IND_2: track 50.9 -> 53.7 mm
- net ~FAULT_IND_1: track 51.4 -> 54.2 mm

Commit message: layout changes
Parts:
- added R8: 1k, Resistor_SMD:R_0603_1608Metric_Pad1.05x0.95mm_HandSolder, F.Cu at (168.4, 95.8)
- U1: value R-78E5.0-0.5 -> R-78E5.0-1
- moved Q1 4.33 mm to (168.4, 91.4)
Connections:
- J8 pad 2: +5V -> +12V
- Q1 pad 3: Net-(J8-Pad1) -> Net-(Q1-Pad3)
Routing:
- net +12V: track 6.92 -> 88.0 mm
- net /RTD_IND: track 33.9 -> 29.5 mm
- net /BRAKE: track 70.3 -> 67.5 mm, vias 1 -> 2
- net Net-(Q1-Pad3): track 0.00 -> 2.44 mm
- net +5V: track 383.8 -> 384.7 mm
- net Net-(J8-Pad1): track 15.8 -> 15.2 mm
- net GND: vias 20 -> 48

Commit message: layout changes
Parts:
- added J4: 1-770966-0, AERO_FOOT:TE_MATE-N-LOK_1-770866-x_1x02_P4.14mm_Vertical, B.Cu at (213.0, 113.3)
- moved H1 8.21 mm to (227.8, 105.7)
Connections:
- J3 pad 15: GND -> /DAMPER_L
- J3 pad 2: +12V -> /SHUTDOWN_IN
- J3 pad 23: GND -> /DAMPER_R
- J3 pad 3: +12V -> /SHUTDOWN_OUT
- J3 pad 5: /DAMPER_R -> +12V
- J3 pad 6: /DAMPER_L -> +12V
Routing:
- net /SHUTDOWN_OUT: track 0.00 -> 53.7 mm
- net /SHUTDOWN_IN: track 0.00 -> 45.1 mm
- net +5V: track 384.7 -> 400.8 mm
- net /DAMPER_R: track 52.8 -> 42.7 mm
- net /DAMPER_L: track 44.8 -> 40.5 mm
- net GND: vias 48 -> 42

Commit message: Review dash
Parts:
- F1: footprint Fuse:Fuse_1812_4532Metric_Pad1.30x3.40mm_HandSolder -> AERO_FOOT:Fuse_1812_4532Metric_Pad1.30x3.40mm_HandSolder
- S1: footprint DigiKey_Lib:Toggle_Switch_100SP1T1B4M2QE -> AERO_FOOT:Toggle_Switch_100SP1T1B4M2QE
Other:
- board text added: "Add a few more ground vias throughout"
- board text added: "All comments are on Dwgs.User"
- board text added: "Careful with acute angles!!"
- board text added: "Check CAN trace widths. I can calculate for you if you wish."
- board text added: "Consider vias for ground pours"
- board text added: "Considre a screw hole near here for stability near LEDs."
- board text added: "For future ref: can trace widths do not need to match. Copy diff. pair settings from other board"
- board text added: "Mark TX, RX, GND. Make sure order matches with the other board."

Commit message: PCB layoutchanges
Parts:
- removed the J4 at (213.0, 113.3)
- removed the TP1 at (152.3, 97.7)
- removed TP11, TP12, TP13, TP15, TP2, TP6, TP7, TP8, TP9: TestPoint, TestPoint:TestPoint_Pad_D1.0mm
- added C1: 0.1uF, Capacitor_SMD:C_0603_1608Metric, F.Cu at (189.0, 60.5)
- added D2: SP0503BAHT, Package_TO_SOT_SMD:SOT-143, F.Cu at (163.6, 90.9)
- added D3: SP0503BAHT, Package_TO_SOT_SMD:SOT-143, F.Cu at (172.2, 80.4)
- added G***: LOGO, AERO_CUSTOM:AERO_Logo_10x4mm, B.Cu at (219.1, 116.8)
- added GND: TestPoint_Plated_Hole_D2.0mm, TestPoint:TestPoint_Plated_Hole_D2.0mm, F.Cu at (144.8, 73.0)
- added J7: 1-770966-0, AERO_FOOT:1-770966-0, B.Cu at (220.2, 106.0)
- added L1: SRF4532, AERO_FOOT:SRF4532-220Y, F.Cu at (184.4, 103.1)
- added R2: 10k, Resistor_SMD:R_0603_1608Metric_Pad1.05x0.95mm_HandSolder, F.Cu at (186.6, 60.5)
- D4: renamed from D1; value LED -> SM0805YCL
- D5: renamed from D4; value LED -> SM0805GCL
- D6: renamed from D5; value LED -> SM0805HCL
- F1: value 1812L075/24 -> MF-MSMF050
- J8: renamed from J11; value Conn_01x03 -> Header 1x3 0.1in
- J9: renamed from J12; value Conn_02x03_Odd_Even -> Header 2x3 0.1in
- R3: renamed from R1; value R_US -> RES 0603 10k 1%
- R4: renamed from R5; value 330 -> 1.5k
- R5: renamed from R2; value 1k -> 1.5k
- R6: renamed from R3; value 1k -> 1.5k
- TH1: value Thermistor -> NCU18XH103F60RB
- moved H1 21.9 mm to (207.3, 113.2)
- moved S1 0.40 mm to (194.1, 67.4)
- renumbered C3 to C2, C4 to C3, C5 to C4, C6 to C5, C7 to C6, C8 to C7, C11 to C8, D3 to D1, D6 to D7, D7 to D8, D8 to D9, J8 to J2, J2 to J3, J13 to J4, J3 to J6, R8 to R1, R6 to R7, R7 to R8, R4 to R9, TP14 to TP1, U4 to U3, U5 to U4, U3 to U5
Connections:
- net /COOLING_MODE_1 renamed /COOLING_MODE
- S1 pad 3: /COOLING_MODE_2 -> (no net)
- U2 pad 28: /COOLING_MODE_2 -> (no net)
- U3 pad 6: /CAN- -> Net-(L1-Pad3)
- U3 pad 7: /CAN+ -> Net-(L1-Pad1)
Routing:
- net /COOLING_MODE_2: track 63.2 -> 0.00 mm
- net +5V: track 400.8 -> 423.5 mm
- net /CAN+: track 43.6 -> 21.8 mm
- net /CAN-: track 43.5 -> 23.2 mm
- net Net-(L1-Pad1): track 0.00 -> 17.7 mm
- net Net-(L1-Pad3): track 0.00 -> 17.4 mm
- net /DAMPER_R: track 42.7 -> 59.5 mm
- net /DAMPER_L: track 40.5 -> 52.7 mm
- net /COOLING_MODE: track 60.4 -> 72.1 mm
- net Net-(U4-Pad7): track 11.8 -> 4.55 mm
- net /LED_CLK: track 18.0 -> 10.9 mm, vias 1 -> 0
- net /~LED_OE: track 27.0 -> 20.1 mm
- net /~LED_LE: track 15.4 -> 10.2 mm, vias 1 -> 0
- net /SCK: track 43.4 -> 38.4 mm, vias 1 -> 0
- net /LED_SDI: track 16.2 -> 11.8 mm, vias 1 -> 0
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Other:
- board text added: "GND"
- board text added: "TX"
- board text removed: "Add a few more ground vias throughout"
- board text removed: "All comments are on Dwgs.User"
- board text removed: "Careful with acute angles!!"
- board text removed: "Check CAN trace widths. I can calculate for you if you wish."
- board text removed: "Consider vias for ground pours"
- board text removed: "Considre a screw hole near here for stability near LEDs."
- board text removed: "For future ref: can trace widths do not need to match. Copy diff. pair settings from other board"
- board text removed: "Mark TX, RX, GND. Make sure order matches with the other board."
