File: dash-2019-2020/Right_rev2/LEDs.sch (KiCad schematic (older format))
At the start: 6 parts, among them U3 STP16CP05

Commit message: PCB layoutchanges
Parts:
- renumbered C11 to C8, D6 to D7, D7 to D8, D8 to D9, R4 to R9, U3 to U5
Changed lines of the file:
@@
 P 6350 3700
 AR Path="/5DF93ADB" Ref="U?"  Part="1"
-AR Path="/5DF8F110/5DF93ADB" Ref="U3"  Part="1"
-F 0 "U3" H 6250 4800 50  0000 C CNN
+AR Path="/5DF8F110/5DF93ADB" Ref="U5"  Part="1"
+F 0 "U5" H 6250 4800 50  0000 C CNN
 F 1 "STP16CP05" H 6600 4800 50  0000 C CNN
 F 2 "Package_SO:TSSOP-24_4.4x7.8mm_P0.65mm" H 6350 3700 50  0001 C CNN
@@
 P 4100 3600
 AR Path="/5DF93AE1" Ref="D?"  Part="1"
-AR Path="/5DF8F110/5DF93AE1" Ref="D6"  Part="1"
-F 0 "D6" H 4100 4097 50  0000 C CNN
+AR Path="/5DF8F110/5DF93AE1" Ref="D7"  Part="1"
+F 0 "D7" H 4100 4097 50  0000 C CNN
 F 1 "COOLING_IND_1" H 4100 4006 50  0000 C CNN
 F 2 "LED_THT:LED_D5.0mm-4_RGB" H 4100 3550 50  0001 C CNN
@@
 P 3900 3600
 AR Path="/5DF93B0B" Ref="#PWR?"  Part="1"
-AR Path="/5DF8F110/5DF93B0B" Ref="#PWR049"  Part="1"
-F 0 "#PWR049" H 3900 3450 50  0001 C CNN
+AR Path="/5DF8F110/5DF93B0B" Ref="#PWR059"  Part="1"
+F 0 "#PWR059" H 3900 3450 50  0001 C CNN
 F 1 "+5V" V 3915 3728 50  0000 L CNN
 F 2 "" H 3900 3600 50  0001 C CNN
@@
 P 4100 4500
 AR Path="/5DF93B35" Ref="D?"  Part="1"
-AR Path="/5DF8F110/5DF93B35" Ref="D7"  Part="1"
-F 0 "D7" H 4100 4997 50  0000 C CNN
+AR Path="/5DF8F110/5DF93B35" Ref="D8"  Part="1"
+F 0 "D8" H 4100 4997 50  0000 C CNN
 F 1 "COOLING_IND_2" H 4100 4906 50  0000 C CNN
 F 2 "LED_THT:LED_D5.0mm-4_RGB" H 4100 4450 50  0001 C CNN
@@
 P 3900 4500
 AR Path="/5DF93B3B" Ref="#PWR?"  Part="1"
-AR Path="/5DF8F110/5DF93B3B" Ref="#PWR050"  Part="1"
-F 0 "#PWR050" H 3900 4350 50  0001 C CNN
+AR Path="/5DF8F110/5DF93B3B" Ref="#PWR060"  Part="1"
+F 0 "#PWR060" H 3900 4350 50  0001 C CNN
 F 1 "+5V" V 3915 4628 50  0000 L CNN
 F 2 "" H 3900 4500 50  0001 C CNN
@@
 P 4100 5400
 AR Path="/5DF93B47" Ref="D?"  Part="1"
-AR Path="/5DF8F110/5DF93B47" Ref="D8"  Part="1"
-F 0 "D8" H 4100 5897 50  0000 C CNN
+AR Path="/5DF8F110/5DF93B47" Ref="D9"  Part="1"
+F 0 "D9" H 4100 5897 50  0000 C CNN
 F 1 "COOLING_IND_3" H 4100 5806 50  0000 C CNN
 F 2 "LED_THT:LED_D5.0mm-4_RGB" H 4100 5350 50  0001 C CNN
@@
 P 3900 5400
 AR Path="/5DF93B4D" Ref="#PWR?"  Part="1"
-AR Path="/5DF8F110/5DF93B4D" Ref="#PWR051"  Part="1"
-F 0 "#PWR051" H 3900 5250 50  0001 C CNN
+AR Path="/5DF8F110/5DF93B4D" Ref="#PWR061"  Part="1"
+F 0 "#PWR061" H 3900 5250 50  0001 C CNN
 F 1 "+5V" V 3915 5528 50  0000 L CNN
 F 2 "" H 3900 5400 50  0001 C CNN
@@
 P 6350 2600
 AR Path="/5DF93B6B" Ref="#PWR?"  Part="1"
-AR Path="/5DF8F110/5DF93B6B" Ref="#PWR056"  Part="1"
-F 0 "#PWR056" H 6350 2450 50  0001 C CNN
+AR Path="/5DF8F110/5DF93B6B" Ref="#PWR062"  Part="1"
+F 0 "#PWR062" H 6350 2450 50  0001 C CNN
 F 1 "+5V" H 6365 2773 50  0000 C CNN
 F 2 "" H 6350 2600 50  0001 C CNN
@@
 P 7000 3200
 AR Path="/5DF93B77" Ref="R?"  Part="1"
-AR Path="/5DF8F110/5DF93B77" Ref="R4"  Part="1"
-F 0 "R4" V 7200 3200 50  0000 C CNN
+AR Path="/5DF8F110/5DF93B77" Ref="R9"  Part="1"
+F 0 "R9" V 7200 3200 50  0000 C CNN
 F 1 "1k" V 7100 3200 50  0000 C CNN
 F 2 "Resistor_SMD:R_0603_1608Metric" V 7040 3190 50  0001 C CNN
@@
 P 7300 3300
 AR Path="/5DF93B7E" Ref="#PWR?"  Part="1"
-AR Path="/5DF8F110/5DF93B7E" Ref="#PWR059"  Part="1"
-F 0 "#PWR059" H 7300 3050 50  0001 C CNN
+AR Path="/5DF8F110/5DF93B7E" Ref="#PWR064"  Part="1"
+F 0 "#PWR064" H 7300 3050 50  0001 C CNN
 F 1 "GND" H 7305 3127 50  0000 C CNN
 F 2 "" H 7300 3300 50  0001 C CNN
@@
 P 6350 4800
 AR Path="/5DF93B86" Ref="#PWR?"  Part="1"
-AR Path="/5DF8F110/5DF93B86" Ref="#PWR057"  Part="1"
-F 0 "#PWR057" H 6350 4550 50  0001 C CNN
+AR Path="/5DF8F110/5DF93B86" Ref="#PWR063"  Part="1"
+F 0 "#PWR063" H 6350 4550 50  0001 C CNN
 F 1 "GND" H 6355 4627 50  0000 C CNN
 F 2 "" H 6350 4800 50  0001 C CNN
@@
 	5950 2800 5400 2800
 $Comp
-L Device:C_Small C11
+L Device:C_Small C8
 U 1 1 5E3DC12C
 P 8000 2950
-F 0 "C11" H 8092 2996 50  0000 L CNN
+F 0 "C8" H 8092 2996 50  0000 L CNN
 F 1 "0.1u" H 8092 2905 50  0000 L CNN
 F 2 "Capacitor_SMD:C_0603_1608Metric" H 8000 2950 50  0001 C CNN
@@
 $EndComp
 $Comp
-L power:+5V #PWR0105
+L power:+5V #PWR065
 U 1 1 5E3DDE79
 P 8000 2850
-F 0 "#PWR0105" H 8000 2700 50  0001 C CNN
+F 0 "#PWR065" H 8000 2700 50  0001 C CNN
 F 1 "+5V" H 8015 3023 50  0000 C CNN
 F 2 "" H 8000 2850 50  0001 C CNN
@@
 $EndComp
 $Comp
-L power:GND #PWR0106
+L power:GND #PWR066
 U 1 1 5E3DE531
 P 8000 3050
-F 0 "#PWR0106" H 8000 2800 50  0001 C CNN
+F 0 "#PWR066" H 8000 2800 50  0001 C CNN
 F 1 "GND" H 8005 2877 50  0000 C CNN
 F 2 "" H 8000 3050 50  0001 C CNN
